File: Pannel/Pannel.kicad_sch (KiCad schematic)
At the start: 126 parts

Commit message: 構成図追加
Parts:
- removed C? (x2): 4.7uF, Capacitor_SMD:C_0603_1608Metric, symbol Device:C
- removed J?: Conn_01x10_Female, Connector_IDC:IDC-Header_2x05_P2.54mm_Horizontal, symbol Connector:Conn_01x10_Female
- added C3, C6: 10uF, Capacitor_SMD:C_0805_2012Metric_Pad1.18x1.45mm_HandSolder, symbol Device:C
- added J?: Conn_01x10_Male, BoxHeader_1.27mm:BoxHeader_2x05_P1.27mm_Vertical_SMD, symbol Connector:Conn_01x10_Male
- D8: renamed from D?; value MA10EB045 -> ?; footprint Diode_Schottky:DO-221BC -> (none)
- JP1, JP2: renamed from JP?; footprint (none) -> Jumper:SolderJumper-3_P2.0mm_Open_TrianglePad1.0x1.5mm_NumberLabels
- L1: renamed from L?; footprint (none) -> Inductor_Power:ETQ-P4M_KVK
- Q11, Q13, Q14, Q6, Q9: renamed from Q?; value 2PB709AR -> S8050; footprint Package_TO_SOT_SMD:SC-59_Handsoldering -> Package_TO_SOT_SMD:SOT-23
- Q5: renamed from Q?; footprint Package_TO_SOT_SMD:SC-59_Handsoldering -> Package_TO_SOT_SMD:SOT-23
- RV1: renamed from RV?; footprint (none) -> Potentiometer:PVZ3A
- SW3: renamed from SW?; footprint (none) -> Slide_Switch:SW_Slide_SPDT_White
- Y1: renamed from Y?; footprint (none) -> Crystal:Crystal_SMD_HC49-SD_HandSoldering
- gave numbers to parts that had none: 110
Connections:
- net +5V: now also C6.1
- net 3.3VBUS: now also J?.1 (Pin_1)
- net GND: now also C3.2, C6.2, J?.4 (Pin_4)
- net NRST: now also J?.6 (Pin_6)
- net STLinkRX: now also J?.9 (Pin_9)
- net STLinkTX: now also J?.8 (Pin_8)
- net TCK: now also J?.3 (Pin_3)
- net TMS: now also J?.5 (Pin_5)
- net at D5.1 (K), U1.6 (Vin), U1.7 (Ipk): now also C3.1
- no-connect marks 19 -> 5

Commit message: diagram_SmallPW
Parts:
- removed C1, C10: 4.7uF, Capacitor_SMD:C_0603_1608Metric, symbol Device:C
- added C? (x2): 1uF, Capacitor_SMD:C_0402_1005Metric, symbol Device:C
Connections:
- net 3.3VSYS: now also C?.1
- net S-S: now also C?.1
- net at Q3.1 (G), R8.2, R9.1: now also C?.2
- net at Q10.1 (G), R30.2, R31.1: now also C?.2
Changed lines of the file:
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@@
     (pin "1")
-  )
-  (symbol (lib_id "Device:C") (at 254 147.32 0) (unit 1)
-    (in_bom yes) (on_board yes) (fields_autoplaced)
-    (property "Reference" "C10" (id 0) (at 257.81 146.0499 0)
-      (effects (font (size 1.27 1.27)) (justify left))
-    )
-    (property "Value" "4.7uF" (id 1) (at 257.81 148.5899 0)
-      (effects (font (size 1.27 1.27)) (justify left))
-    )
-    (property "Footprint" "Capacitor_SMD:C_0603_1608Metric" (id 2) (at 254.9652 151.13 0)
-      (effects (font (size 1.27 1.27)) hide)
-    )
-    (property "Datasheet" "~" (id 3) (at 254 147.32 0)
-      (effects (font (size 1.27 1.27)) hide)
-    )
-    (pin "1")
-    (pin "2")
   )
   (symbol (lib_id "power:GND") (at 365.76 93.98 0) (mirror y) (unit 1)
@@
     (pin "1")
   )
+  (symbol (lib_id "Device:C") (at 71.12 137.16 0) (unit 1)
+    (in_bom yes) (on_board yes) (fields_autoplaced)
+    (property "Reference" "C?" (id 0) (at 74.93 135.8899 0)
+      (effects (font (size 1.27 1.27)) (justify left))
+    )
+    (property "Value" "1uF" (id 1) (at 74.93 138.4299 0)
+      (effects (font (size 1.27 1.27)) (justify left))
+    )
+    (property "Footprint" "Capacitor_SMD:C_0402_1005Metric" (id 2) (at 72.0852 140.97 0)
+      (effects (font (size 1.27 1.27)) hide)
+    )
+    (property "Datasheet" "~" (id 3) (at 71.12 137.16 0)
+      (effects (font (size 1.27 1.27)) hide)
+    )
+    (pin "1")
+    (pin "2")
+  )
   (symbol (lib_id "Switch:SW_SPST") (at 259.08 248.92 0) (unit 1)
     (in_bom yes) (on_board yes)
@@
     )
     (property "Datasheet" "~" (id 3) (at 154.94 157.48 0)
-      (effects (font (size 1.27 1.27)) hide)
-    )
-    (pin "1")
-    (pin "2")
-  )
-  (symbol (lib_id "Device:C") (at 71.12 137.16 0) (unit 1)
-    (in_bom yes) (on_board yes) (fields_autoplaced)
-    (property "Reference" "C1" (id 0) (at 74.93 135.8899 0)
-      (effects (font (size 1.27 1.27)) (justify left))
-    )
-    (property "Value" "4.7uF" (id 1) (at 74.93 138.4299 0)
-      (effects (font (size 1.27 1.27)) (justify left))
-    )
-    (property "Footprint" "Capacitor_SMD:C_0603_1608Metric" (id 2) (at 72.0852 140.97 0)
-      (effects (font (size 1.27 1.27)) hide)
-    )
-    (property "Datasheet" "~" (id 3) (at 71.12 137.16 0)
       (effects (font (size 1.27 1.27)) hide)
     )
@@
     (pin "1")
   )
+  (symbol (lib_id "Device:C") (at 254 147.32 0) (unit 1)
+    (in_bom yes) (on_board yes) (fields_autoplaced)
+    (property "Reference" "C?" (id 0) (at 257.81 146.0499 0)
+      (effects (font (size 1.27 1.27)) (justify left))
+    )
+    (property "Value" "1uF" (id 1) (at 257.81 148.5899 0)
+      (effects (font (size 1.27 1.27)) (justify left))
+    )
+    (property "Footprint" "Capacitor_SMD:C_0402_1005Metric" (id 2) (at 254.9652 151.13 0)
+      (effects (font (size 1.27 1.27)) hide)
+    )
+    (property "Datasheet" "~" (id 3) (at 254 147.32 0)
+      (effects (font (size 1.27 1.27)) hide)
+    )
+    (pin "1")
+    (pin "2")
+  )
   (symbol (lib_id "Device:Q_PMOS_GSD") (at 154.94 144.78 270) (mirror x) (unit 1)
     (in_bom yes) (on_board yes) (fields_autoplaced)
@@
       (reference "#PWR058") (unit 1) (value "GND") (footprint "")
     )
-    (path "/c7ee1ac1-3707-48f9-90c3-d3b71e642d3b"
-      (reference "C1") (unit 1) (value "4.7uF") (footprint "Capacitor_SMD:C_0603_1608Metric")
-    )
     (path "/67c490cc-fc2c-4fab-9127-c49a9a5a1dc6"
       (reference "C2") (unit 1) (value "0.1uF") (footprint "Capacitor_SMD:C_0402_1005Metric")
@@
       (reference "C9") (unit 1) (value "22pF") (footprint "Capacitor_SMD:C_0603_1608Metric")
     )
-    (path "/5c21c013-b35e-4392-a637-b97b44708c4f"
-      (reference "C10") (unit 1) (value "4.7uF") (footprint "Capacitor_SMD:C_0603_1608Metric")
-    )
     (path "/fb026700-6304-4c85-b7fa-1f1e7a63a43a"
       (reference "C11") (unit 1) (value "1uF") (footprint "Capacitor_SMD:C_0402_1005Metric")
@@
       (reference "C18") (unit 1) (value "0.1uF") (footprint "Capacitor_SMD:C_0402_1005Metric")
     )
+    (path "/b6840320-619e-43d4-96f6-547c766d63b2"
+      (reference "C?") (unit 1) (value "1uF") (footprint "Capacitor_SMD:C_0402_1005Metric")
+    )
+    (path "/f85c989d-562e-47b3-83cb-ab114c33cb01"
+      (reference "C?") (unit 1) (value "1uF") (footprint "Capacitor_SMD:C_0402_1005Metric")
+    )
     (path "/3ed5ee36-eed7-4c90-9b4e-319b8feaa820"

Commit message: 進捗
Parts:
- C3, C6: footprint Capacitor_SMD:C_0805_2012Metric_Pad1.18x1.45mm_HandSolder -> Capacitor_SMD:C_0805_2012Metric
- D1, D11: value SBR1A40SA -> 1N5819WS; footprint Diode_SMD:D_SMA_Handsoldering -> Diode_SMD:D_SOD-323_HandSoldering
- D7: value SBR1A40SA -> SS2040FL; footprint Diode_SMD:D_SMA_Handsoldering -> Diode_SMD:D_SOD-123
- gave numbers to parts that had none: 3
Changed lines of the file:
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@@
       (effects (font (size 1.27 1.27)) (justify left))
     )
-    (property "Footprint" "Capacitor_SMD:C_0805_2012Metric_Pad1.18x1.45mm_HandSolder" (id 2) (at 206.7052 97.79 0)
+    (property "Footprint" "Capacitor_SMD:C_0805_2012Metric" (id 2) (at 206.7052 97.79 0)
       (effects (font (size 1.27 1.27)) hide)
     )
@@
     (pin "9")
   )
-  (symbol (lib_name "D_Schottky_3") (lib_id "Device:D_Schottky") (at 93.98 149.86 270) (unit 1)
+  (symbol (lib_name "D_Schottky_1") (lib_id "Device:D_Schottky") (at 93.98 149.86 270) (unit 1)
     (in_bom yes) (on_board yes)
     (property "Reference" "D1" (id 0) (at 88.9 154.94 90)
       (effects (font (size 1.27 1.27)) (justify left))
     )
-    (property "Value" "SBR1A40SA" (id 1) (at 88.9 157.48 90)
-      (effects (font (size 1.27 1.27)) (justify left))
-    )
-    (property "Footprint" "Diode_SMD:D_SMA_Handsoldering" (id 2) (at 93.98 149.86 0)
+    (property "Value" "1N5819WS" (id 1) (at 88.9 157.48 90)
+      (effects (font (size 1.27 1.27)) (justify left))
+    )
+    (property "Footprint" "Diode_SMD:D_SOD-323_HandSoldering" (id 2) (at 93.98 149.86 0)
       (effects (font (size 1.27 1.27)) hide)
     )
@@
     (in_bom yes) (on_board yes) (fields_autoplaced)
     (property "Reference" "D11" (id 0) (at 279.0825 67.31 0))
-    (property "Value" "SBR1A40SA" (id 1) (at 279.0825 69.85 0))
-    (property "Footprint" "Diode_SMD:D_SMA_Handsoldering" (id 2) (at 279.4 73.66 0)
+    (property "Value" "1N5819WS" (id 1) (at 279.0825 69.85 0))
+    (property "Footprint" "Diode_SMD:D_SOD-323_HandSoldering" (id 2) (at 279.4 73.66 0)
       (effects (font (size 1.27 1.27)) hide)
     )
@@
   (symbol (lib_id "Device:C") (at 71.12 137.16 0) (unit 1)
     (in_bom yes) (on_board yes) (fields_autoplaced)
-    (property "Reference" "C?" (id 0) (at 74.93 135.8899 0)
+    (property "Reference" "C1" (id 0) (at 74.93 135.8899 0)
       (effects (font (size 1.27 1.27)) (justify left))
     )
@@
       (effects (font (size 1.27 1.27)) (justify left))
     )
-    (property "Footprint" "Capacitor_SMD:C_0805_2012Metric_Pad1.18x1.45mm_HandSolder" (id 2) (at 135.5852 95.25 0)
+    (property "Footprint" "Capacitor_SMD:C_0805_2012Metric" (id 2) (at 135.5852 95.25 0)
       (effects (font (size 1.27 1.27)) hide)
     )
@@
     (pin "2")
   )
-  (symbol (lib_name "D_Schottky_3") (lib_id "Device:D_Schottky") (at 172.72 81.28 0) (unit 1)
-    (in_bom yes) (on_board yes)
-    (property "Reference" "D7" (id 0) (at 172.72 83.82 0))
-    (property "Value" "SBR1A40SA" (id 1) (at 172.72 86.36 0))
-    (property "Footprint" "Diode_SMD:D_SMA_Handsoldering" (id 2) (at 172.72 81.28 0)
-      (effects (font (size 1.27 1.27)) hide)
-    )
-    (property "Datasheet" "~" (id 3) (at 172.72 81.28 0)
-      (effects (font (size 1.27 1.27)) hide)
-    )
-    (pin "1")
-    (pin "2")
-  )
   (symbol (lib_id "power:GND") (at 548.64 134.62 0) (mirror y) (unit 1)
     (in_bom yes) (on_board yes)
@@
   (symbol (lib_id "Connector:Conn_01x10_Male") (at 71.12 246.38 0) (unit 1)
     (in_bom yes) (on_board yes) (fields_autoplaced)
-    (property "Reference" "J?" (id 0) (at 71.755 231.14 0))
+    (property "Reference" "J3" (id 0) (at 71.755 231.14 0))
     (property "Value" "Conn_01x10_Male" (id 1) (at 71.755 233.68 0))
     (property "Footprint" "BoxHeader_1.27mm:BoxHeader_2x05_P1.27mm_Vertical_SMD" (id 2) (at 71.12 246.38 0)
@@
   (symbol (lib_id "Device:C") (at 254 147.32 0) (unit 1)
     (in_bom yes) (on_board yes) (fields_autoplaced)
-    (property "Reference" "C?" (id 0) (at 257.81 146.0499 0)
+    (property "Reference" "C10" (id 0) (at 257.81 146.0499 0)
       (effects (font (size 1.27 1.27)) (justify left))
     )
@@
     (pin "1")
   )
+  (symbol (lib_id "Device:D_Schottky") (at 172.72 81.28 0) (unit 1)
+    (in_bom yes) (on_board yes)
+    (property "Reference" "D7" (id 0) (at 172.72 86.36 0))
+    (property "Value" "SS2040FL" (id 1) (at 172.72 83.82 0))
+    (property "Footprint" "Diode_SMD:D_SOD-123" (id 2) (at 172.72 81.28 0)
+      (effects (font (size 1.27 1.27)) hide)
+    )
+    (property "Datasheet" "~" (id 3) (at 172.72 81.28 0)
+      (effects (font (size 1.27 1.27)) hide)
+    )
+    (pin "1")
+    (pin "2")
+  )
   (symbol (lib_id "Device:R") (at 144.78 157.48 180) (unit 1)
     (in_bom yes) (on_board yes) (fields_autoplaced)
@@
       (reference "#PWR058") (unit 1) (value "GND") (footprint "")
     )
+    (path "/b6840320-619e-43d4-96f6-547c766d63b2"
+      (reference "C1") (unit 1) (value "1uF") (footprint "Capacitor_SMD:C_0402_1005Metric")
+    )
     (path "/67c490cc-fc2c-4fab-9127-c49a9a5a1dc6"
       (reference "C2") (unit 1) (value "0.1uF") (footprint "Capacitor_SMD:C_0402_1005Metric")
     )
     (path "/cfd5ba1c-1821-4334-910d-17809a83c077"
-      (reference "C3") (unit 1) (value "10uF") (footprint "Capacitor_SMD:C_0805_2012Metric_Pad1.18x1.45mm_HandSolder")
+      (reference "C3") (unit 1) (value "10uF") (footprint "Capacitor_SMD:C_0805_2012Metric")
     )
     (path "/1f16eb18-06a3-4445-83cc-1586203ce83e"
@@
     )
     (path "/3b27e57e-fe07-46ab-86e1-64b9b39500eb"
-      (reference "C6") (unit 1) (value "10uF") (footprint "Capacitor_SMD:C_0805_2012Metric_Pad1.18x1.45mm_HandSolder")
+      (reference "C6") (unit 1) (value "10uF") (footprint "Capacitor_SMD:C_0805_2012Metric")
     )
     (path "/c148735d-6e17-473a-a353-7c706f3310f6"
@@
       (reference "C9") (unit 1) (value "22pF") (footprint "Capacitor_SMD:C_0603_1608Metric")
     )
+    (path "/f85c989d-562e-47b3-83cb-ab114c33cb01"
+      (reference "C10") (unit 1) (value "1uF") (footprint "Capacitor_SMD:C_0402_1005Metric")
+    )
     (path "/fb026700-6304-4c85-b7fa-1f1e7a63a43a"
       (reference "C11") (unit 1) (value "1uF") (footprint "Capacitor_SMD:C_0402_1005Metric")
@@
       (reference "C18") (unit 1) (value "0.1uF") (footprint "Capacitor_SMD:C_0402_1005Metric")
     )
-    (path "/b6840320-619e-43d4-96f6-547c766d63b2"
-      (reference "C?") (unit 1) (value "1uF") (footprint "Capacitor_SMD:C_0402_1005Metric")
-    )
-    (path "/f85c989d-562e-47b3-83cb-ab114c33cb01"
-      (reference "C?") (unit 1) (value "1uF") (footprint "Capacitor_SMD:C_0402_1005Metric")
-    )
     (path "/3ed5ee36-eed7-4c90-9b4e-319b8feaa820"
-      (reference "D1") (unit 1) (value "SBR1A40SA") (footprint "Diode_SMD:D_SMA_Handsoldering")
+      (reference "D1") (unit 1) (value "1N5819WS") (footprint "Diode_SMD:D_SOD-323_HandSoldering")
     )
     (path "/0f81055f-6090-415e-91f0-ad4b905afc67"
@@
       (reference "D6") (unit 1) (value "Yellow") (footprint "LED_SMD:LED_0603_1608Metric_Pad1.05x0.95mm_HandSolder")
     )
-    (path "/eae35d4e-62ff-4876-bc6a-d913690e54d3"
-      (reference "D7") (unit 1) (value "SBR1A40SA") (footprint "Diode_SMD:D_SMA_Handsoldering")
+    (path "/fab4256d-8d63-4f41-8c03-103850ad50eb"
+      (reference "D7") (unit 1) (value "SS2040FL") (footprint "Diode_SMD:D_SOD-123")
     )
     (path "/40afe149-baf4-4592-b353-ea703d34a68d"
@@
     )
     (path "/85e596eb-2d05-4aa4-9d56-5790c6f6caf0"
-      (reference "D11") (unit 1) (value "SBR1A40SA") (footprint "Diode_SMD:D_SMA_Handsoldering")
+      (reference "D11") (unit 1) (value "1N5819WS") (footprint "Diode_SMD:D_SOD-323_HandSoldering")
     )
     (path "/82236554-b4fd-4c66-afd6-3216e7099810"
@@
       (reference "J2") (unit 1) (value "Conn_01x02_Female") (footprint "Connector_AMASS:AMASS_XT30PW-F_1x02_P2.50mm_Horizontal")
     )
+    (path "/f165734e-04b8-4bb6-a673-21efc01c3361"
+      (reference "J3") (unit 1) (value "Conn_01x10_Male") (footprint "BoxHeader_1.27mm:BoxHeader_2x05_P1.27mm_Vertical_SMD")
+    )
     (path "/1ac864ba-2dc7-41c2-b122-44cef9d40964"
       (reference "J4") (unit 1) (value "Conn_01x04_Male") (footprint "Connector_Molex:Molex_SPOX_5268-04A_1x04_P2.50mm_Horizontal")
@@
       (reference "J5") (unit 1) (value "Conn_01x04_Male") (footprint "Connector_Molex:Molex_SPOX_5268-04A_1x04_P2.50mm_Horizontal")
     )
-    (path "/f165734e-04b8-4bb6-a673-21efc01c3361"
-      (reference "J?") (unit 1) (value "Conn_01x10_Male") (footprint "BoxHeader_1.27mm:BoxHeader_2x05_P1.27mm_Vertical_SMD")
-    )
     (path "/b32e5410-6977-4f5d-844f-cbb8e8ef66fe"
