File: Encoder/Encoder.kicad_sch (KiCad schematic)
At the start: 90 parts, among them J1 Conn_01x02_Male, J2 Conn_01x04_Male, J3 Conn_01x04_Male, Q1 SSM3J332R, Q10 SSM3J332R, Q11 Q_PNP_BEC, Q12 Q_PNP_BEC, Q2 Q_NMOS_GSD, Q3 SSM3J332R, Q4 SSM3J332R, Q5 Q_PNP_BEC, Q6 SSM3J332R, Q7 Q_PNP_BEC, Q8 SSM3J332R, Q9 Q_PNP_BEC, SW1 SW_DIP_x05, SW2 SW_SPDT, SW3 SW_SPST, U1 AZ1084CD-3.3, U2 MAX3485, Y1 48MHz

Commit message: 回路設計
Parts:
- removed C10, C11: 4.7uF, Capacitor_SMD:C_0603_1608Metric, symbol Device:C
- removed C13, C14: 470uF, Capacitor_SMD:C_Elec_8x10.2, symbol Device:C_Polarized
- removed C2, C8: 0.1uF, Capacitor_SMD:C_0402_1005Metric, symbol Device:C
- removed C9: ADJ_ST, Capacitor_THT:C_Disc_D5.0mm_W2.5mm_P5.00mm, symbol Device:C
- removed D2, D3: D, Diode_SMD:D_SOD-123, symbol Device:D
- removed D4: D_Zener, Diode_SMD:D_SOD-323_HandSoldering, symbol Device:D_Zener
- removed D6, D7: Green, LED_SMD:LED_0603_1608Metric_Pad1.05x0.95mm_HandSolder, symbol Device:LED
- removed H1, H6, H7: MountingHole_Pad, TestPoint:TestPoint_Keystone_5019_Minature, symbol Mechanical:MountingHole_Pad
- removed H10, H9: MountingHole_Pad, TestPoint:TestPoint_Pad_1.5x1.5mm, symbol Mechanical:MountingHole_Pad
- removed Q10, Q4, Q6, Q8: SSM3J332R, Package_TO_SOT_SMD:SOT-23, symbol Device:Q_PMOS_GSD
- removed Q11, Q5, Q7, Q9: Q_PNP_BEC, Package_TO_SOT_SMD:SC-59_Handsoldering, symbol Device:Q_PNP_BEC
- removed R12, R14, R16, R17, R19, R20, R21, R22, R23: 10k, Resistor_SMD:R_0402_1005Metric, symbol Device:R
- removed R15, R25, R26: 1k, Resistor_SMD:R_0402_1005Metric, symbol Device:R
- removed R18: 100k, Resistor_SMD:R_0402_1005Metric, symbol Device:R
- added C? (x2): 10uF, Capacitor_SMD:C_0805_2012Metric_Pad1.18x1.45mm_HandSolder, symbol Device:C
- added C?: 0.1uF, Capacitor_SMD:C_0402_1005Metric, symbol Device:C
- added D? (x2): SBR1A40SA, Diode_SMD:D_SMA_Handsoldering, symbol Device:D_Schottky
- added R? (x2): 3.9k, Resistor_SMD:R_0603_1608Metric, symbol Device:R
- added U?: STM32C011F4P6, Package_SO:TSSOP-20_4.4x6.5mm_P0.65mm, symbol STM32C011F4P6:STM32C011F4P6
- added U?: AS5600, Package_SO:SOP-8_3.9x4.9mm_P1.27mm, symbol AS5600:AS5600
- C5, C6: footprint (none) -> Capacitor_SMD:C_0603_1608Metric
- Q1, Q3: footprint Package_TO_SOT_SMD:SOT-23 -> Package_TO_SOT_SMD:SOT-23W
- Q12: value Q_PNP_BEC -> 2PB709AR
- Q2: value Q_NMOS_GSD -> BSS138
- R11: value 1k -> 10k
- SW1: footprint Package_DIP:DIP-10_W7.62mm -> Package_DIP:SMDIP-10_W7.62mm
- SW2: value SW_SPDT -> SW_SPDT_White
Connections:
- net 3.3VSYS is gone; now on net +3.3V: C4.1, R13.2, U1.2 (VO)
- net +3.3V: now also C?.1, C?.1, D?.2 (A), R?.1, R?.1, U?.1 (VDD5V), U?.2 (VDD3V3), U?.4 (VDD/VDDA)
- net GND: now also C?.2, C?.2, C?.2, D?.2 (A), U?.4 (GND), U?.5 (VSS/VSSA), U?.8 (DIR)
- net VDD: now also C?.1, D?.1 (K), D?.1 (K)
- net OSC_IN: now reaches C5.2, Y1.2
- net OSC_IN: no longer C6.2, Y1.1
- new net I2C_SCL: R?.2, U?.7 (SCL)
- new net I2C_SDA: R?.2, U?.6 (SDA)
- new net OSC_OUT: C6.2, Y1.1
Other:
- note added: "5Pスイッチ"
- note added: "C011F4"
- note removed: "4Pスイッチ"
- note removed: "F446RE"
- note removed: "理想ダイオード/3.3VSYS"
- note removed: "電源切替/STLink"
- moved on the sheet: C12, C3, C4, C5, C6, C7, D1, D5, D8, H2, H4, H5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

Commit message: 回路設計
Parts:
- removed H2, H3, H4, H5: MountingHole_Pad, TestPoint:TestPoint_Keystone_5019_Minature, symbol Mechanical:MountingHole_Pad
- added J?: Conn_01x04_Female, Connector_PinHeader_2.54mm:PinHeader_1x04_P2.54mm_Vertical, symbol Connector:Conn_01x04_Female
Connections:
- net GND: now also J?.2 (Pin_2)
- net NRST: now also J?.4 (Pin_4)
- net TCK: now also J?.1 (Pin_1)
- net TMS: now also J?.3 (Pin_3)
Changed lines of the file:
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@@
     (stroke (width 0) (type default) (color 0 0 0 0))
   )
-  (wire (pts (xy 88.9 238.76) (xy 91.44 238.76))
+  (wire (pts (xy 81.28 236.22) (xy 83.82 236.22))
     (stroke (width 0) (type default) (color 0 0 0 0))
   )
@@
     (stroke (width 0) (type default) (color 0 0 0 0))
   )
-  (wire (pts (xy 88.9 243.84) (xy 91.44 243.84))
+  (wire (pts (xy 81.28 238.76) (xy 83.82 238.76))
     (stroke (width 0) (type default) (color 0 0 0 0))
   )
@@
     (stroke (width 0) (type default) (color 0 0 0 0))
   )
-  (wire (pts (xy 88.9 233.68) (xy 91.44 233.68))
+  (wire (pts (xy 81.28 233.68) (xy 93.98 233.68))
     (stroke (width 0) (type default) (color 0 0 0 0))
   )
@@
     (stroke (width 0) (type default) (color 0 0 0 0))
   )
-  (wire (pts (xy 88.9 228.6) (xy 91.44 228.6))
+  (wire (pts (xy 81.28 231.14) (xy 83.82 231.14))
     (stroke (width 0) (type default) (color 0 0 0 0))
   )
@@
     )
   )
-  (global_label "NRST" (shape output) (at 91.44 243.84 0) (fields_autoplaced)
-    (effects (font (size 1.27 1.27)) (justify left))
-    (property "Intersheet References" "${INTERSHEET_REFS}" (id 0) (at 50.8 66.04 0)
+  (global_label "NRST" (shape output) (at 83.82 238.76 0) (fields_autoplaced)
+    (effects (font (size 1.27 1.27)) (justify left))
+    (property "Intersheet References" "${INTERSHEET_REFS}" (id 0) (at 43.18 60.96 0)
       (effects (font (size 1.27 1.27)) hide)
     )
@@
     )
   )
-  (global_label "TCK" (shape bidirectional) (at 91.44 228.6 0) (fields_autoplaced)
-    (effects (font (size 1.27 1.27)) (justify left))
-    (property "Intersheet References" "${INTERSHEET_REFS}" (id 0) (at 50.8 58.42 0)
+  (global_label "TCK" (shape bidirectional) (at 83.82 231.14 0) (fields_autoplaced)
+    (effects (font (size 1.27 1.27)) (justify left))
+    (property "Intersheet References" "${INTERSHEET_REFS}" (id 0) (at 43.18 60.96 0)
       (effects (font (size 1.27 1.27)) hide)
     )
@@
     )
   )
-  (global_label "TMS" (shape bidirectional) (at 91.44 238.76 0) (fields_autoplaced)
-    (effects (font (size 1.27 1.27)) (justify left))
-    (property "Intersheet References" "${INTERSHEET_REFS}" (id 0) (at 50.8 63.5 0)
+  (global_label "TMS" (shape bidirectional) (at 83.82 236.22 0) (fields_autoplaced)
+    (effects (font (size 1.27 1.27)) (justify left))
+    (property "Intersheet References" "${INTERSHEET_REFS}" (id 0) (at 43.18 60.96 0)
       (effects (font (size 1.27 1.27)) hide)
     )
@@
     (pin "1")
     (pin "2")
-  )
-  (symbol (lib_id "Mechanical:MountingHole_Pad") (at 86.36 243.84 90) (mirror x) (unit 1)
-    (in_bom yes) (on_board yes)
-    (property "Reference" "H5" (id 0) (at 78.74 241.3 90)
-      (effects (font (size 1.27 1.27)) (justify right))
-    )
-    (property "Value" "MountingHole_Pad" (id 1) (at 63.5 243.84 90)
-      (effects (font (size 1.27 1.27)) (justify right))
-    )
-    (property "Footprint" "TestPoint:TestPoint_Keystone_5019_Minature" (id 2) (at 86.36 243.84 0)
-      (effects (font (size 1.27 1.27)) hide)
-    )
-    (property "Datasheet" "~" (id 3) (at 86.36 243.84 0)
-      (effects (font (size 1.27 1.27)) hide)
-    )
-    (pin "1")
   )
   (symbol (lib_id "power:+3.3V") (at 60.96 320.04 0) (unit 1)
@@
     (pin "1")
   )
-  (symbol (lib_id "Mechanical:MountingHole_Pad") (at 86.36 228.6 90) (mirror x) (unit 1)
-    (in_bom yes) (on_board yes)
-    (property "Reference" "H2" (id 0) (at 78.74 226.06 90)
-      (effects (font (size 1.27 1.27)) (justify right))
-    )
-    (property "Value" "MountingHole_Pad" (id 1) (at 63.5 228.6 90)
-      (effects (font (size 1.27 1.27)) (justify right))
-    )
-    (property "Footprint" "TestPoint:TestPoint_Keystone_5019_Minature" (id 2) (at 86.36 228.6 0)
-      (effects (font (size 1.27 1.27)) hide)
-    )
-    (property "Datasheet" "~" (id 3) (at 86.36 228.6 0)
-      (effects (font (size 1.27 1.27)) hide)
-    )
-    (pin "1")
-  )
   (symbol (lib_id "power:GND") (at 60.96 144.78 0) (unit 1)
     (in_bom yes) (on_board yes) (fields_autoplaced)
@@
     (pin "1")
     (pin "2")
-  )
-  (symbol (lib_id "Mechanical:MountingHole_Pad") (at 86.36 233.68 90) (mirror x) (unit 1)
-    (in_bom yes) (on_board yes)
-    (property "Reference" "H3" (id 0) (at 78.74 231.14 90)
-      (effects (font (size 1.27 1.27)) (justify right))
-    )
-    (property "Value" "MountingHole_Pad" (id 1) (at 63.5 233.68 90)
-      (effects (font (size 1.27 1.27)) (justify right))
-    )
-    (property "Footprint" "TestPoint:TestPoint_Keystone_5019_Minature" (id 2) (at 86.36 233.68 0)
-      (effects (font (size 1.27 1.27)) hide)
-    )
-    (property "Datasheet" "~" (id 3) (at 86.36 233.68 0)
-      (effects (font (size 1.27 1.27)) hide)
-    )
-    (pin "1")
   )
   (symbol (lib_id "Connector:TestPoint") (at 152.4 152.4 180) (unit 1)
@@
     (pin "2")
   )
-  (symbol (lib_id "power:GND") (at 91.44 233.68 0) (unit 1)
-    (in_bom yes) (on_board yes)
-    (property "Reference" "#PWR0109" (id 0) (at 91.44 240.03 0)
-      (effects (font (size 1.27 1.27)) hide)
-    )
-    (property "Value" "GND" (id 1) (at 93.98 236.22 0))
-    (property "Footprint" "" (id 2) (at 91.44 233.68 0)
-      (effects (font (size 1.27 1.27)) hide)
-    )
-    (property "Datasheet" "" (id 3) (at 91.44 233.68 0)
+  (symbol (lib_id "power:GND") (at 93.98 233.68 0) (unit 1)
+    (in_bom yes) (on_board yes)
+    (property "Reference" "#PWR0109" (id 0) (at 93.98 240.03 0)
+      (effects (font (size 1.27 1.27)) hide)
+    )
+    (property "Value" "GND" (id 1) (at 96.52 236.22 0))
+    (property "Footprint" "" (id 2) (at 93.98 233.68 0)
+      (effects (font (size 1.27 1.27)) hide)
+    )
+    (property "Datasheet" "" (id 3) (at 93.98 233.68 0)
       (effects (font (size 1.27 1.27)) hide)
     )
@@
     (pin "1")
   )
-  (symbol (lib_id "Mechanical:MountingHole_Pad") (at 86.36 238.76 90) (mirror x) (unit 1)
-    (in_bom yes) (on_board yes)
-    (property "Reference" "H4" (id 0) (at 78.74 236.22 90)
-      (effects (font (size 1.27 1.27)) (justify right))
-    )
-    (property "Value" "MountingHole_Pad" (id 1) (at 63.5 238.76 90)
-      (effects (font (size 1.27 1.27)) (justify right))
-    )
-    (property "Footprint" "TestPoint:TestPoint_Keystone_5019_Minature" (id 2) (at 86.36 238.76 0)
-      (effects (font (size 1.27 1.27)) hide)
-    )
-    (property "Datasheet" "~" (id 3) (at 86.36 238.76 0)
-      (effects (font (size 1.27 1.27)) hide)
-    )
-    (pin "1")
-  )
   (symbol (lib_id "power:VDD") (at 152.4 149.86 0) (unit 1)
     (in_bom yes) (on_board yes) (fields_autoplaced)
@@
     )
     (pin "1")
+  )
+  (symbol (lib_id "Connector:Conn_01x04_Female") (at 76.2 233.68 0) (mirror y) (unit 1)
+    (in_bom yes) (on_board yes) (fields_autoplaced)
+    (property "Reference" "J?" (id 0) (at 76.835 226.06 0))
+    (property "Value" "Conn_01x04_Female" (id 1) (at 76.835 228.6 0))
+    (property "Footprint" "Connector_PinHeader_2.54mm:PinHeader_1x04_P2.54mm_Vertical" (id 2) (at 76.2 233.68 0)
+      (effects (font (size 1.27 1.27)) hide)
+    )
+    (property "Datasheet" "~" (id 3) (at 76.2 233.68 0)
+      (effects (font (size 1.27 1.27)) hide)
+    )
+    (pin "1")
+    (pin "2")
+    (pin "3")
+    (pin "4")
   )
   (symbol (lib_id "Connector:TestPoint") (at 172.72 152.4 180) (unit 1)
@@
       (reference "D?") (unit 1) (value "SBR1A40SA") (footprint "Diode_SMD:D_SMA_Handsoldering")
     )
-    (path "/51b101dc-3fd8-439d-ba1a-45dee2ee1e7b"
-      (reference "H2") (unit 1) (value "MountingHole_Pad") (footprint "TestPoint:TestPoint_Keystone_5019_Minature")
-    )
-    (path "/5c96fa03-528c-4014-a8f5-77eb363f51fb"
-      (reference "H3") (unit 1) (value "MountingHole_Pad") (footprint "TestPoint:TestPoint_Keystone_5019_Minature")
-    )
-    (path "/d87199d4-5a00-485e-b489-b46c49d12f4d"
-      (reference "H4") (unit 1) (value "MountingHole_Pad") (footprint "TestPoint:TestPoint_Keystone_5019_Minature")
-    )
-    (path "/0a0b4be0-d712-4820-ad45-b5f3164cf350"
-      (reference "H5") (unit 1) (value "MountingHole_Pad") (footprint "TestPoint:TestPoint_Keystone_5019_Minature")
-    )
     (path "/748f3f23-7352-40c9-8bc7-ffe8531b9c38"
       (reference "H8") (unit 1) (value "MountingHole_Pad") (footprint "TestPoint:TestPoint_Pad_1.5x1.5mm")
@@
       (reference "J3") (unit 1) (value "Conn_01x04_Male") (footprint "Connector_Molex:Molex_SPOX_5268-04A_1x04_P2.50mm_Horizontal")
     )
+    (path "/e00540e1-46e4-4278-8f7c-20405075d788"
+      (reference "J?") (unit 1) (value "Conn_01x04_Female") (footprint "Connector_PinHeader_2.54mm:PinHeader_1x04_P2.54mm_Vertical")
+    )
     (path "/837550e3-e9e9-40db-91e8-a23399732e65"

Commit message: 構成図追加
Parts:
- Q12: value 2PB709AR -> S8050; footprint Package_TO_SOT_SMD:SC-59_Handsoldering -> Package_TO_SOT_SMD:SOT-23
- SW2: footprint (none) -> Slide_Switch:SW_Slide_SPDT_White
- Y1: footprint (none) -> Crystal:Crystal_SMD_HC49-SD_HandSoldering
- gave numbers to parts that had none: 10
Connections:
- no-connect marks 15 -> 3
Other:
- moved on the sheet: C1, C12, C15, C2, C3, C4, C5, C6, C7, C8, C9, D1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

Commit message: diagram_SmallPW
Parts:
- removed C1: 4.7uF, Capacitor_SMD:C_0603_1608Metric, symbol Device:C
- added C?: 1uF, Capacitor_SMD:C_0402_1005Metric, symbol Device:C
Connections:
- net S-S: now also C?.1
- net at Q3.1 (G), R7.2, R9.1: now also C?.2
Changed lines of the file:
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@@
     (pin "9")
+  )
+  (symbol (lib_id "Device:C") (at 66.04 109.22 0) (unit 1)
+    (in_bom yes) (on_board yes) (fields_autoplaced)
+    (property "Reference" "C?" (id 0) (at 69.85 107.9499 0)
+      (effects (font (size 1.27 1.27)) (justify left))
+    )
+    (property "Value" "1uF" (id 1) (at 69.85 110.4899 0)
+      (effects (font (size 1.27 1.27)) (justify left))
+    )
+    (property "Footprint" "Capacitor_SMD:C_0402_1005Metric" (id 2) (at 67.0052 113.03 0)
+      (effects (font (size 1.27 1.27)) hide)
+    )
+    (property "Datasheet" "~" (id 3) (at 66.04 109.22 0)
+      (effects (font (size 1.27 1.27)) hide)
+    )
+    (pin "1")
+    (pin "2")
   )
   (symbol (lib_id "Switch:SW_SPST") (at 223.52 124.46 0) (unit 1)
@@
     (pin "2")
   )
-  (symbol (lib_id "Device:C") (at 66.04 109.22 0) (unit 1)
-    (in_bom yes) (on_board yes) (fields_autoplaced)
-    (property "Reference" "C1" (id 0) (at 69.85 107.9499 0)
-      (effects (font (size 1.27 1.27)) (justify left))
-    )
-    (property "Value" "4.7uF" (id 1) (at 69.85 110.4899 0)
-      (effects (font (size 1.27 1.27)) (justify left))
-    )
-    (property "Footprint" "Capacitor_SMD:C_0603_1608Metric" (id 2) (at 67.0052 113.03 0)
-      (effects (font (size 1.27 1.27)) hide)
-    )
-    (property "Datasheet" "~" (id 3) (at 66.04 109.22 0)
-      (effects (font (size 1.27 1.27)) hide)
-    )
-    (pin "1")
-    (pin "2")
-  )
   (symbol (lib_id "power:VDD") (at 121.92 45.72 0) (unit 1)
     (in_bom yes) (on_board yes) (fields_autoplaced)
@@
       (reference "#PWR0140") (unit 1) (value "GND") (footprint "")
     )
-    (path "/bfba173c-3ca4-479c-aa1b-4c022ac8f368"
-      (reference "C1") (unit 1) (value "4.7uF") (footprint "Capacitor_SMD:C_0603_1608Metric")
-    )
     (path "/bd314a8a-0117-486e-9eed-42afc9c18d15"
       (reference "C2") (unit 1) (value "0.1uF") (footprint "Capacitor_SMD:C_0402_1005Metric")
@@
       (reference "C15") (unit 1) (value "0.1uF") (footprint "Capacitor_SMD:C_0402_1005Metric")
     )
+    (path "/0e6a2fe5-ba1d-49cf-a83c-0f84c7463e92"
+      (reference "C?") (unit 1) (value "1uF") (footprint "Capacitor_SMD:C_0402_1005Metric")
+    )
     (path "/89289daf-7d4f-42a1-81cb-0c98167c5d41"

Commit message: 回路図pdf出力
Parts:
- D2, D3: footprint Diode_SMD:D_SMA_Handsoldering -> Diode_SMD:D_SMA
- JP1: footprint Connector_PinHeader_2.54mm:PinHeader_1x02_P2.54mm_Vertical -> Jumper:SolderJumper-2_P1.3mm_Open_TrianglePad1.0x1.5mm
- Y1: footprint Crystal:Crystal_SMD_HC49-SD_HandSoldering -> Crystal:Crystal_SMD_HC49-SD
- gave numbers to parts that had none: 1

Commit message: 定期更新
Connections:
- net NRST: now also U4.6 (PF2-NRST)
- net OSC_IN: now also U4.2 (PC14-OSCX_IN)
- net OSC_OUT: now also U4.3 (PC15-OSCX_OUT)

Commit message: 進捗
Parts:
- added H1, H2: MountingHole_Pad, TestPoint:TestPoint_Pad_1.5x1.5mm, symbol Mechanical:MountingHole_Pad
- C8, C9: footprint Capacitor_SMD:C_0805_2012Metric_Pad1.18x1.45mm_HandSolder -> Capacitor_SMD:C_0805_2012Metric
- D2, D3: value SBR1A40SA -> 1N5819WS; footprint Diode_SMD:D_SMA -> Diode_SMD:D_SOD-323_HandSoldering
Other:
- note added: "UART引き出す"
