File: IR/IR.kicad_sch (KiCad schematic)
At the start: 191 parts, among them J1 Conn_01x02_Male, J2 Conn_01x10_Male, J3 Conn_01x04_Male, J4 Conn_01x04_Male, Q1 SSM3J332R, Q12 S8050, Q13 SSM3K345R, Q14 SSM3K345R, Q15 SSM3K345R, Q16 SSM3K345R, Q2 BSS138, Q3 SSM3J332R, SW1 SW_DIP_x05, SW2 SW_SPDT, SW3 SW_SPDT_White, SW4 SW_SPST, U1 TSSP58038, U10 TSSP58038, U11 TSSP58038, U12 TSSP58038, U13 TSSP58038, U14 TSSP58038, U15 TSSP58038, U16 TSSP58038, U17 TSSP58038, U18 74HC4051, U19 74HC4051, U2 TSSP58038, U20 STM32G030K6T6, U21 MAX3485, U22 NJU6319AE, U3 TSSP58038, U4 TSSP58038, U5 AZ1084CD-3.3, U6 TSSP58038, U7 TSSP58038, U8 TSSP58038, U9 TSSP58038, Y1 16MHz

Commit message: LargeMDほぼ完成
Connections:
- net at U22.6 (NC): no longer U22.7 (NC)
- net MainRX_RS485TX renamed MainRX2_RS485TX
- net MainRX_STLinkTX renamed MainRX1_STLinkTX
- net MainTX_RS485RX renamed MainTX2_RS485RX
- net MainTX_STLinkRX renamed MainTX1_STLinkRX
- no-connect marks 8 -> 9
Changed lines of the file:
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@@
   (no_connect (at 381 299.72))
   (no_connect (at 165.1 261.62))
+  (no_connect (at 381 327.66))
   (no_connect (at 129.54 309.88))
   (wire (pts (xy 154.94 137.16) (xy 160.02 137.16))
@@
     )
   )
-  (global_label "MainTX_RS485RX" (shape bidirectional) (at 449.58 142.24 180) (fields_autoplaced)
+  (global_label "MainTX2_RS485RX" (shape bidirectional) (at 449.58 142.24 180) (fields_autoplaced)
     (effects (font (size 1.27 1.27)) (justify right))
-    (property "Intersheet References" "${INTERSHEET_REFS}" (id 0) (at 431.0802 142.1606 0)
+    (property "Intersheet References" "${INTERSHEET_REFS}" (id 0) (at 429.8707 142.1606 0)
       (effects (font (size 1.27 1.27)) (justify right) hide)
     )
@@
     )
   )
-  (global_label "MainRX_RS485TX" (shape bidirectional) (at 449.58 134.62 180) (fields_autoplaced)
+  (global_label "MainRX2_RS485TX" (shape bidirectional) (at 449.58 134.62 180) (fields_autoplaced)
     (effects (font (size 1.27 1.27)) (justify right))
-    (property "Intersheet References" "${INTERSHEET_REFS}" (id 0) (at 431.0802 134.5406 0)
+    (property "Intersheet References" "${INTERSHEET_REFS}" (id 0) (at 429.8707 134.5406 0)
       (effects (font (size 1.27 1.27)) (justify right) hide)
     )
   )
-  (global_label "MainRX_STLinkTX" (shape bidirectional) (at 378.46 304.8 180) (fields_autoplaced)
+  (global_label "MainRX1_STLinkTX" (shape bidirectional) (at 378.46 304.8 180) (fields_autoplaced)
     (effects (font (size 1.27 1.27)) (justify right))
-    (property "Intersheet References" "${INTERSHEET_REFS}" (id 0) (at 360.0812 304.7206 0)
+    (property "Intersheet References" "${INTERSHEET_REFS}" (id 0) (at 358.8717 304.7206 0)
       (effects (font (size 1.27 1.27)) (justify right) hide)
     )
@@
     )
   )
-  (global_label "MainTX_STLinkRX" (shape bidirectional) (at 378.46 302.26 180) (fields_autoplaced)
+  (global_label "MainTX1_STLinkRX" (shape bidirectional) (at 378.46 302.26 180) (fields_autoplaced)
     (effects (font (size 1.27 1.27)) (justify right))
-    (property "Intersheet References" "${INTERSHEET_REFS}" (id 0) (at 360.0812 302.1806 0)
+    (property "Intersheet References" "${INTERSHEET_REFS}" (id 0) (at 358.8717 302.1806 0)
       (effects (font (size 1.27 1.27)) (justify right) hide)
     )
@@
     )
   )
-  (global_label "MainRX_STLinkTX" (shape bidirectional) (at 167.64 256.54 0) (fields_autoplaced)
+  (global_label "MainRX1_STLinkTX" (shape bidirectional) (at 167.64 256.54 0) (fields_autoplaced)
     (effects (font (size 1.27 1.27)) (justify left))
-    (property "Intersheet References" "${INTERSHEET_REFS}" (id 0) (at 186.0188 256.4606 0)
+    (property "Intersheet References" "${INTERSHEET_REFS}" (id 0) (at 187.2283 256.4606 0)
       (effects (font (size 1.27 1.27)) (justify left) hide)
     )
@@
     )
   )
-  (global_label "MainTX_RS485RX" (shape bidirectional) (at 378.46 284.48 180) (fields_autoplaced)
+  (global_label "MainTX2_RS485RX" (shape bidirectional) (at 378.46 284.48 180) (fields_autoplaced)
     (effects (font (size 1.27 1.27)) (justify right))
-    (property "Intersheet References" "${INTERSHEET_REFS}" (id 0) (at 359.9602 284.4006 0)
+    (property "Intersheet References" "${INTERSHEET_REFS}" (id 0) (at 358.7507 284.4006 0)
       (effects (font (size 1.27 1.27)) (justify right) hide)
     )
@@
     )
   )
-  (global_label "MainTX_STLinkRX" (shape bidirectional) (at 167.64 259.08 0) (fields_autoplaced)
+  (global_label "MainTX1_STLinkRX" (shape bidirectional) (at 167.64 259.08 0) (fields_autoplaced)
     (effects (font (size 1.27 1.27)) (justify left))
-    (property "Intersheet References" "${INTERSHEET_REFS}" (id 0) (at 186.0188 259.0006 0)
+    (property "Intersheet References" "${INTERSHEET_REFS}" (id 0) (at 187.2283 259.0006 0)
       (effects (font (size 1.27 1.27)) (justify left) hide)
     )
@@
     )
   )
-  (global_label "MainRX_RS485TX" (shape bidirectional) (at 378.46 317.5 180) (fields_autoplaced)
+  (global_label "MainRX2_RS485TX" (shape bidirectional) (at 378.46 317.5 180) (fields_autoplaced)
     (effects (font (size 1.27 1.27)) (justify right))
-    (property "Intersheet References" "${INTERSHEET_REFS}" (id 0) (at 359.9602 317.4206 0)
+    (property "Intersheet References" "${INTERSHEET_REFS}" (id 0) (at 358.7507 317.4206 0)
       (effects (font (size 1.27 1.27)) (justify right) hide)
     )
