File: LargeMD/LargeMD.kicad_sch (KiCad schematic)
At the start: 238 parts

Commit message: 回路設計
Parts:
- removed C? (x9): 0.1uF, Capacitor_SMD:C_0402_1005Metric, symbol Device:C
- removed C? (x7): 470uF, Capacitor_SMD:C_Elec_8x10.2, symbol Device:C_Polarized
- removed C? (x5): 1uF, Capacitor_SMD:C_0402_1005Metric, symbol Device:C
- removed C?: 4.7uF, Capacitor_SMD:C_0603_1608Metric, symbol Device:C
- removed C? (x2): C, Capacitor_SMD:C_1210_3225Metric_Pad1.33x2.70mm_HandSolder, symbol Device:C
- removed C? (x3): 4.7uF, Capacitor_SMD:C_0805_2012Metric_Pad1.18x1.45mm_HandSolder, symbol Device:C
- removed C?: 10uF, Capacitor_SMD:C_0805_2012Metric_Pad1.18x1.45mm_HandSolder, symbol Device:C
- removed D? (x6): D_Schottky, Diode_SMD:D_SOD-123, symbol Device:D_Schottky
- removed D?: D_Schottky, Diode_Schottky:DO-221BC, symbol Device:D_Schottky
- removed D? (x6): LED, LED_SMD:LED_0603_1608Metric_Pad1.05x0.95mm_HandSolder, symbol Device:LED
- removed D? (x6): D, Diode_SMD:D_SOD-123, symbol Device:D
- removed J? (x2): Conn_01x05_Female, Connector_Molex:Molex_SPOX_5268-05A_1x05_P2.50mm_Horizontal, symbol Connector:Conn_01x05_Female
- removed J? (x2): Conn_01x02_Female, Connector_AMASS:AMASS_XT30PW-M_1x02_P2.50mm_Horizontal, symbol Connector:Conn_01x02_Female
- removed JP?: Jumper_2_Open, Connector_PinHeader_2.54mm:PinHeader_1x02_P2.54mm_Vertical, symbol Jumper:Jumper_2_Open
- removed Q? (x4): FDMS8050, SOP-Advance-8:SOP-Advance, symbol Transistor_FET:FDMS8050
- removed Q?: Q_PNP_BEC, Package_TO_SOT_SMD:SC-59_Handsoldering, symbol Device:Q_PNP_BEC
- removed Q? (x3): Q_NMOS_GSD, Package_TO_SOT_SMD:SOT-23_Handsoldering, symbol Device:Q_NMOS_GSD
- removed R? (x9): R, Resistor_SMD:R_0603_1608Metric_Pad0.98x0.95mm_HandSolder, symbol Device:R
- removed R? (x2): 2.2k, Resistor_SMD:R_0603_1608Metric_Pad0.98x0.95mm_HandSolder, symbol Device:R
- removed R? (x7): 1k, Resistor_SMD:R_0402_1005Metric, symbol Device:R
- removed R? (x22): 10k, Resistor_SMD:R_0402_1005Metric, symbol Device:R
- removed R?: MPR, Resistor_THT:R_Axial_DIN0309_L9.0mm_D3.2mm_P12.70mm_Horizontal, symbol Device:R
- removed R? (x4): 510, Resistor_SMD:R_0603_1608Metric_Pad0.98x0.95mm_HandSolder, symbol Device:R
- removed R?: 20k, Resistor_SMD:R_0603_1608Metric_Pad0.98x0.95mm_HandSolder, symbol Device:R
- removed R?: 120, Resistor_SMD:R_0603_1608Metric_Pad0.98x0.95mm_HandSolder, symbol Device:R
- removed R?: 7.5k, Resistor_SMD:R_0603_1608Metric_Pad0.98x0.95mm_HandSolder, symbol Device:R
- removed SW? (x2): SW_SPST, Button_Switch_SMD:SW_SPST_Omron_B3FS-100xP, symbol Switch:SW_SPST
- removed SW? (x3): SW_SPDT, Slide_Switch:3P_SPDT_SlideSwitch, symbol Switch:SW_SPDT
- removed SW?: SW_DIP_x04, Package_DIP:DIP-8_W7.62mm, symbol Switch:SW_DIP_x04
- removed TP? (x5): TestPoint, TestPoint:TestPoint_THTPad_D2.0mm_Drill1.0mm, symbol Connector:TestPoint
- removed U?: 74HC4051, symbol 74xx:74HC4051
- removed U? (x2): IR2302, Package_SO:SOP-8_3.9x4.9mm_P1.27mm, symbol Driver_FET:IR2302
- removed U?: STM32F303K8Tx, Package_QFP:LQFP-32_7x7mm_P0.8mm, symbol MCU_ST_STM32F3:STM32F303K8Tx
- removed U? (x2): TLP785, Package_DIP:DIP-4_W7.62mm, symbol Isolator:TLP785
- removed U?: LF50_TO220, DCDC_Regulator:BP5293, symbol Regulator_Linear:LF50_TO220
- removed U?: AMS1117CD-3.3, Package_TO_SOT_SMD:TO-252-3_TabPin2, symbol Regulator_Linear:AMS1117CD-3.3
- removed U?: MAX3485, Package_SO:SOP-8_3.9x4.9mm_P1.27mm, symbol Interface_UART:MAX3485
- added C? (x2): C, Capacitor_SMD:C_1210_3225Metric_Pad1.33x2.70mm_HandSolder, symbol Device:C
- added C? (x2): 4.7uF, Capacitor_SMD:C_0805_2012Metric_Pad1.18x1.45mm_HandSolder, symbol Device:C
- added C?: 1uF, Capacitor_SMD:C_0402_1005Metric, symbol Device:C
- added C? (x5): 0.1uF, Capacitor_SMD:C_0402_1005Metric, symbol Device:C
- added D? (x4): SS2040FL, Diode_SMD:D_SOD-123, symbol Device:D_Schottky
- added D? (x7): SBR1A40SA, Diode_SMD:D_SMA_Handsoldering, symbol Device:D_Schottky
- added D? (x4): Red, LED_SMD:LED_0603_1608Metric_Pad1.05x0.95mm_HandSolder, symbol Device:LED
- added J? (x2): Conn_01x04_Male, Connector_Molex:Molex_SPOX_5268-04A_1x04_P2.50mm_Horizontal, symbol Connector:Conn_01x04_Male
- added J?: Conn_01x03_Male, Connector_Molex:Molex_SPOX_5268-03A_1x03_P2.50mm_Horizontal, symbol Connector:Conn_01x03_Male
- added J?: Conn_01x02_Female, Connector_AMASS:AMASS_XT30PW-F_1x02_P2.50mm_Horizontal, symbol Connector:Conn_01x02_Female
- added JP?: Jumper_2_Open, Connector_PinHeader_2.54mm:PinHeader_1x02_P2.54mm_Vertical, symbol Jumper:Jumper_2_Open
- added JP? (x2): SolderJumper_3_Bridged12, symbol Jumper:SolderJumper_3_Bridged12
- added Q? (x4): TPH3R704PL, SOP-Advance-8:SOP-Advance, symbol Transistor_FET:FDMS8050
- added Q? (x2): BSS138, Package_TO_SOT_SMD:SOT-23_Handsoldering, symbol Device:Q_NMOS_GSD
- added Q?: 2PB709AR, Package_TO_SOT_SMD:SC-59_Handsoldering, symbol Device:Q_PNP_BEC
- added R? (x4): 47, Resistor_SMD:R_0603_1608Metric, symbol Device:R
- added R? (x7): 10k, Resistor_SMD:R_0402_1005Metric, symbol Device:R
- added R? (x4): 1k, Resistor_SMD:R_0402_1005Metric, symbol Device:R
- added R?: MPR, Resistor_THT:R_Axial_DIN0309_L9.0mm_D3.2mm_P12.70mm_Horizontal, symbol Device:R
- added R?: 120, Resistor_SMD:R_0402_1005Metric, symbol Device:R
- added R? (x4): 510, Resistor_SMD:R_0402_1005Metric, symbol Device:R
- added R?: 3.3k, Resistor_SMD:R_0603_1608Metric_Pad0.98x0.95mm_HandSolder, symbol Device:R
- added R? (x2): 2.2k, Resistor_SMD:R_0402_1005Metric, symbol Device:R
- added R?: 39, Resistor_SMD:R_0603_1608Metric_Pad0.98x0.95mm_HandSolder, symbol Device:R
- added R?: 7.5k, Resistor_SMD:R_0603_1608Metric, symbol Device:R
- added R?: 20k, Resistor_SMD:R_0402_1005Metric, symbol Device:R
- added R?: 10mR, symbol Device:R
- added U?: STM32C031K4T6, Package_QFP:LQFP-32_7x7mm_P0.8mm, symbol STM32C031K4T6:STM32C031K4T6
- added U?: LT6106, Package_TO_SOT_SMD:SOT-23-5, symbol Amplifier_Current:LT6106
- added U? (x2): IR2302, Package_SO:SOP-8_3.9x4.9mm_P1.27mm, symbol Driver_FET:IR2302
- added U? (x2): TLP785, Package_DIP:DIP-4_W7.62mm, symbol Isolator:TLP785
- added U?: MAX3485, Package_SO:SOP-8_3.9x4.9mm_P1.27mm, symbol Interface_UART:MAX3485
- C?: footprint Capacitor_THT:C_Disc_D5.0mm_W2.5mm_P5.00mm -> Capacitor_SMD:C_0603_1608Metric
- C? (x2): footprint (none) -> Capacitor_SMD:C_0603_1608Metric
- Q? (x2): value Q_PMOS_GDS -> TJ60S04M3L
- Q?: value Q_NMOS_GSD -> BSS138
- Q? (x7): value Q_PNP_BEC -> 2PB709AR
- Q? (x5): footprint Package_TO_SOT_SMD:SOT-23 -> Package_TO_SOT_SMD:SOT-23W
- R?: value V_Divider -> 33k; footprint Resistor_SMD:R_0603_1608Metric_Pad0.98x0.95mm_HandSolder -> Resistor_SMD:R_0603_1608Metric
- R?: value V_Divider -> 10k; footprint Resistor_SMD:R_0603_1608Metric_Pad0.98x0.95mm_HandSolder -> Resistor_SMD:R_0603_1608Metric
Connections:
- net IND_3.3V is gone; now on net 3.3V_IND: R?.2
- net +3.3V: now also C?.1, D?.1 (K), D?.1 (K), Q?.2 (E), R?.1, R?.1, R?.1, U?.4 (VDD/VDDA), U?.8 (VCC)
- net +5V: now also D?.1 (K), D?.2 (A), J?.2 (Pin_2), R?.2, R?.2
- net 3.3VBUS: now also J?.1 (Pin_1), C?.1
- net 3.3VSYS: now also R?.2, D?.2 (A); no longer R?.1
- net GND: now also C?.1, C?.2, C?.2, C?.2, C?.2, C?.2, C?.2, D?.1 (K), D?.1 (K), D?.2 (A), D?.2 (A), D?.2 (A), J?.1 (Pin_1), J?.1 (Pin_1), J?.1 (Pin_1), J?.2 (Pin_2), J?.2 (Pin_2), Q?.1 (S), Q?.1 (S), Q?.2 (S), Q?.2 (S), Q?.2 (S), Q?.2 (S), Q?.3 (S), Q?.3 (S), R?.1, R?.1, R?.1, R?.1, R?.2, R?.2, R?.2, U?.2, U?.2, U?.2 (V-), U?.3, U?.3, U?.4 (COM), U?.4 (COM), U?.5 (GND), U?.5 (VSS/VSSA)
- net LED1: now also R?.2
- net LED2: now also R?.2
- net Motor_A: now also C?.2, D?.1 (K), D?.2 (A), J?.1 (Pin_1), Q?.1 (S), Q?.2 (S), Q?.3 (S), Q?.5 (D), R?.1, R?.1, R?.2, U?.6 (VS)
- net Motor_B: now also C?.2, C?.2, D?.1 (K), D?.1 (K), D?.2 (A), D?.2 (A), J?.2 (Pin_2), Q?.1 (S), Q?.2 (S), Q?.3 (S), Q?.5 (D), R?.1, U?.6 (VS)
- net PWM_A: now also R?.1
- net PWM_B: now also R?.1
- net VCC: now also D?.1 (K)
- net VDD: now also C?.2, D?.1 (K), R?.2, R?.2, U?.5 (V+)
- net at C?.2, H?.1, Q?.1 (G): now also R?.1; no longer R?.2
- net 3.3V_IND: now reaches Q?.2 (E), Q?.3 (D), Q?.3 (D), R?.2
- net OSC_IN: now reaches C?.2, Y?.2
- net OSC_IN: no longer C?.2, Y?.1
- net MainRX2_STLinkTX renamed STLinkTX
- net STLinkTX: now also JP?.3 (B)
- net MainRX_RS485TX renamed MainRX_RS485aTX
- net MainTX2_STLinkRX renamed STLinkRX
- net STLinkRX: now also JP?.3 (B)
- net MainTX_RS485RX renamed MainTX_RS485aRX
- net RS485_A renamed RS485a_A
- net RS485_B renamed RS485a_B
- new net: Q?.4 (G), R?.2, R?.2 (x4)
- new net: R?.1, U?.5 (LO) (x2)
- new net: C?.1, D?.1 (K), U?.8 (VB) (x2)
- new net: D?.2 (A), R?.1 (x2)
- new net: Q?.1 (G), R?.2, R?.2 (x2)
- new net: Q?.3 (D), R?.2, U?.1 (x2)
- new net: R?.1, U?.7 (HO) (x2)
- new net: JP?.2 (B), R?.1
- new net: C?.1, R?.2
- new net: R?.1, U?.3 (-)
- new net: R?.1, U?.2 (IN), U?.4 (x2)
- new net: Q?.1 (B), R?.1
- new net: D?.1 (K), D?.2 (A), R?.1
- new net: Q?.3 (C), R?.1, U?.2 (~{RE}), U?.3 (DE)
- new net Current_Sence: D?.2 (A), R?.1, U?.1
- new net MainRX_RS485bTX: JP?.2 (C)
- new net MainTX_RS485bRX: JP?.2 (C)
- new net OSC_OUT: C?.2, Y?.1
- new net RS485bRX: JP?.1 (A), R?.2, U?.4 (DI)
- new net RS485bTX: JP?.1 (A), U?.1 (RO)
- new net RS485b_A: J?.3 (Pin_3), J?.3 (Pin_3), JP?.1 (A), R?.2, U?.6 (A)
- new net RS485b_B: J?.4 (Pin_4), J?.4 (Pin_4), R?.1, R?.2, U?.7 (B)
- new net SHDN: U?.3 (~{SD}), U?.3 (~{SD})
- new net Sensor0: D?.2 (A), J?.3 (Pin_3)
- new net Vdrive: C?.1, C?.1, C?.1, C?.1, D?.1 (K), D?.1 (K), D?.2 (A), D?.2 (A), Q?.5 (D), Q?.5 (D), R?.1, U?.1 (VCC), U?.1 (VCC), U?.4 (+)
- no-connect marks 28 -> 19
Other:
- note added: "5Pスイッチ"
- note added: "C031K4"
- note added: "Conn to sensor"
- note added: "CurrentSensor"
- note added: "Hブリッジ"
- note added: "Jumper"
- note added: "RS485a"
- note added: "RS485b"
- note added: "Snubber"
- note removed: "3.3V"
- note removed: "4Pスイッチ"
- note removed: "5V"
- note removed: "BOOT0"
- note removed: "Conn to Main"
- note removed: "Encoder"
- note removed: "F303K8"
- note removed: "F446RE"
- note removed: "Hブリッジ回路"
- note removed: "RS485"
- note removed: "タクトスイッチ"
- note removed: "モタドラ"
- moved on the sheet: C?, D?, H?, J?, JP?, Q?, R?, SW?, TP?, U?, Y?

Commit message: 構成図追加
Parts:
- removed J?: Conn_01x10_Female, Connector_IDC:IDC-Header_2x05_P2.54mm_Horizontal, symbol Connector:Conn_01x10_Female
- removed Q? (x2): BSS138, Package_TO_SOT_SMD:SOT-23_Handsoldering, symbol Device:Q_NMOS_GSD
- removed R? (x4): 510, Resistor_SMD:R_0402_1005Metric, symbol Device:R
- removed R? (x2): 1k, Resistor_SMD:R_0402_1005Metric, symbol Device:R
- removed R? (x2): 10k, Resistor_SMD:R_0402_1005Metric, symbol Device:R
- removed U? (x2): TLP785, Package_DIP:DIP-4_W7.62mm, symbol Isolator:TLP785
- added C23, C24: 0.1uF, Capacitor_SMD:C_0402_1005Metric, symbol Device:C
- added J3: Conn_01x10_Male, BoxHeader_1.27mm:BoxHeader_2x05_P1.27mm_Horizontal, symbol Connector:Conn_01x10_Male
- added Q17, Q18: BSS138, Package_TO_SOT_SMD:SOT-23, symbol Device:Q_NMOS_GSD
- added R38, R39: 47, Resistor_SMD:R_0603_1608Metric, symbol Device:R
- added R43, R44, R54, R55: 10k, Resistor_SMD:R_0402_1005Metric, symbol Device:R
- added R47, R48: 470, Resistor_SMD:R_0402_1005Metric, symbol Device:R
- added U7, U8: TLP2361, Package_SO:SO-6_4.4x3.6mm_P1.27mm, symbol Isolator:TLP2761
- JP1, JP2: renamed from JP?; footprint (none) -> Jumper:SolderJumper-3_P2.0mm_Open_TrianglePad1.0x1.5mm_NumberLabels
- Q10, Q12, Q14, Q15, Q16, Q4, Q6, Q8: renamed from Q?; value 2PB709AR -> S8050; footprint Package_TO_SOT_SMD:SC-59_Handsoldering -> Package_TO_SOT_SMD:SOT-23
- Y1: renamed from Y?; footprint (none) -> Crystal:Crystal_SMD_HC49-SD_HandSoldering
- gave numbers to parts that had none: 160
Connections:
- net +3.3V: now also R47.1, R48.1
- net +5V: now also C23.1, C24.1, U7.6 (VDD), U8.6 (VDD)
- net 3.3VBUS: now also J3.1 (Pin_1)
- net GND: now also C23.2, C24.2, J3.4 (Pin_4), Q17.2 (S), Q18.2 (S), R43.1, R44.1, R54.1, R55.1, U7.3 (K), U7.4 (GND), U8.3 (K), U8.4 (GND)
- net NRST: now also J3.6 (Pin_6)
- net PWM_A: now also R38.1
- net PWM_B: now also R39.1
- net STLinkRX: now also J3.9 (Pin_9)
- net STLinkTX: now also J3.8 (Pin_8)
- net TCK: now also J3.3 (Pin_3)
- net TMS: now also J3.5 (Pin_5)
- net VCC: now also C22.2, C27.1, C28.1, D16.2 (A), D17.2 (A), U10.1 (VCC), U4.5 (V+), U9.1 (VCC)
- net VDD: no longer C22.2, U4.5 (V+)
- net Vdrive: no longer C27.1, C28.1, D16.2 (A), D17.2 (A), U10.1 (VCC), U9.1 (VCC)
- net at U10.2 (IN): now also R55.2, U8.5 (VO)
- net at U9.2 (IN): now also R54.2, U7.5 (VO)
- new net: Q18.1 (G), R39.2, R44.2
- new net: Q18.3 (D), R48.2, U8.1 (A)
- new net: Q17.3 (D), R47.2, U7.1 (A)
- new net: Q17.1 (G), R38.2, R43.2
- no-connect marks 19 -> 5
Other:
- moved on the sheet: C22, C27, C28, C29, C30, D16, D17, D20, D21, D22, D23, Q19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

Commit message: diagram_SmallPW
Parts:
- removed C1, C12: 4.7uF, Capacitor_SMD:C_0603_1608Metric, symbol Device:C
- removed J10: Conn_01x04_Male, Connector_Molex:Molex_SPOX_5268-04A_1x04_P2.50mm_Horizontal, symbol Connector:Conn_01x04_Male
- added C? (x2): 1uF, Capacitor_SMD:C_0402_1005Metric, symbol Device:C
- added J?: Conn_01x04_Male, Connector_Molex:Molex_SPOX_5267-04A_1x04_P2.50mm_Vertical, symbol Connector:Conn_01x04_Male
- J4: footprint Connector_Molex:Molex_SPOX_5268-02A_1x02_P2.50mm_Horizontal -> Connector_Molex:Molex_SPOX_5267-02A_1x02_P2.50mm_Vertical
- J9: footprint Connector_Molex:Molex_SPOX_5268-04A_1x04_P2.50mm_Horizontal -> Connector_Molex:Molex_SPOX_5267-04A_1x04_P2.50mm_Vertical
Connections:
- net 3.3VSYS: now also C?.1
- net GND: now also J?.1 (Pin_1), J?.2 (Pin_2)
- net RS485b_A: now also J?.3 (Pin_3)
- net RS485b_B: now also J?.4 (Pin_4)
- net S-S: now also C?.1
- net at Q3.1 (G), R8.2, R9.1: now also C?.2
- net at Q11.1 (G), R27.2, R29.1: now also C?.2
Changed lines of the file:
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@@
   (junction (at 127 167.64) (diameter 0) (color 0 0 0 0)
   )
-  (junction (at 708.66 251.46) (diameter 0) (color 0 0 0 0)
-  )
   (junction (at 640.08 215.9) (diameter 0) (color 0 0 0 0)
   )
@@
   (junction (at 629.92 388.62) (diameter 0) (color 0 0 0 0)
   )
+  (junction (at 708.66 251.46) (diameter 0) (color 0 0 0 0)
+  )
   (junction (at 116.84 492.76) (diameter 0) (color 0 0 0 0)
   )
@@
     (pin "2")
   )
+  (symbol (lib_id "Connector:Conn_01x04_Male") (at 713.74 254 0) (mirror y) (unit 1)
+    (in_bom yes) (on_board yes)
+    (property "Reference" "J?" (id 0) (at 693.42 243.84 0)
+      (effects (font (size 1.27 1.27)) (justify right))
+    )
+    (property "Value" "Conn_01x04_Male" (id 1) (at 693.42 246.38 0)
+      (effects (font (size 1.27 1.27)) (justify right))
+    )
+    (property "Footprint" "Connector_Molex:Molex_SPOX_5267-04A_1x04_P2.50mm_Vertical" (id 2) (at 713.74 254 0)
+      (effects (font (size 1.27 1.27)) hide)
+    )
+    (property "Datasheet" "~" (id 3) (at 713.74 254 0)
+      (effects (font (size 1.27 1.27)) hide)
+    )
+    (pin "1")
+    (pin "2")
+    (pin "3")
+    (pin "4")
+  )
   (symbol (lib_id "Connector:Conn_01x04_Male") (at 713.74 226.06 0) (mirror y) (unit 1)
     (in_bom yes) (on_board yes)
@@
       (effects (font (size 1.27 1.27)) (justify right))
     )
-    (property "Footprint" "Connector_Molex:Molex_SPOX_5268-04A_1x04_P2.50mm_Horizontal" (id 2) (at 713.74 226.06 0)
+    (property "Footprint" "Connector_Molex:Molex_SPOX_5267-04A_1x04_P2.50mm_Vertical" (id 2) (at 713.74 226.06 0)
       (effects (font (size 1.27 1.27)) hide)
     )
@@
     (pin "2")
   )
-  (symbol (lib_id "Device:C") (at 134.62 172.72 0) (unit 1)
-    (in_bom yes) (on_board yes) (fields_autoplaced)
-    (property "Reference" "C1" (id 0) (at 138.43 171.4499 0)
-      (effects (font (size 1.27 1.27)) (justify left))
-    )
-    (property "Value" "4.7uF" (id 1) (at 138.43 173.9899 0)
-      (effects (font (size 1.27 1.27)) (justify left))
-    )
-    (property "Footprint" "Capacitor_SMD:C_0603_1608Metric" (id 2) (at 135.5852 176.53 0)
-      (effects (font (size 1.27 1.27)) hide)
-    )
-    (property "Datasheet" "~" (id 3) (at 134.62 172.72 0)
-      (effects (font (size 1.27 1.27)) hide)
-    )
-    (pin "1")
-    (pin "2")
-  )
   (symbol (lib_id "power:+5V") (at 203.2 177.8 0) (unit 1)
     (in_bom yes) (on_board yes) (fields_autoplaced)
@@
     (pin "2")
   )
+  (symbol (lib_id "Device:C") (at 335.28 114.3 0) (unit 1)
+    (in_bom yes) (on_board yes) (fields_autoplaced)
+    (property "Reference" "C?" (id 0) (at 339.09 113.0299 0)
+      (effects (font (size 1.27 1.27)) (justify left))
+    )
+    (property "Value" "1uF" (id 1) (at 339.09 115.5699 0)
+      (effects (font (size 1.27 1.27)) (justify left))
+    )
+    (property "Footprint" "Capacitor_SMD:C_0402_1005Metric" (id 2) (at 336.2452 118.11 0)
+      (effects (font (size 1.27 1.27)) hide)
+    )
+    (property "Datasheet" "~" (id 3) (at 335.28 114.3 0)
+      (effects (font (size 1.27 1.27)) hide)
+    )
+    (pin "1")
+    (pin "2")
+  )
   (symbol (lib_id "power:GND") (at 231.14 175.26 0) (mirror y) (unit 1)
     (in_bom yes) (on_board yes) (fields_autoplaced)
@@
     (pin "2")
   )
+  (symbol (lib_id "Device:C") (at 134.62 172.72 0) (unit 1)
+    (in_bom yes) (on_board yes) (fields_autoplaced)
+    (property "Reference" "C?" (id 0) (at 138.43 171.4499 0)
+      (effects (font (size 1.27 1.27)) (justify left))
+    )
+    (property "Value" "1uF" (id 1) (at 138.43 173.9899 0)
+      (effects (font (size 1.27 1.27)) (justify left))
+    )
+    (property "Footprint" "Capacitor_SMD:C_0402_1005Metric" (id 2) (at 135.5852 176.53 0)
+      (effects (font (size 1.27 1.27)) hide)
+    )
+    (property "Datasheet" "~" (id 3) (at 134.62 172.72 0)
+      (effects (font (size 1.27 1.27)) hide)
+    )
+    (pin "1")
+    (pin "2")
+  )
   (symbol (lib_id "Device:R") (at 640.08 111.76 0) (unit 1)
     (in_bom yes) (on_board yes) (fields_autoplaced)
@@
       (effects (font (size 1.27 1.27)) (justify right))
     )
-    (property "Footprint" "Connector_Molex:Molex_SPOX_5268-02A_1x02_P2.50mm_Horizontal" (id 2) (at 238.76 175.26 0)
+    (property "Footprint" "Connector_Molex:Molex_SPOX_5267-02A_1x02_P2.50mm_Vertical" (id 2) (at 238.76 175.26 0)
       (effects (font (size 1.27 1.27)) hide)
     )
@@
     (pin "2")
   )
-  (symbol (lib_id "Connector:Conn_01x04_Male") (at 713.74 254 0) (mirror y) (unit 1)
-    (in_bom yes) (on_board yes)
-    (property "Reference" "J10" (id 0) (at 693.42 243.84 0)
-      (effects (font (size 1.27 1.27)) (justify right))
-    )
-    (property "Value" "Conn_01x04_Male" (id 1) (at 693.42 246.38 0)
-      (effects (font (size 1.27 1.27)) (justify right))
-    )
-    (property "Footprint" "Connector_Molex:Molex_SPOX_5268-04A_1x04_P2.50mm_Horizontal" (id 2) (at 713.74 254 0)
-      (effects (font (size 1.27 1.27)) hide)
-    )
-    (property "Datasheet" "~" (id 3) (at 713.74 254 0)
-      (effects (font (size 1.27 1.27)) hide)
-    )
-    (pin "1")
-    (pin "2")
-    (pin "3")
-    (pin "4")
-  )
   (symbol (lib_id "Device:LED") (at 177.8 467.36 180) (unit 1)
     (in_bom yes) (on_board yes)
@@
     (pin "8")
   )
-  (symbol (lib_id "Device:C") (at 335.28 114.3 0) (unit 1)
-    (in_bom yes) (on_board yes) (fields_autoplaced)
-    (property "Reference" "C12" (id 0) (at 339.09 113.0299 0)
-      (effects (font (size 1.27 1.27)) (justify left))
-    )
-    (property "Value" "4.7uF" (id 1) (at 339.09 115.5699 0)
-      (effects (font (size 1.27 1.27)) (justify left))
-    )
-    (property "Footprint" "Capacitor_SMD:C_0603_1608Metric" (id 2) (at 336.2452 118.11 0)
-      (effects (font (size 1.27 1.27)) hide)
-    )
-    (property "Datasheet" "~" (id 3) (at 335.28 114.3 0)
-      (effects (font (size 1.27 1.27)) hide)
-    )
-    (pin "1")
-    (pin "2")
-  )
   (symbol (lib_id "Jumper:SolderJumper_3_Bridged12") (at 149.86 383.54 90) (mirror x) (unit 1)
     (in_bom yes) (on_board yes)
@@
       (reference "#PWR?") (unit 1) (value "VCC") (footprint "")
     )
-    (path "/6936d961-11c4-4e09-9223-0262ada36838"
-      (reference "C1") (unit 1) (value "4.7uF") (footprint "Capacitor_SMD:C_0603_1608Metric")
-    )
     (path "/bbdd3b61-11a7-46b7-b4b7-a55454e7cad2"
       (reference "C2") (unit 1) (value "0.1uF") (footprint "Capacitor_SMD:C_0402_1005Metric")
@@
       (reference "C11") (unit 1) (value "1uF") (footprint "Capacitor_SMD:C_0402_1005Metric")
     )
-    (path "/c5a6ad3d-dcca-4acd-aa27-b58b7ca69e3e"
-      (reference "C12") (unit 1) (value "4.7uF") (footprint "Capacitor_SMD:C_0603_1608Metric")
-    )
     (path "/1dc44e7f-991a-4259-ba61-292d4bc7617c"
       (reference "C13") (unit 1) (value "470uF") (footprint "Capacitor_SMD:C_Elec_8x10.2")
@@
       (reference "C31") (unit 1) (value "1uF") (footprint "Capacitor_SMD:C_0402_1005Metric")
     )
+    (path "/7062d2aa-fe52-48ef-9275-c028cc8f7d47"
+      (reference "C?") (unit 1) (value "1uF") (footprint "Capacitor_SMD:C_0402_1005Metric")
+    )
+    (path "/92eed252-6949-45d7-9800-913c151ec4a1"
+      (reference "C?") (unit 1) (value "1uF") (footprint "Capacitor_SMD:C_0402_1005Metric")
+    )
     (path "/aeefa2bc-73c3-4c64-9371-e521f6cfa836"
       (reference "D1") (unit 1) (value "SBR1A40SA") (footprint "Diode_SMD:D_SMA_Handsoldering")
@@
     )
     (path "/a45597b6-5df7-4cc7-856e-5e345443f290"
-      (reference "J4") (unit 1) (value "Conn_01x02_Male") (footprint "Connector_Molex:Molex_SPOX_5268-02A_1x02_P2.50mm_Horizontal")
+      (reference "J4") (unit 1) (value "Conn_01x02_Male") (footprint "Connector_Molex:Molex_SPOX_5267-02A_1x02_P2.50mm_Vertical")
     )
     (path "/a767b4f7-7e2c-4234-b3fb-7f60e8d3efbf"
@@
     )
     (path "/378ab376-8e97-4a76-83f3-df0bb036d26c"
-      (reference "J9") (unit 1) (value "Conn_01x04_Male") (footprint "Connector_Molex:Molex_SPOX_5268-04A_1x04_P2.50mm_Horizontal")
+      (reference "J9") (unit 1) (value "Conn_01x04_Male") (footprint "Connector_Molex:Molex_SPOX_5267-04A_1x04_P2.50mm_Vertical")
     )
-    (path "/bc1ece65-651e-4f69-a556-534813865c76"
-      (reference "J10") (unit 1) (value "Conn_01x04_Male") (footprint "Connector_Molex:Molex_SPOX_5268-04A_1x04_P2.50mm_Horizontal")
+    (path "/352c4f13-d60c-469c-b25c-52a3262bc664"
+      (reference "J?") (unit 1) (value "Conn_01x04_Male") (footprint "Connector_Molex:Molex_SPOX_5267-04A_1x04_P2.50mm_Vertical")
     )
     (path "/4f60d6c5-3451-445a-8755-7109c9c928d5"

Commit message: 回路図pdf出力
Parts:
- removed R37: 10mR, symbol Device:R
- added R? (x4): 40mR, Resistor_SMD:R_2512_6332Metric, symbol Device:R
Connections:
- net VDD: now also R?.2, R?.2, R?.2, R?.2
- net Vdrive: now also R?.1, R?.1, R?.1, R?.1

Commit message: 進捗
Parts:
- C20, C21: value 4.7uF -> 10uF; footprint Capacitor_SMD:C_0805_2012Metric_Pad1.18x1.45mm_HandSolder -> Capacitor_SMD:C_0805_2012Metric
- C3: footprint Capacitor_SMD:C_0805_2012Metric_Pad1.18x1.45mm_HandSolder -> Capacitor_SMD:C_0805_2012Metric
- D1, D15, D7, D8, D9: value SBR1A40SA -> 1N5819WS; footprint Diode_SMD:D_SMA_Handsoldering -> Diode_SMD:D_SOD-323_HandSoldering
- D16, D17: value SBR1A40SA -> SS2040FL; footprint Diode_SMD:D_SMA_Handsoldering -> Diode_SMD:D_SOD-123
- gave numbers to parts that had none: 7

Commit message: エンコーダー基板配線完了
Parts:
- removed C12: 1uF, Capacitor_SMD:C_0402_1005Metric, symbol Device:C
- removed C8, C9: 22pF, Capacitor_SMD:C_0603_1608Metric, symbol Device:C
- removed D10: D_Zener, Diode_SMD:D_SOD-323_HandSoldering, symbol Device:D_Zener
- removed D12, D13: Green, LED_SMD:LED_0603_1608Metric_Pad1.05x0.95mm_HandSolder, symbol Device:LED
- removed H1, H3: MountingHole_Pad, TestPoint:TestPoint_Pad_1.5x1.5mm, symbol Mechanical:MountingHole_Pad
- removed Q10, Q12, Q14, Q8: S8050, Package_TO_SOT_SMD:SOT-23, symbol Device:Q_PNP_BEC
- removed Q11, Q13, Q7, Q9: SSM3J332R, Package_TO_SOT_SMD:SOT-23W, symbol Device:Q_PMOS_GSD
- removed R21, R23, R25, R26, R28, R29, R30, R31, R32: 10k, Resistor_SMD:R_0402_1005Metric, symbol Device:R
- removed R24, R34, R35: 1k, Resistor_SMD:R_0402_1005Metric, symbol Device:R
- removed R27: 100k, Resistor_SMD:R_0402_1005Metric, symbol Device:R
- removed R69, R70: 40mR, Resistor_SMD:R_2512_6332Metric, symbol Device:R
- removed Y1: 48MHz, Crystal:Crystal_SMD_HC49-SD_HandSoldering, symbol Device:Crystal
- added U11: NJU6319AE, Package_SO:SOP-8_3.9x4.9mm_P1.27mm, symbol CrystalOSC_Control:NJU6319AE
- added Y1: 16MHz, Crystal:Crystal_SMD_3225-4Pin_3.2x2.5mm_HandSoldering, symbol Device:Crystal_GND24
- C7: value ADJ_ST -> 0.1uF; footprint Capacitor_SMD:C_0603_1608Metric -> Capacitor_SMD:C_0402_1005Metric
- Q1, Q3: footprint Package_TO_SOT_SMD:TO-252-3_TabPin2 -> Package_TO_SOT_SMD:TO-252-2
- R37, R68: value 40mR -> 20mR
Connections:
- net 3.3VSYS is gone; now on net +3.3V: C6.1, D8.2 (A), R22.2, U2.2 (VO)
- net +3.3V: now also C7.1, U11.1 (~{CONT}), U11.8 (VDD)
- net GND: now also C7.2, U11.4 (VSS), Y1.2, Y1.4; no longer C7.1
- net Motor_A: now also C31.2, D18.1 (K), D19.2 (A); no longer R62.1, R67.2
- net Motor_B: now also R62.1, R67.2; no longer C31.2, D18.1 (K), D19.2 (A)
- net NRST: now also U3.6 (PF2-NRST)
- net OSC_IN: now also U3.2 (PC14-OSCX_IN), U11.5 (FOUT)
- new net: U11.2 (XT), Y1.1
- new net: U11.3 (~{XT}), Y1.3
- new net: U11.6 (NC), U11.7 (NC)
- no-connect marks 5 -> 6
Other:
- note removed: "理想ダイオード/3.3VSYS"
- note removed: "電源切替/STLink"
- moved on the sheet: C11, C13, C14, C15, C16, C17, C18, C19, C22, C5, C6, D11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
