File: LargeMD/LargeMD.kicad_sch (KiCad schematic)
At the start: 159 parts, among them J1 Conn_01x02_Male, J10 Conn_01x04_Male, J2 Conn_01x02_Female, J3 Conn_01x10_Male, J4 Conn_01x02_Male, J5 Conn_01x03_Male, J6 Conn_01x02_Female, J7 Conn_01x04_Male, J8 Conn_01x04_Male, J9 Conn_01x04_Male, Q1 TJ60S04M3L, Q15 S8050, Q16 S8050, Q17 BSS138, Q18 BSS138, Q19 TPH3R704PL, Q2 BSS138, Q20 TPH3R704PL, Q21 TPH3R704PL, Q22 TPH3R704PL, Q3 TJ60S04M3L, Q4 S8050, Q5 SSM3J332R, Q6 S8050, SW1 SW_DIP_x05, SW2 SW_SPDT, SW3 SW_SPDT, SW4 SW_SPST, U1 LF50_TO220, U10 IR2302, U11 NJU6319AE, U2 AZ1084CD-3.3, U3 STM32C031K4T6, U4 LT6106, U5 MAX3485, U6 MAX3485, U7 TLP2361, U8 TLP2361, U9 IR2302, Y1 16MHz

Commit message: LargeMD
Parts:
- removed C2: 0.1uF, Capacitor_SMD:C_0402_1005Metric, symbol Device:C
Connections:
- net 3.3VBUS: no longer names the net of J3.1 (Pin_1)
- no-connect marks 6 -> 7
Changed lines of the file:
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@@
   (junction (at 134.62 167.64) (diameter 0) (color 0 0 0 0)
   )
-  (junction (at 165.1 312.42) (diameter 0) (color 0 0 0 0)
-  )
   (junction (at 629.92 340.36) (diameter 0) (color 0 0 0 0)
   )
@@
   (junction (at 231.14 116.84) (diameter 0) (color 0 0 0 0)
   )
-  (junction (at 160.02 304.8) (diameter 0) (color 0 0 0 0)
-  )
   (junction (at 78.74 474.98) (diameter 0) (color 0 0 0 0)
   )
@@
   (no_connect (at 157.48 111.76))
   (no_connect (at 104.14 436.88))
+  (no_connect (at 152.4 304.8))
   (no_connect (at 152.4 307.34))
   (no_connect (at 152.4 320.04))
@@
     (stroke (width 0.5) (type solid) (color 0 0 0 0))
   )
-  (wire (pts (xy 160.02 304.8) (xy 165.1 304.8))
-    (stroke (width 0) (type default) (color 0 0 0 0))
-  )
   (wire (pts (xy 299.72 368.3) (xy 299.72 369.57))
     (stroke (width 0) (type default) (color 0 0 0 0))
@@
     (stroke (width 0) (type default) (color 0 0 0 0))
   )
-  (wire (pts (xy 152.4 304.8) (xy 160.02 304.8))
-    (stroke (width 0) (type default) (color 0 0 0 0))
-  )
   (wire (pts (xy 703.58 494.03) (xy 703.58 500.38))
     (stroke (width 0) (type default) (color 0 0 0 0))
@@
     (stroke (width 0) (type default) (color 0 0 0 0))
   )
-  (wire (pts (xy 160.02 302.26) (xy 160.02 304.8))
-    (stroke (width 0) (type default) (color 0 0 0 0))
-  )
   (polyline (pts (xy 726.44 170.18) (xy 726.44 76.2))
     (stroke (width 0.5) (type solid) (color 0 0 0 0))
@@
     (effects (font (size 1.27 1.27)) (justify left bottom))
   )
-  (label "3.3VBUS" (at 160.02 302.26 0)
-    (effects (font (size 1.27 1.27)) (justify left bottom))
-  )
   (label "12VBAT" (at 121.92 121.92 0)
     (effects (font (size 1.27 1.27)) (justify left bottom))
@@
     (pin "1")
   )
-  (symbol (lib_id "Device:C") (at 165.1 308.61 0) (unit 1)
-    (in_bom yes) (on_board yes)
-    (property "Reference" "C2" (id 0) (at 170.18 307.34 0)
-      (effects (font (size 1.27 1.27)) (justify left))
-    )
-    (property "Value" "0.1uF" (id 1) (at 170.18 309.88 0)
-      (effects (font (size 1.27 1.27)) (justify left))
-    )
-    (property "Footprint" "Capacitor_SMD:C_0402_1005Metric" (id 2) (at 166.0652 312.42 0)
-      (effects (font (size 1.27 1.27)) hide)
-    )
-    (property "Datasheet" "~" (id 3) (at 165.1 308.61 0)
-      (effects (font (size 1.27 1.27)) hide)
-    )
-    (pin "1")
-    (pin "2")
-  )
   (symbol (lib_id "Device:LED") (at 177.8 467.36 180) (unit 1)
     (in_bom yes) (on_board yes)
@@
       (reference "C1") (unit 1) (value "1uF") (footprint "Capacitor_SMD:C_0402_1005Metric")
     )
-    (path "/bbdd3b61-11a7-46b7-b4b7-a55454e7cad2"
-      (reference "C2") (unit 1) (value "0.1uF") (footprint "Capacitor_SMD:C_0402_1005Metric")
-    )
     (path "/ef77236e-b70d-44a5-85a4-b73389d29ea2"

Commit message: LargeMDほぼ完成
Parts:
- removed H4, H5, H6, H7, H8, H9: MountingHole, MountingHole:MountingHole_3.2mm_M3, symbol Mechanical:MountingHole
- removed TP1, TP2, TP3: TestPoint, TestPoint:TestPoint_THTPad_D2.0mm_Drill1.0mm, symbol Connector:TestPoint
- U3: value STM32C031K4T6 -> STM32G030K6T6
Connections:
- net MainRX_RS485aTX is gone; now on net MainRX2_RS485bTX: U5.1 (RO)
- net MainRX_RS485bTX is gone; now on net MainRX1_RS485aTX: JP1.2 (C)
- net MainTX_RS485aRX is gone; now on net MainTX2_RS485bRX: R40.2, U5.4 (DI)
- net MainTX_RS485bRX is gone; now on net MainTX1_RS485aRX: JP2.2 (C)
- net Current_Sence: now also U3.11 (PA4)
- net DIP_SW0: now also U3.22 (PA11[PA9])
- net DIP_SW1: now also U3.20 (PC6)
- net DIP_SW2: now also U3.18 (PA8)
- net DIP_SW3: now also U3.17 (PB2)
- net DIP_SW4: now also U3.16 (PB1)
- net LED0: now also U3.29 (PB5)
- net LED1: now also U3.28 (PB4)
- net LED2: now also U3.27 (PB3)
- net MonitorLED0: now also U3.31 (PB7)
- net PWM_A: now also U3.13 (PA6)
- net PWM_B: now also U3.30 (PB6)
- net RS485a_A: now also J10.3 (Pin_3), J9.3 (Pin_3), JP4.1 (A), R52.2, U6.6 (A); no longer J7.3 (Pin_3), J8.3 (Pin_3), JP3.1 (A), R50.2, U5.6 (A)
- net RS485a_B: now also J10.4 (Pin_4), J9.4 (Pin_4), R53.1, R57.2, U6.7 (B); no longer J7.4 (Pin_4), J8.4 (Pin_4), R51.1, R56.2, U5.7 (B)
- net RS485b_A: now also J7.3 (Pin_3), J8.3 (Pin_3), JP3.1 (A), R50.2, U5.6 (A); no longer J10.3 (Pin_3), J9.3 (Pin_3), JP4.1 (A), R52.2, U6.6 (A)
- net RS485b_B: now also J7.4 (Pin_4), J8.4 (Pin_4), R51.1, R56.2, U5.7 (B); no longer J10.4 (Pin_4), J9.4 (Pin_4), R53.1, R57.2, U6.7 (B)
- net SHDN: now also U3.12 (PA5)
- net Sensor0: now also U3.15 (PB0)
- net Slide_SW0: now also U3.8 (PA1)
- net TCK: now also U3.25 (PA14-BOOT0)
- net TMS: now also U3.24 (PA13)
- net V_Measure: now also U3.10 (PA3)
- net MainTX1_RS485aRX: now reaches U3.19 (PA9)
- net MainRX1_RS485aTX: now reaches U3.21 (PA10)
- net MainRX2_RS485bTX: now reaches U3.26 (PA15)
- net MainTX2_RS485bRX: now reaches U3.9 (PA2)
- net at U11.6 (NC): no longer U11.7 (NC)
- net RS485bRX renamed RS485aRX
- net RS485bTX renamed RS485aTX
- no-connect marks 7 -> 12
Other:
- note removed: "ねじ穴"
- moved on the sheet: C25, C26, J10, J7, J8, J9, JP3, JP4, Q15, Q16, R40, R41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
