File: LargeMD/LargeMD.kicad_pcb (KiCad board)
At the start: 2 copper layers, 110 x 60 mm, 149 parts, among them J1 Conn_01x02_Male, J10 Conn_01x04_Male, J2 Conn_01x02_Female, J3 Conn_01x10_Male, J4 Conn_01x02_Male, J5 Conn_01x03_Male, J6 Conn_01x02_Female, J7 Conn_01x04_Male, J8 Conn_01x04_Male, J9 Conn_01x04_Male, Q1 TJ60S04M3L, Q15 S8050, Q16 S8050, Q17 BSS138, Q18 BSS138, Q19 TPH3R704PL, Q2 BSS138, Q20 TPH3R704PL, Q21 TPH3R704PL, Q22 TPH3R704PL, Q3 TJ60S04M3L, Q4 S8050, Q5 SSM3J332R, Q6 S8050, SW1 SW_DIP_x05, SW2 SW_SPDT, SW3 SW_SPDT, SW4 SW_SPST, U1 LF50_TO220, U10 IR2302, U11 NJU6319AE, U2 AZ1084CD-3.3, U3 STM32G030K6T6, U4 LT6106, U5 MAX3485, U6 MAX3485, U7 TLP2361, U8 TLP2361, U9 IR2302, Y1 16MHz

Commit message: 製造ファイル出力
Other:
- board text added: "3.3V"
- board text added: "5V"
- board text added: "ADC"
- board text added: "Designed by @cat_nekonekone"
- board text added: "GND"
- board text added: "ID"
- board text added: "JLCJLCJLCJLC"
- board text added: "Motor"
- board text added: "MotorOUT"
- board text added: "NRST"
- board text added: "PA1"
- board text added: "PA11"
- board text added: "PA8"
- board text added: "PB1"
- board text added: "PB2"
- board text added: "PB3"
- board text added: "PB4"
- board text added: "PB5"
- board text added: "PB7"
- board text added: "PC6"
- board text added: "POWER"
- board text added: "RX1:PA10"
- board text added: "RX2:PA15"
- board text added: "TX1:PA9"
- board text added: "TX2:PA2"
- board text added: "Tomoshibi"
- board text added: "[5VOUT]"
- board text added: "[I_meas.]PA4"
- board text added: "[PWM_A]PA6"
- board text added: "[PWM_B]PB6"
- board text added: "[RS485a]"
- board text added: "[RS485b]"
- board text added: "[SHDN]PA5"
- board text added: "[Sensor0]"
- board text added: "[Sensor0]PB0"
- board text added: "[V_meas.]PA3"
- board text added: "燈"

Commit message: 製造ファイル出力その2
Other:
- board text added: "[Volume]"
- board text added: "[Volume]PB0"
- board text removed: "[Sensor0]"
- board text removed: "[Sensor0]PB0"
Changed lines of the file:
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@@
     (effects (font (size 1.2 1.2) (thickness 0.15)))
   )
-  (gr_text "[Sensor0]" (at 78 89.95 90) (layer "F.SilkS")
+  (gr_text "[Volume]" (at 78 90 90) (layer "F.SilkS")
     (effects (font (size 1 1) (thickness 0.13)))
   )
@@
     (effects (font (size 1 1) (thickness 0.12)))
   )
-  (gr_text "[Sensor0]PB0" (at 124 89.325) (layer "F.SilkS")
+  (gr_text "[Volume]PB0" (at 124.3 89.3) (layer "F.SilkS")
     (effects (font (size 1 1) (thickness 0.12)))
   )
@@
     (effects (font (size 1 1) (thickness 0.12)))
   )
-  (gr_text "[RS485a]" (at 113.5 46) (layer "F.SilkS")
+  (gr_text "[RS485b]" (at 113.5 46) (layer "F.SilkS")
     (effects (font (size 1 1) (thickness 0.13)))
   )
