File: Panel/Panel.kicad_sch (KiCad schematic)
At the start: 130 parts, among them J1 Conn_01x02_Male, J2 Conn_01x02_Female, J3 Conn_01x10_Male, J4 Conn_01x04_Male, J5 Conn_01x04_Male, Q1 MTP4835I3, Q10 SSM3J332R, Q11 S8050, Q12 SSM3J332R, Q13 S8050, Q14 S8050, Q15 BSS138, Q2 BSS138, Q3 MTP4835I3, Q4 SSM3J332R, Q5 2SC3265, Q6 S8050, Q7 SSM3J332R, Q8 MTP4835I3, Q9 S8050, SW1 SW_DIP_x05, SW2 SW_SPDT, SW3 SW_SPDT_White, SW4 SW_SPST, U1 MC34063AD, U2 AZ1084CD-3.3, U3 STM32G050F6P6, U4 MAX3485, U5 NJU6319AE, Y1 16MHz

Commit message: LargeMD
Parts:
- added U?: STM32C031K4T6, Package_QFP:LQFP-32_7x7mm_P0.8mm, symbol STM32C031K4T6:STM32C031K4T6
Connections:
- net +3.3V: now also U?.4 (VDD/VDDA)
- net GND: now also U?.5 (VSS/VSSA)
- no-connect marks 6 -> 7
Other:
- moved on the sheet: U3

Commit message: LargeMDほぼ完成
Parts:
- gave numbers to parts that had none: 1
Connections:
- net at U5.6 (NC): no longer U5.7 (NC)
- net LED1_or_MainRX_STLinkTX renamed LED1_or_MainRX1_STLinkTX
- net LED2_or_MainTX_STLinkRX renamed LED2_or_MainTX1_STLinkRX
- net MainRX_RS485TX renamed MainRX2_RS485TX
- net MainTX_RS485RX renamed MainTX2_RS485RX
Changed lines of the file:
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@@
     )
   )
-  (global_label "LED1_or_MainRX_STLinkTX" (shape bidirectional) (at 162.56 233.68 0) (fields_autoplaced)
+  (global_label "LED1_or_MainRX1_STLinkTX" (shape bidirectional) (at 162.56 233.68 0) (fields_autoplaced)
     (effects (font (size 1.27 1.27)) (justify left))
-    (property "Intersheet References" "${INTERSHEET_REFS}" (id 0) (at 189.466 233.6006 0)
+    (property "Intersheet References" "${INTERSHEET_REFS}" (id 0) (at 190.6755 233.6006 0)
       (effects (font (size 1.27 1.27)) (justify left) hide)
     )
@@
     )
   )
-  (global_label "MainRX_RS485TX" (shape bidirectional) (at 327.66 309.88 180) (fields_autoplaced)
+  (global_label "MainRX2_RS485TX" (shape bidirectional) (at 327.66 309.88 180) (fields_autoplaced)
     (effects (font (size 1.27 1.27)) (justify right))
-    (property "Intersheet References" "${INTERSHEET_REFS}" (id 0) (at 309.1602 309.8006 0)
+    (property "Intersheet References" "${INTERSHEET_REFS}" (id 0) (at 307.9507 309.8006 0)
       (effects (font (size 1.27 1.27)) (justify right) hide)
     )
@@
     )
   )
-  (global_label "MainTX_RS485RX" (shape bidirectional) (at 327.66 307.34 180) (fields_autoplaced)
+  (global_label "MainTX2_RS485RX" (shape bidirectional) (at 327.66 307.34 180) (fields_autoplaced)
     (effects (font (size 1.27 1.27)) (justify right))
-    (property "Intersheet References" "${INTERSHEET_REFS}" (id 0) (at 309.1602 307.2606 0)
+    (property "Intersheet References" "${INTERSHEET_REFS}" (id 0) (at 307.9507 307.2606 0)
       (effects (font (size 1.27 1.27)) (justify right) hide)
     )
@@
     )
   )
-  (global_label "MainTX_RS485RX" (shape bidirectional) (at 449.58 121.92 180) (fields_autoplaced)
+  (global_label "MainTX2_RS485RX" (shape bidirectional) (at 449.58 121.92 180) (fields_autoplaced)
     (effects (font (size 1.27 1.27)) (justify right))
-    (property "Intersheet References" "${INTERSHEET_REFS}" (id 0) (at 431.0802 121.8406 0)
+    (property "Intersheet References" "${INTERSHEET_REFS}" (id 0) (at 429.8707 121.8406 0)
       (effects (font (size 1.27 1.27)) (justify right) hide)
     )
   )
-  (global_label "LED1_or_MainRX_STLinkTX" (shape bidirectional) (at 327.66 279.4 180) (fields_autoplaced)
+  (global_label "LED1_or_MainRX1_STLinkTX" (shape bidirectional) (at 327.66 279.4 180) (fields_autoplaced)
     (effects (font (size 1.27 1.27)) (justify right))
-    (property "Intersheet References" "${INTERSHEET_REFS}" (id 0) (at 300.754 279.4794 0)
+    (property "Intersheet References" "${INTERSHEET_REFS}" (id 0) (at 299.5445 279.3206 0)
       (effects (font (size 1.27 1.27)) (justify right) hide)
     )
@@
     )
   )
-  (global_label "MainRX_RS485TX" (shape bidirectional) (at 449.58 114.3 180) (fields_autoplaced)
+  (global_label "MainRX2_RS485TX" (shape bidirectional) (at 449.58 114.3 180) (fields_autoplaced)
     (effects (font (size 1.27 1.27)) (justify right))
-    (property "Intersheet References" "${INTERSHEET_REFS}" (id 0) (at 431.0802 114.2206 0)
+    (property "Intersheet References" "${INTERSHEET_REFS}" (id 0) (at 429.8707 114.2206 0)
       (effects (font (size 1.27 1.27)) (justify right) hide)
     )
@@
     )
   )
-  (global_label "LED2_or_MainTX_STLinkRX" (shape bidirectional) (at 327.66 276.86 180) (fields_autoplaced)
+  (global_label "LED2_or_MainTX1_STLinkRX" (shape bidirectional) (at 327.66 276.86 180) (fields_autoplaced)
     (effects (font (size 1.27 1.27)) (justify right))
-    (property "Intersheet References" "${INTERSHEET_REFS}" (id 0) (at 300.754 276.9394 0)
+    (property "Intersheet References" "${INTERSHEET_REFS}" (id 0) (at 299.5445 276.7806 0)
       (effects (font (size 1.27 1.27)) (justify right) hide)
     )
@@
     )
   )
-  (global_label "LED2_or_MainTX_STLinkRX" (shape bidirectional) (at 162.56 254 0) (fields_autoplaced)
+  (global_label "LED2_or_MainTX1_STLinkRX" (shape bidirectional) (at 162.56 254 0) (fields_autoplaced)
     (effects (font (size 1.27 1.27)) (justify left))
-    (property "Intersheet References" "${INTERSHEET_REFS}" (id 0) (at 189.466 253.9206 0)
+    (property "Intersheet References" "${INTERSHEET_REFS}" (id 0) (at 190.6755 253.9206 0)
       (effects (font (size 1.27 1.27)) (justify left) hide)
     )
@@
   (symbol (lib_id "power:GND") (at 393.7 332.74 0) (unit 1)
     (in_bom yes) (on_board yes)
-    (property "Reference" "#PWR?" (id 0) (at 393.7 339.09 0)
+    (property "Reference" "#PWR066" (id 0) (at 393.7 339.09 0)
       (effects (font (size 1.27 1.27)) hide)
     )
@@
   (symbol (lib_id "STM32C031K4T6:STM32C031K4T6") (at 378.46 256.54 0) (unit 1)
     (in_bom yes) (on_board yes) (fields_autoplaced)
-    (property "Reference" "U?" (id 0) (at 395.7194 245.11 0)
+    (property "Reference" "U6" (id 0) (at 395.7194 245.11 0)
       (effects (font (size 1.524 1.524)) (justify left))
     )
@@
   (symbol (lib_id "power:+3.3V") (at 393.7 246.38 0) (unit 1)
     (in_bom yes) (on_board yes) (fields_autoplaced)
-    (property "Reference" "#PWR?" (id 0) (at 393.7 250.19 0)
+    (property "Reference" "#PWR065" (id 0) (at 393.7 250.19 0)
       (effects (font (size 1.27 1.27)) hide)
     )
@@
       (reference "#PWR064") (unit 1) (value "GND") (footprint "")
     )
-    (path "/03a398ba-731a-497e-9db6-d68027e54cd6"
-      (reference "#PWR?") (unit 1) (value "GND") (footprint "")
-    )
     (path "/f4a6c672-4a9c-4257-b0ca-63e49eff18d5"
-      (reference "#PWR?") (unit 1) (value "+3.3V") (footprint "")
+      (reference "#PWR065") (unit 1) (value "+3.3V") (footprint "")
+    )
+    (path "/03a398ba-731a-497e-9db6-d68027e54cd6"
+      (reference "#PWR066") (unit 1) (value "GND") (footprint "")
     )
     (path "/80a753df-19c0-4d84-8de2-267b7a2c52b0"
@@
     )
     (path "/bd1399d5-9df0-410b-a8e0-dc6e6fab4ca5"
-      (reference "U?") (unit 1) (value "STM32C031K4T6") (footprint "Package_QFP:LQFP-32_7x7mm_P0.8mm")
+      (reference "U6") (unit 1) (value "STM32C031K4T6") (footprint "Package_QFP:LQFP-32_7x7mm_P0.8mm")
     )
     (path "/4ef317b3-fc20-43ef-a923-3db8650b082d"
