File: Panel/Panel.kicad_sch (KiCad schematic)
At the start: 118 parts, among them J1 Conn_01x02_Male, J2 Conn_01x02_Female, J3 Conn_01x10_Male, J4 Conn_01x04_Male, J5 Conn_01x04_Male, Q1 MTP4835I3, Q14 S8050, Q15 BSS138, Q2 BSS138, Q3 MTP4835I3, Q5 2SC3265, Q8 MTP4835I3, SW1 SW_DIP_x05, SW2 SW_SPDT, SW3 SW_SPDT_White, SW4 SW_SPST, U1 MC34063AD, U2 AZ1084CD-3.3, U3 STM32G050F6P6, U4 MAX3485, U5 NJU6319AE, U6 STM32C031K4T6, Y1 16MHz

Commit message: 回路図ほぼ完成
Parts:
- removed C2: 0.1uF, Capacitor_SMD:C_0402_1005Metric, symbol Device:C
- removed H4: MountingHole_Pad, TestPoint:TestPoint_THTPad_D3.0mm_Drill1.5mm, symbol Mechanical:MountingHole_Pad
- removed JP1, JP2: SolderJumper_3_Bridged12, Jumper:SolderJumper-3_P2.0mm_Open_TrianglePad1.0x1.5mm_NumberLabels, symbol Jumper:SolderJumper_3_Bridged12
- removed JP3: Jumper_2_Open, Connector_PinHeader_2.54mm:PinHeader_1x02_P2.54mm_Vertical, symbol Jumper:Jumper_2_Open
- removed U3: STM32G050F6P6, Package_SO:TSSOP-20_4.4x6.5mm_P0.65mm, symbol STM32C011F4P6:STM32C011F4P6
- added C10: 10uF, Capacitor_SMD:C_0805_2012Metric, symbol Device:C
- added D13, D9: 1N5819WS, Diode_SMD:D_SOD-323_HandSoldering, symbol Device:D_Schottky
- added H1: MountingHole_Pad, TestPoint:TestPoint_Pad_1.5x1.5mm, symbol Mechanical:MountingHole_Pad
- added JP1: Jumper_2_Open, Jumper:SolderJumper-2_P1.3mm_Open_TrianglePad1.0x1.5mm, symbol Jumper:Jumper_2_Open
- added R18: 10k, Resistor_SMD:R_0402_1005Metric, symbol Device:R
- added SW5: SW_SPDT, Slide_Switch:3P_SPDT_SlideSwitch, symbol Switch:SW_SPDT
- Q1, Q3, Q8, U2: footprint Package_TO_SOT_SMD:TO-252-3_TabPin2 -> Package_TO_SOT_SMD:TO-252-2
- Q4: renamed from Q?; footprint Package_TO_SOT_SMD:TO-252-3_TabPin2 -> Package_TO_SOT_SMD:TO-252-2
- U6: value STM32C031K4T6 -> STM32G030K6T6
- gave numbers to parts that had none: 14
Connections:
- net STLinkRX is gone; now on net MainTX1_STLinkRX: J3.9 (Pin_9)
- net STLinkTX is gone; now on net MainRX1_STLinkTX: J3.8 (Pin_8)
- net +3.3V: now also SW5.2 (B)
- net +5V: now also D9.2 (A)
- net DIP_SW0: now also U6.23 (PA12[PA10])
- net DIP_SW1: now also U6.27 (PB3)
- net DIP_SW2: now also U6.28 (PB4)
- net DIP_SW3: now also U6.29 (PB5)
- net DIP_SW4: now also U6.30 (PB6)
- net GND: now also C10.2, R18.2
- net LED0: now also U6.18 (PA8)
- net LED1: now also U6.22 (PA11[PA9])
- net LED2: now also U6.20 (PC6)
- net LEDPannel_L: now also U6.14 (PA7)
- net MainRX2_RS485TX: now also U6.26 (PA15)
- net MainTX2_RS485RX: now also U6.9 (PA2)
- net MonitorLED0: now also U6.17 (PB2)
- net NRST: now also U6.6 (PF2-NRST)
- net OSC_IN: now also U6.2 (PC14-OSCX_IN)
- net RS485_A: now also JP1.1 (A)
- net Slide_SW0: now also U6.31 (PB7)
- net TCK: now also U6.25 (PA14-BOOT0)
- net TMS: now also U6.24 (PA13)
- net VDD: now also C10.1, D13.1 (K)
- net V_Measure: now also U6.7 (PA0)
- net at C7.1, C8.1, L1.2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: now also D13.2 (A), D9.1 (K)
- net at D16.2 (DOUT): now also H1.1
- net at R46.1: now also JP1.2 (B)
- net MainTX1_STLinkRX: now reaches U6.19 (PA9)
- net MainRX1_STLinkTX: now reaches U6.21 (PA10)
- net Slide_SW1: now reaches U6.32 (PB8)
- net Slide_SW1: now also R18.1, SW5.1 (A)
- net 3.3VBUS: no longer names the net of J3.1 (Pin_1)
- no-connect marks 7 -> 16
Other:
- note removed: "Jumper"
- note removed: "パワースイッチ要らない？"
- moved on the sheet: C11, C14, C15, C16, C17, C18, C2, C21, C23, C25, C3, C4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

Commit message: 回路図プロット
Parts:
- added C22: 0.1uF, Capacitor_SMD:C_0402_1005Metric, symbol Device:C
Connections:
- net GND: now also C22.1
- net VDD: now also C22.2
Other:
- moved on the sheet: R17
Changed lines of the file:
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@@
   (junction (at 485.14 124.46) (diameter 0) (color 0 0 0 0)
   )
+  (junction (at 149.86 68.58) (diameter 0) (color 0 0 0 0)
+  )
   (junction (at 462.28 314.96) (diameter 0) (color 0 0 0 0)
   )
@@
   (junction (at 157.48 68.58) (diameter 0) (color 0 0 0 0)
   )
+  (junction (at 142.24 68.58) (diameter 0) (color 0 0 0 0)
+  )
   (junction (at 236.22 104.14) (diameter 0) (color 0 0 0 0)
   )
@@
   (junction (at 317.5 154.94) (diameter 0) (color 0 0 0 0)
   )
-  (junction (at 149.86 109.22) (diameter 0) (color 0 0 0 0)
+  (junction (at 142.24 109.22) (diameter 0) (color 0 0 0 0)
   )
   (junction (at 254 109.22) (diameter 0) (color 0 0 0 0)
@@
   (junction (at 261.62 279.4) (diameter 0) (color 0 0 0 0)
   )
-  (junction (at 149.86 68.58) (diameter 0) (color 0 0 0 0)
-  )
   (junction (at 297.18 88.9) (diameter 0) (color 0 0 0 0)
   )
@@
   (junction (at 279.4 170.18) (diameter 0) (color 0 0 0 0)
   )
+  (junction (at 149.86 109.22) (diameter 0) (color 0 0 0 0)
+  )
   (junction (at 195.58 68.58) (diameter 0) (color 0 0 0 0)
   )
@@
     (stroke (width 0) (type default) (color 0 0 0 0))
   )
-  (wire (pts (xy 144.78 66.04) (xy 144.78 68.58))
+  (wire (pts (xy 137.16 66.04) (xy 137.16 68.58))
     (stroke (width 0) (type default) (color 0 0 0 0))
   )
@@
     (stroke (width 0) (type default) (color 0 0 0 0))
   )
+  (wire (pts (xy 149.86 109.22) (xy 157.48 109.22))
+    (stroke (width 0) (type default) (color 0 0 0 0))
+  )
   (wire (pts (xy 172.72 86.36) (xy 180.34 86.36))
     (stroke (width 0) (type default) (color 0 0 0 0))
@@
     (stroke (width 0) (type default) (color 0 0 0 0))
   )
-  (wire (pts (xy 144.78 109.22) (xy 149.86 109.22))
+  (wire (pts (xy 137.16 109.22) (xy 142.24 109.22))
     (stroke (width 0) (type default) (color 0 0 0 0))
   )
@@
     (stroke (width 0) (type default) (color 0 0 0 0))
   )
-  (wire (pts (xy 149.86 92.71) (xy 149.86 109.22))
+  (wire (pts (xy 142.24 92.71) (xy 142.24 109.22))
     (stroke (width 0) (type default) (color 0 0 0 0))
   )
@@
     (stroke (width 0) (type default) (color 0 0 0 0))
   )
+  (wire (pts (xy 149.86 92.71) (xy 149.86 109.22))
+    (stroke (width 0) (type default) (color 0 0 0 0))
+  )
   (polyline (pts (xy 35.56 218.44) (xy 35.56 269.24))
     (stroke (width 0.5) (type solid) (color 0 0 0 0))
@@
     (stroke (width 0) (type default) (color 0 0 0 0))
   )
+  (wire (pts (xy 149.86 68.58) (xy 149.86 85.09))
+    (stroke (width 0) (type default) (color 0 0 0 0))
+  )
   (wire (pts (xy 287.02 100.33) (xy 287.02 104.14))
     (stroke (width 0) (type default) (color 0 0 0 0))
@@
     (stroke (width 0) (type default) (color 0 0 0 0))
   )
-  (wire (pts (xy 149.86 109.22) (xy 157.48 109.22))
+  (wire (pts (xy 142.24 109.22) (xy 149.86 109.22))
     (stroke (width 0) (type default) (color 0 0 0 0))
   )
@@
     (stroke (width 0) (type default) (color 0 0 0 0))
   )
-  (wire (pts (xy 149.86 68.58) (xy 149.86 85.09))
+  (wire (pts (xy 142.24 68.58) (xy 142.24 85.09))
     (stroke (width 0) (type default) (color 0 0 0 0))
   )
@@
     (stroke (width 0) (type default) (color 0 0 0 0))
   )
-  (wire (pts (xy 149.86 68.58) (xy 157.48 68.58))
-    (stroke (width 0) (type default) (color 0 0 0 0))
-  )
   (wire (pts (xy 195.58 73.66) (xy 196.85 73.66))
     (stroke (width 0) (type default) (color 0 0 0 0))
@@
     (stroke (width 0) (type default) (color 0 0 0 0))
   )
+  (wire (pts (xy 149.86 68.58) (xy 157.48 68.58))
+    (stroke (width 0) (type default) (color 0 0 0 0))
+  )
   (wire (pts (xy 113.03 309.88) (xy 116.84 309.88))
     (stroke (width 0) (type default) (color 0 0 0 0))
@@
     (stroke (width 0) (type default) (color 0 0 0 0))
   )
-  (wire (pts (xy 144.78 109.22) (xy 144.78 111.76))
+  (wire (pts (xy 137.16 109.22) (xy 137.16 111.76))
     (stroke (width 0) (type default) (color 0 0 0 0))
   )
@@
     (stroke (width 0) (type default) (color 0 0 0 0))
   )
-  (wire (pts (xy 144.78 68.58) (xy 149.86 68.58))
+  (wire (pts (xy 137.16 68.58) (xy 142.24 68.58))
     (stroke (width 0) (type default) (color 0 0 0 0))
   )
@@
     (stroke (width 0) (type default) (color 0 0 0 0))
   )
+  (wire (pts (xy 142.24 68.58) (xy 149.86 68.58))
+    (stroke (width 0) (type default) (color 0 0 0 0))
+  )
   (text "5V監視" (at 121.92 132.08 0)
     (effects (font (size 1.27 1.27)) (justify left bottom))
@@
     (pin "1")
   )
-  (symbol (lib_id "power:VDD") (at 144.78 66.04 0) (unit 1)
+  (symbol (lib_id "power:VDD") (at 137.16 66.04 0) (unit 1)
     (in_bom yes) (on_board yes) (fields_autoplaced)
-    (property "Reference" "#PWR011" (id 0) (at 144.78 69.85 0)
+    (property "Reference" "#PWR011" (id 0) (at 137.16 69.85 0)
       (effects (font (size 1.27 1.27)) hide)
     )
-    (property "Value" "VDD" (id 1) (at 144.78 60.96 0))
-    (property "Footprint" "" (id 2) (at 144.78 66.04 0)
+    (property "Value" "VDD" (id 1) (at 137.16 60.96 0))
+    (property "Footprint" "" (id 2) (at 137.16 66.04 0)
       (effects (font (size 1.27 1.27)) hide)
     )
-    (property "Datasheet" "" (id 3) (at 144.78 66.04 0)
+    (property "Datasheet" "" (id 3) (at 137.16 66.04 0)
       (effects (font (size 1.27 1.27)) hide)
     )
@@
     (pin "2")
   )
+  (symbol (lib_id "Device:C") (at 149.86 88.9 0) (mirror x) (unit 1)
+    (in_bom yes) (on_board yes)
+    (property "Reference" "C22" (id 0) (at 147.32 91.44 0)
+      (effects (font (size 1.27 1.27)) (justify left))
+    )
+    (property "Value" "0.1uF" (id 1) (at 144.78 93.98 0)
+      (effects (font (size 1.27 1.27)) (justify left))
+    )
+    (property "Footprint" "Capacitor_SMD:C_0402_1005Metric" (id 2) (at 150.8252 85.09 0)
+      (effects (font (size 1.27 1.27)) hide)
+    )
+    (property "Datasheet" "~" (id 3) (at 149.86 88.9 0)
+      (effects (font (size 1.27 1.27)) hide)
+    )
+    (pin "1")
+    (pin "2")
+  )
   (symbol (lib_id "Device:R") (at 86.36 147.32 0) (unit 1)
     (in_bom yes) (on_board yes) (fields_autoplaced)
@@
     (pin "4")
   )
-  (symbol (lib_id "power:GND") (at 144.78 111.76 0) (mirror y) (unit 1)
+  (symbol (lib_id "power:GND") (at 137.16 111.76 0) (mirror y) (unit 1)
     (in_bom yes) (on_board yes)
-    (property "Reference" "#PWR012" (id 0) (at 144.78 118.11 0)
+    (property "Reference" "#PWR012" (id 0) (at 137.16 118.11 0)
       (effects (font (size 1.27 1.27)) hide)
     )
-    (property "Value" "GND" (id 1) (at 144.653 116.1542 0))
-    (property "Footprint" "" (id 2) (at 144.78 111.76 0)
+    (property "Value" "GND" (id 1) (at 137.033 116.1542 0))
+    (property "Footprint" "" (id 2) (at 137.16 111.76 0)
       (effects (font (size 1.27 1.27)) hide)
     )
-    (property "Datasheet" "" (id 3) (at 144.78 111.76 0)
+    (property "Datasheet" "" (id 3) (at 137.16 111.76 0)
       (effects (font (size 1.27 1.27)) hide)
     )
@@
     (pin "1")
   )
-  (symbol (lib_id "Device:R") (at 149.86 88.9 0) (mirror y) (unit 1)
+  (symbol (lib_id "Device:R") (at 142.24 88.9 0) (mirror y) (unit 1)
     (in_bom yes) (on_board yes)
-    (property "Reference" "R17" (id 0) (at 149.86 88.9 90))
-    (property "Value" "1k" (id 1) (at 147.32 88.9 90))
-    (property "Footprint" "Resistor_SMD:R_0402_1005Metric" (id 2) (at 151.638 88.9 90)
+    (property "Reference" "R17" (id 0) (at 142.24 88.9 90))
+    (property "Value" "1k" (id 1) (at 139.7 88.9 90))
+    (property "Footprint" "Resistor_SMD:R_0402_1005Metric" (id 2) (at 144.018 88.9 90)
       (effects (font (size 1.27 1.27)) hide)
     )
-    (property "Datasheet" "~" (id 3) (at 149.86 88.9 0)
+    (property "Datasheet" "~" (id 3) (at 142.24 88.9 0)
       (effects (font (size 1.27 1.27)) hide)
     )
@@
       (reference "C21") (unit 1) (value "470uF") (footprint "Capacitor_SMD:C_Elec_8x10.2")
     )
+    (path "/45364e79-a3f3-4746-9c5f-7336d5074df1"
+      (reference "C22") (unit 1) (value "0.1uF") (footprint "Capacitor_SMD:C_0402_1005Metric")
+    )
     (path "/888c50eb-7f36-4dd1-9049-8f0b796c1bc2"

Commit message: 更新
Other:
- note added: "Panel"
- moved on the sheet: C1, C10, C11, C12, C13, C14, C15, C16, C17, C18, C19, C2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
