File: Panel/_autosave-Panel.kicad_sch (KiCad schematic)
At the start: 118 parts, among them J1 Conn_01x02_Male, J2 Conn_01x02_Female, J3 Conn_01x10_Male, J4 Conn_01x04_Male, J5 Conn_01x04_Male, Q1 MTP4835I3, Q14 S8050, Q15 BSS138, Q2 BSS138, Q3 MTP4835I3, Q5 2SC3265, Q8 MTP4835I3, SW1 SW_DIP_x05, SW2 SW_SPDT, SW3 SW_SPDT_White, SW4 SW_SPST, U1 MC34063AD, U2 AZ1084CD-3.3, U3 STM32G050F6P6, U4 MAX3485, U5 NJU6319AE, U6 STM32C031K4T6, Y1 16MHz

Commit message: DCDC回路図変更
Parts:
- removed U3: STM32G050F6P6, Package_SO:TSSOP-20_4.4x6.5mm_P0.65mm, symbol STM32C011F4P6:STM32C011F4P6
- removed U6: STM32C031K4T6, Package_QFP:LQFP-32_7x7mm_P0.8mm, symbol STM32C031K4T6:STM32C031K4T6
- added U?: STM32G030K6T6, Package_QFP:LQFP-32_7x7mm_P0.8mm, symbol STM32C031K4T6:STM32C031K4T6
Connections:
- net +3.3V: now also U?.4 (VDD/VDDA)
- net GND: now also U?.5 (VSS/VSSA)
- net LEDPannel_L: now also U?.14 (PA7)
- net NRST: now also U?.6 (PF2-NRST)
- net OSC_IN: now also U?.2 (PC14-OSCX_IN)
- net TCK: now also U?.25 (PA14-BOOT0)
- net TMS: now also U?.24 (PA13)
- no-connect marks 7 -> 6
