File: Panel/Panel.kicad_pcb (KiCad board)
At the start: 2 copper layers, 90 x 62 mm, 119 parts, among them J1 Conn_01x02_Male, J2 Conn_01x02_Female, J3 Conn_01x10_Male, J4 Conn_01x04_Male, J5 Conn_01x04_Male, Q1 MTP4835I3, Q14 S8050, Q15 BSS138, Q2 BSS138, Q3 MTP4835I3, Q4 MTP4835I3, Q5 2SC3265, Q8 MTP4835I3, SW1 SW_DIP_x05, SW2 SW_SPDT, SW3 SW_SPDT_White, SW4 SW_SPST, SW5 SW_SPDT, U1 MC34063AD, U2 AZ1084CD-3.3, U3 M51957B, U4 MAX3485, U5 NJU6319AE, U6 STM32G030K6T6, Y1 16MHz

Commit message: 回路図プロット
Parts:
- added C22: 0.1uF, Capacitor_SMD:C_0402_1005Metric, F.Cu at (-12.3, 10.5)
- moved TP4 5.01 mm to (-37.2, -19.2)
- moved C21 1.15 mm to (16.3, -4.02)
- moved C19 0.95 mm to (16.7, -22.6), turned to 0 degrees
- moved TP1 0.35 mm to (-15.2, 6.78)
- moved C10 0.12 mm to (-14.0, 10.6)
- moved C11 0.12 mm to (-15.2, 13.1)
- moved R19 0.12 mm to (-16.0, 10.6)
Routing:
- net GND: track 0.00 -> 215.2 mm, vias 0 -> 339
- net +3.3V: track 189.7 -> 185.7 mm
- net Net-(U5-Pad3): track 8.09 -> 7.36 mm

Commit message: Pole,Panelほぼ完成
Parts:
- C23, R24: moved to F.Cu
- moved R24 7.00 mm to (-0.86, 10.9)
- moved C23 6.82 mm to (-2.80, 10.9), turned to 90 degrees
- moved C11 0.51 mm to (-15.8, 13.2)
- moved R19 0.51 mm to (-16.5, 10.7)
- moved C10 0.51 mm to (-14.5, 10.7)
- moved C22 0.50 mm to (-12.8, 10.4)
- moved D8 0.50 mm to (-5.16, 10.9)
- moved C8 0.31 mm to (8.04, 19.4)
- moved L1 0.30 mm to (5.32, 5.56)
- moved C25 0.25 mm to (4.00, 13.8)
- moved C7 0.25 mm to (7.05, 11.8)
- moved R37 0.25 mm to (7.00, 13.8)
Routing:
- net GND: track 215.2 -> 226.1 mm, vias 339 -> 820
- net Net-(D8-Pad2): track 2.10 -> 0.00 mm
- net Net-(C23-Pad2): track 1.77 -> 2.60 mm

Commit message: Mother_Ctrl回路図プロット
Changed lines of the file:
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@@
       (effects (font (size 1 1) (thickness 0.15)))
     )
-    (fp_text user "1" (at -4.15 -1.6 90) (layer "F.SilkS")
+    (fp_text user "1" (at -2.48 -3.8 90) (layer "F.SilkS")
       (effects (font (size 1 1) (thickness 0.15)))
     )

Commit message: 多分完成
Parts:
- moved C1 162.4 mm to (113.2, 91.3)
- moved C11 162.4 mm to (125.2, 93.8)
- moved C12 162.4 mm to (105.2, 76.8)
- moved C13 162.4 mm to (105.2, 75.2)
- moved C14 162.4 mm to (141.1, 56.1)
- moved C15 162.4 mm to (135.7, 54.9)
- moved C16 162.4 mm to (124.2, 79.1)
- moved C17 162.4 mm to (148.2, 61.0)
- moved C18 162.4 mm to (124.5, 58.8)
- moved C19 162.4 mm to (157.7, 57.9)
- moved C2 162.4 mm to (138.5, 77.7)
- moved C20 162.4 mm to (93.0, 61.9)
- moved C21 162.4 mm to (157.3, 76.5)
- moved C23 162.4 mm to (138.2, 91.5)
- moved C25 162.4 mm to (145.0, 94.4)
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Other:
- board text added: "+5V"
- board text added: "3.3V"
- board text added: "DIN"
- board text added: "DOUT"
- board text added: "Designed by @cat_nekonekone"
- board text added: "GND"
- board text added: "JLCJLCJLCJLC"
- board text added: "NRST"
- board text added: "PA11"
- board text added: "PA12"
- board text added: "PA8"
- board text added: "PB2"
- board text added: "PB3"
- board text added: "PB4"
- board text added: "PB5"
- board text added: "PB6"
- board text added: "PB7"
- board text added: "PB8"
- board text added: "PC6"
- board text added: "POWER"
- board text added: "RX1:PA10"
- board text added: "RX2:PA15"
- board text added: "TX1:PA9"
- board text added: "TX2:PA2"
- board text added: "Tomoshibi"
- board text added: "VCC"
- board text added: "[RS485]"
- board text added: "[STLink]"
- board text added: "燈"
