File: SmallMD/SmallMD.kicad_sch (KiCad schematic)
At the start: 150 parts, among them J1 Conn_01x02_Male, J3 Conn_01x10_Male, J4 Conn_01x02_Female, J5 Conn_01x04_Male, J6 Conn_01x04_Male, J7 Conn_01x10_Male, J8 Conn_01x06_Male, Q1 SSM6J808R, Q14 BSS138, Q15 BSS138, Q16 S8050, Q18 μPA2753GR, Q19 μPA2753GR, Q2 BSS138, Q3 SSM6J808R, SW1 SW_DIP_x05, SW2 SW_SPDT, SW3 SW_SPDT_White, SW4 SW_SPST, U1 AZ1084CD-3.3, U10 IR2302, U11 IR2302, U12 MAX3485, U13 NJU6319AE, U2 AZ1084CD-5.0, U3 STM32G030K6T6, U4 MAX3485, U5 MAX3485, U6 LT6106, U7 MAX3485, U8 TLP2361, U9 TLP2361, Y1 16MHz

Commit message: SmallMDほぼ完成
Parts:
- removed H5, H7, H9: MountingHole, MountingHole:MountingHole_3.2mm_M3, symbol Mechanical:MountingHole
- removed TP1, TP2, TP3, TP4: TestPoint, TestPoint:TestPoint_THTPad_D2.0mm_Drill1.0mm, symbol Connector:TestPoint
Connections:
- net Current_Sence: now also U3.23 (PA12[PA10])
- net DIP_SW0: now also U3.8 (PA1)
- net DIP_SW1: now also U3.29 (PB5)
- net DIP_SW2: now also U3.31 (PB7)
- net DIP_SW3: now also U3.32 (PB8)
- net DIP_SW4: now also U3.1 (PB9)
- net LED0: now also U3.12 (PA5)
- net LED1: now also U3.15 (PB0)
- net LED2: now also U3.16 (PB1)
- net Maxon_I: now also U3.27 (PB3)
- net MonitorLED0: now also U3.11 (PA4)
- net PWM_B: now also U3.30 (PB6)
- net SHDN: now also U3.28 (PB4)
- net Slide_SW0: now also U3.7 (PA0)
- net V_Measure: now also U3.22 (PA11[PA9])
- no-connect marks 9 -> 12
Other:
- note removed: "ねじ穴"
