File: SmallPW/SmallPW.kicad_sch (KiCad schematic)
At the start: 47 parts

Commit message: 定期更新
Parts:
- removed C?: 10uF, Capacitor_SMD:C_0805_2012Metric_Pad1.18x1.45mm_HandSolder, symbol Device:C
- removed C?: 4.7uF, Capacitor_SMD:C_0805_2012Metric_Pad1.18x1.45mm_HandSolder, symbol Device:C
- removed C?: 22uF, Capacitor_SMD:C_1210_3225Metric_Pad1.33x2.70mm_HandSolder, symbol Device:C
- removed D? (x2): D, Diode_SMD:D_SOD-123, symbol Device:D
- removed D?: WS2812B, LED_SMD:LED_WS2812B_PLCC4_5.0x5.0mm_P3.2mm, symbol LED:WS2812B
- removed H? (x4): MountingHole_Pad, TestPoint:TestPoint_THTPad_D3.0mm_Drill1.5mm, symbol Mechanical:MountingHole_Pad
- removed J? (x3): Conn_01x02_Female, Connector_AMASS:AMASS_XT30PW-M_1x02_P2.50mm_Horizontal, symbol Connector:Conn_01x02_Female
- removed J? (x2): Conn_01x02_Female, Connector_Molex:Molex_SPOX_5268-02A_1x02_P2.50mm_Horizontal, symbol Connector:Conn_01x02_Female
- removed MD?: OKL-T/6-W12N-C, DCDC_Regulator:MURATA_OKL-T-6-W12N-C, symbol DCDC_Regulator:OKL-T/6-W12N-C
- removed Q?: Q_NMOS_GSD, Package_TO_SOT_SMD:SOT-23_Handsoldering, symbol Device:Q_NMOS_GSD
- removed Q? (x4): Q_PMOS_GDS, Package_TO_SOT_SMD:TO-252-3_TabPin2, symbol Device:Q_PMOS_GDS
- removed R? (x2): 1k, Resistor_SMD:R_0603_1608Metric_Pad0.98x0.95mm_HandSolder, symbol Device:R
- removed R?: 100k, Resistor_SMD:R_0603_1608Metric_Pad0.98x0.95mm_HandSolder, symbol Device:R
- removed R?: 1.2k, Resistor_SMD:R_0603_1608Metric_Pad0.98x0.95mm_HandSolder, symbol Device:R
- removed R? (x3): 10k, Resistor_SMD:R_0603_1608Metric_Pad0.98x0.95mm_HandSolder, symbol Device:R
- removed R?: 10, Resistor_SMD:R_0603_1608Metric_Pad0.98x0.95mm_HandSolder, symbol Device:R
- removed R?: 330, Resistor_SMD:R_0603_1608Metric_Pad0.98x0.95mm_HandSolder, symbol Device:R
- removed R? (x2): 510, Resistor_SMD:R_0603_1608Metric_Pad0.98x0.95mm_HandSolder, symbol Device:R
- removed SW?: SW_SPDT, Slide_Switch:3P_SPDT_SlideSwitch, symbol Switch:SW_SPDT
- added C1: 1uF, Capacitor_SMD:C_0402_1005Metric, symbol Device:C
- added C3: 22uF, Capacitor_SMD:C_0805_2012Metric, symbol Device:C
- added C4: 10uF, Capacitor_SMD:C_0805_2012Metric, symbol Device:C
- added D1, D2: SBR1A40SA, Diode_SMD:D_SMA_Handsoldering, symbol Device:D_Schottky
- added J1: Conn_01x02_Male, Connector_AMASS:AMASS_XT30PW-M_1x02_P2.50mm_Horizontal, symbol Connector:Conn_01x02_Male
- added MD1: OKL-T/6-W12N-C, DCDC_Regulator:MURATA_OKL-T-6-W12N-C, symbol DCDC_Regulator:OKL-T/6-W12N-C
- added Q1, Q3: MTP4835I3, Package_TO_SOT_SMD:TO-252-3_TabPin2, symbol Device:Q_PMOS_GDS
- added Q2: BSS138, Package_TO_SOT_SMD:SOT-23, symbol Device:Q_NMOS_GSD
- added R1, R3, R4: 10k, Resistor_SMD:R_0402_1005Metric, symbol Device:R
- added R10: 1.2k, Resistor_SMD:R_0402_1005Metric, symbol Device:R
- added R2, R6: 100k, Resistor_SMD:R_0402_1005Metric, symbol Device:R
- added R7: 1k, Resistor_SMD:R_0402_1005Metric, symbol Device:R
- added R8: 330, Resistor_SMD:R_0402_1005Metric, symbol Device:R
- added R9: 10, Resistor_SMD:R_0402_1005Metric, symbol Device:R
- J2, J3, J4: renamed from J?; footprint Connector_AMASS:AMASS_XT30PW-M_1x02_P2.50mm_Horizontal -> Connector_AMASS:AMASS_XT30PW-F_1x02_P2.50mm_Horizontal
- gave numbers to parts that had none: 11
Connections:
- net DIN is gone; now on net +5V: J6.2 (Pin_2), J7.2 (Pin_2)
- net +5V: now also C4.1, D1.2 (A), MD1.4 (VOUT), MD1.5 (SENSE), R10.2, R6.2
- net GND: now also C3.2, C4.2, D2.2 (A), J1.1 (Pin_1), MD1.1 (ON/OFF), MD1.3 (GND), MD1.7 (GND), Q1.1 (G), Q2.2 (S), R1.2, R10.1, R4.2, R9.2
- net S-S: now also C1.1, Q1.3 (S), Q3.3 (S), R1.1, R2.1
- net VDD: now also C3.1, D1.1 (K), D2.1 (K), MD1.2 (VIN), Q3.2 (D), R4.1
- net 主電源スイッチ: now also C1.2, Q3.1 (G), R2.2, R3.1
- net at R5.1, SW1.1 (A): now also Q2.1 (G)
- net at F1.2: now also Q1.2 (D)
- net +12V renamed 12VBAT
- net 12VBAT: now also J1.2 (Pin_2)
- new net: R8.1, R9.1
- new net: Q2.3 (D), R3.2
- new net: R7.2, R8.2
- new net: MD1.10 (PGOOD), R6.1
- new net: MD1.6 (TRIM), R7.1
- no-connect marks 5 -> 4
Other:
- note removed: "5V生成"
- note removed: "Board LED"
- note removed: "Conn to Display"
- note removed: "Power Conn"
- note removed: "Signal Conn"
- moved on the sheet: C2, F1, J2, J3, J4, J6, J7, MES1

Commit message: 進捗
Parts:
- removed C3: 22uF, Capacitor_SMD:C_0805_2012Metric, symbol Device:C
- removed C4: 10uF, Capacitor_SMD:C_0805_2012Metric, symbol Device:C
- removed D1: SBR1A40SA, Diode_SMD:D_SMA_Handsoldering, symbol Device:D_Schottky
- removed J6, J7: Conn_01x02_Female, Connector_Molex:Molex_SPOX_5268-02A_1x02_P2.50mm_Horizontal, symbol Connector:Conn_01x02_Female
- removed MD1: OKL-T/6-W12N-C, DCDC_Regulator:MURATA_OKL-T-6-W12N-C, symbol DCDC_Regulator:OKL-T/6-W12N-C
- removed R10: 1.2k, Resistor_SMD:R_0402_1005Metric, symbol Device:R
- removed R4: 10k, Resistor_SMD:R_0402_1005Metric, symbol Device:R
- removed R6: 100k, Resistor_SMD:R_0402_1005Metric, symbol Device:R
- removed R7: 1k, Resistor_SMD:R_0402_1005Metric, symbol Device:R
- removed R8: 330, Resistor_SMD:R_0402_1005Metric, symbol Device:R
- removed R9: 10, Resistor_SMD:R_0402_1005Metric, symbol Device:R
- added J5: Conn_01x02_Female, Connector_AMASS:AMASS_XT30U-F_1x02_P5.0mm_Vertical, symbol Connector:Conn_01x02_Female
- D2: value SBR1A40SA -> 1N5819WS; footprint Diode_SMD:D_SMA_Handsoldering -> Diode_SMD:D_SOD-323_HandSoldering
- J1: footprint Connector_AMASS:AMASS_XT30PW-M_1x02_P2.50mm_Horizontal -> Connector_AMASS:AMASS_XT30U-M_1x02_P5.0mm_Vertical
- J2, J3, J4: footprint Connector_AMASS:AMASS_XT30PW-F_1x02_P2.50mm_Horizontal -> Connector_AMASS:AMASS_XT30U-F_1x02_P5.0mm_Vertical
Connections:
- net GND: now also J5.1 (Pin_1)
- net VDD: now also J5.2 (Pin_2)
- no-connect marks 4 -> 0
Other:
- note added: "Conn to Board"
- note removed: "Conn to CircuitBoard"
- moved on the sheet: J2, J3, J4

Commit message: LargeMDほぼ完成
Parts:
- removed H1, H2, H3, H4: MountingHole, MountingHole:MountingHole_3.2mm_M3, symbol Mechanical:MountingHole
Other:
- note removed: "ねじ穴"
Changed lines of the file:
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@@
     (stroke (width 0) (type default) (color 0 0 0 0))
-  )
-  (polyline (pts (xy 116.84 154.94) (xy 116.84 187.96))
-    (stroke (width 0.5) (type solid) (color 0 0 0 0))
   )
   (wire (pts (xy 121.92 50.8) (xy 127 50.8))
     (stroke (width 0) (type default) (color 0 0 0 0))
-  )
-  (polyline (pts (xy 162.56 187.96) (xy 162.56 154.94))
-    (stroke (width 0.5) (type solid) (color 0 0 0 0))
   )
   (wire (pts (xy 109.22 83.82) (xy 109.22 90.17))
@@
     (stroke (width 0) (type default) (color 0 0 0 0))
   )
-  (polyline (pts (xy 116.84 154.94) (xy 162.56 154.94))
-    (stroke (width 0.5) (type solid) (color 0 0 0 0))
-  )
   (wire (pts (xy 86.36 83.82) (xy 93.98 83.82))
     (stroke (width 0) (type default) (color 0 0 0 0))
@@
     (stroke (width 0) (type default) (color 0 0 0 0))
   )
-  (polyline (pts (xy 116.84 187.96) (xy 162.56 187.96))
-    (stroke (width 0.5) (type solid) (color 0 0 0 0))
-  )
   (wire (pts (xy 132.08 81.28) (xy 132.08 83.82))
     (stroke (width 0) (type default) (color 0 0 0 0))
@@
   (text "電源" (at 38.1 22.86 0)
     (effects (font (size 2.54 2.54)) (justify left bottom))
-  )
-  (text "ねじ穴" (at 119.38 152.4 0)
-    (effects (font (size 2.54 2.54) (thickness 0.508) bold) (justify left bottom))
   )
   (label "12VBAT" (at 60.96 50.8 0)
@@
     )
   )
-  (symbol (lib_id "Mechanical:MountingHole") (at 124.46 165.1 0) (unit 1)
-    (in_bom yes) (on_board yes) (fields_autoplaced)
-    (property "Reference" "H1" (id 0) (at 127 163.8299 0)
-      (effects (font (size 1.27 1.27)) (justify left))
-    )
-    (property "Value" "MountingHole" (id 1) (at 127 166.3699 0)
-      (effects (font (size 1.27 1.27)) (justify left))
-    )
-    (property "Footprint" "MountingHole:MountingHole_3.2mm_M3" (id 2) (at 124.46 165.1 0)
-      (effects (font (size 1.27 1.27)) hide)
-    )
-    (property "Datasheet" "~" (id 3) (at 124.46 165.1 0)
-      (effects (font (size 1.27 1.27)) hide)
-    )
-  )
   (symbol (lib_id "power:VDD") (at 160.02 96.52 0) (mirror y) (unit 1)
     (in_bom yes) (on_board yes) (fields_autoplaced)
@@
     (pin "3")
   )
-  (symbol (lib_id "Mechanical:MountingHole") (at 144.78 180.34 0) (unit 1)
-    (in_bom yes) (on_board yes) (fields_autoplaced)
-    (property "Reference" "H4" (id 0) (at 147.32 179.0699 0)
-      (effects (font (size 1.27 1.27)) (justify left))
-    )
-    (property "Value" "MountingHole" (id 1) (at 147.32 181.6099 0)
-      (effects (font (size 1.27 1.27)) (justify left))
-    )
-    (property "Footprint" "MountingHole:MountingHole_3.2mm_M3" (id 2) (at 144.78 180.34 0)
-      (effects (font (size 1.27 1.27)) hide)
-    )
-    (property "Datasheet" "~" (id 3) (at 144.78 180.34 0)
-      (effects (font (size 1.27 1.27)) hide)
-    )
-  )
   (symbol (lib_id "power:VDD") (at 132.08 81.28 0) (unit 1)
     (in_bom yes) (on_board yes) (fields_autoplaced)
@@
     (pin "1")
   )
-  (symbol (lib_id "Mechanical:MountingHole") (at 144.78 165.1 0) (unit 1)
-    (in_bom yes) (on_board yes) (fields_autoplaced)
-    (property "Reference" "H3" (id 0) (at 147.32 163.8299 0)
-      (effects (font (size 1.27 1.27)) (justify left))
-    )
-    (property "Value" "MountingHole" (id 1) (at 147.32 166.3699 0)
-      (effects (font (size 1.27 1.27)) (justify left))
-    )
-    (property "Footprint" "MountingHole:MountingHole_3.2mm_M3" (id 2) (at 144.78 165.1 0)
-      (effects (font (size 1.27 1.27)) hide)
-    )
-    (property "Datasheet" "~" (id 3) (at 144.78 165.1 0)
-      (effects (font (size 1.27 1.27)) hide)
-    )
-  )
   (symbol (lib_id "power:GND") (at 162.56 93.98 0) (mirror y) (unit 1)
     (in_bom yes) (on_board yes) (fields_autoplaced)
@@
     (pin "3")
   )
-  (symbol (lib_id "Mechanical:MountingHole") (at 124.46 180.34 0) (unit 1)
-    (in_bom yes) (on_board yes) (fields_autoplaced)
-    (property "Reference" "H2" (id 0) (at 127 179.0699 0)
-      (effects (font (size 1.27 1.27)) (justify left))
-    )
-    (property "Value" "MountingHole" (id 1) (at 127 181.6099 0)
-      (effects (font (size 1.27 1.27)) (justify left))
-    )
-    (property "Footprint" "MountingHole:MountingHole_3.2mm_M3" (id 2) (at 124.46 180.34 0)
-      (effects (font (size 1.27 1.27)) hide)
-    )
-    (property "Datasheet" "~" (id 3) (at 124.46 180.34 0)
-      (effects (font (size 1.27 1.27)) hide)
-    )
-  )
   (symbol (lib_id "power:GND") (at 58.42 48.26 0) (unit 1)
     (in_bom yes) (on_board yes) (fields_autoplaced)
@@
       (reference "F1") (unit 1) (value "Fuse") (footprint "Fuse:Fuseholder_Blade_Mini_Keystone_3568")
     )
-    (path "/0181a6e1-7c54-468e-8392-dacac2eae964"
-      (reference "H1") (unit 1) (value "MountingHole") (footprint "MountingHole:MountingHole_3.2mm_M3")
-    )
-    (path "/c0ac9d52-cacf-4d7a-bafe-e1b7637dd8f0"
-      (reference "H2") (unit 1) (value "MountingHole") (footprint "MountingHole:MountingHole_3.2mm_M3")
-    )
-    (path "/9e6543ef-7fe2-44ed-9f4c-679153033295"
-      (reference "H3") (unit 1) (value "MountingHole") (footprint "MountingHole:MountingHole_3.2mm_M3")
-    )
-    (path "/69320ecc-187c-4ab1-a856-35f68df4362d"
-      (reference "H4") (unit 1) (value "MountingHole") (footprint "MountingHole:MountingHole_3.2mm_M3")
-    )
     (path "/0ec49e2a-601b-4b21-9f6a-1a36f6a4d7e1"

Commit message: SmallMDほぼ完成
Parts:
- C1: footprint Capacitor_SMD:C_0402_1005Metric -> Capacitor_SMD:C_0603_1608Metric_Pad1.08x0.95mm_HandSolder
- R1, R2, R3: footprint Resistor_SMD:R_0402_1005Metric -> Resistor_SMD:R_0603_1608Metric_Pad0.98x0.95mm_HandSolder
Changed lines of the file:
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@@
     (property "Reference" "R3" (id 0) (at 101.6 44.45 90))
     (property "Value" "10k" (id 1) (at 101.6 46.99 90))
-    (property "Footprint" "Resistor_SMD:R_0402_1005Metric" (id 2) (at 101.6 52.578 90)
+    (property "Footprint" "Resistor_SMD:R_0603_1608Metric_Pad0.98x0.95mm_HandSolder" (id 2) (at 101.6 52.578 90)
       (effects (font (size 1.27 1.27)) hide)
     )
@@
       (effects (font (size 1.27 1.27)) (justify left))
     )
-    (property "Footprint" "Capacitor_SMD:C_0402_1005Metric" (id 2) (at 87.3252 92.71 0)
+    (property "Footprint" "Capacitor_SMD:C_0603_1608Metric_Pad1.08x0.95mm_HandSolder" (id 2) (at 87.3252 92.71 0)
       (effects (font (size 1.27 1.27)) hide)
     )
@@
       (effects (font (size 1.27 1.27)) (justify left))
     )
-    (property "Footprint" "Resistor_SMD:R_0402_1005Metric" (id 2) (at 92.202 88.9 90)
+    (property "Footprint" "Resistor_SMD:R_0603_1608Metric_Pad0.98x0.95mm_HandSolder" (id 2) (at 92.202 88.9 90)
       (effects (font (size 1.27 1.27)) hide)
     )
@@
       (effects (font (size 1.27 1.27)) (justify left))
     )
-    (property "Footprint" "Resistor_SMD:R_0402_1005Metric" (id 2) (at 76.962 91.44 90)
+    (property "Footprint" "Resistor_SMD:R_0603_1608Metric_Pad0.98x0.95mm_HandSolder" (id 2) (at 76.962 91.44 90)
       (effects (font (size 1.27 1.27)) hide)
     )
@@
     )
     (path "/36199e68-1997-47ca-b44b-443b1e5b373a"
-      (reference "C1") (unit 1) (value "1uF") (footprint "Capacitor_SMD:C_0402_1005Metric")
+      (reference "C1") (unit 1) (value "1uF") (footprint "Capacitor_SMD:C_0603_1608Metric_Pad1.08x0.95mm_HandSolder")
     )
     (path "/4e904d34-ca0d-4bde-a434-7a3eb283f0ad"
@@
     )
     (path "/a5ae3b0f-96e9-44a3-8eb1-2bb525e38212"
-      (reference "R1") (unit 1) (value "10k") (footprint "Resistor_SMD:R_0402_1005Metric")
+      (reference "R1") (unit 1) (value "10k") (footprint "Resistor_SMD:R_0603_1608Metric_Pad0.98x0.95mm_HandSolder")
     )
     (path "/849008c9-d3e4-4de1-8473-8517407231bc"
-      (reference "R2") (unit 1) (value "100k") (footprint "Resistor_SMD:R_0402_1005Metric")
+      (reference "R2") (unit 1) (value "100k") (footprint "Resistor_SMD:R_0603_1608Metric_Pad0.98x0.95mm_HandSolder")
     )
     (path "/315d8b9c-409b-409b-a05b-fd3ab84fd3a7"
-      (reference "R3") (unit 1) (value "10k") (footprint "Resistor_SMD:R_0402_1005Metric")
+      (reference "R3") (unit 1) (value "10k") (footprint "Resistor_SMD:R_0603_1608Metric_Pad0.98x0.95mm_HandSolder")
     )
     (path "/55d20af3-1852-4bff-a90f-7672e4877e8e"
