File: SmallPW/SmallPW.kicad_pcb (KiCad board)
At the start: 2 copper layers, 28.3 x 11 mm, 33 parts, among them J1 Conn_01x02_Male, J2 Conn_01x02_Female, J3 Conn_01x02_Female, J4 Conn_01x02_Female, J6 Conn_01x02_Female, J7 Conn_01x02_Female, Q1 MTP4835I3, Q2 BSS138, Q3 MTP4835I3, SW1 SW_SPST

Commit message: 進捗
Parts:
- removed C3: 22uF, Capacitor_SMD:C_0805_2012Metric
- removed C4: 10uF, Capacitor_SMD:C_0805_2012Metric
- removed D1: SBR1A40SA, Diode_SMD:D_SMA_Handsoldering
- removed J6, J7: Conn_01x02_Female, Connector_Molex:Molex_SPOX_5268-02A_1x02_P2.50mm_Horizontal
- removed MD1: OKL-T/6-W12N-C, DCDC_Regulator:MURATA_OKL-T-6-W12N-C
- removed R10: 1.2k, Resistor_SMD:R_0402_1005Metric
- removed R4: 10k, Resistor_SMD:R_0402_1005Metric
- removed R6: 100k, Resistor_SMD:R_0402_1005Metric
- removed R7: 1k, Resistor_SMD:R_0402_1005Metric
- removed R8: 330, Resistor_SMD:R_0402_1005Metric
- removed R9: 10, Resistor_SMD:R_0402_1005Metric
- added J5: Conn_01x02_Female, Connector_AMASS:AMASS_XT30U-F_1x02_P5.0mm_Vertical, F.Cu at (61.5, 5.00)
- D2: value SBR1A40SA -> 1N5819WS; footprint Diode_SMD:D_SMA_Handsoldering -> Diode_SMD:D_SOD-323_HandSoldering
- J1: footprint Connector_AMASS:AMASS_XT30PW-M_1x02_P2.50mm_Horizontal -> Connector_AMASS:AMASS_XT30U-M_1x02_P5.0mm_Vertical
- J2, J3, J4: footprint Connector_AMASS:AMASS_XT30PW-F_1x02_P2.50mm_Horizontal -> Connector_AMASS:AMASS_XT30U-F_1x02_P5.0mm_Vertical
- moved H4 170.2 mm to (5.00, 5.00)
- moved H1 146.2 mm to (5.00, 35.0)
- moved H3 129.2 mm to (71.0, 5.00)
- moved H2 105.6 mm to (71.0, 35.0)
- moved Q2 71.5 mm to (29.0, 46.0)
- moved R3 66.8 mm to (49.3, 47.5)
- moved R5 66.8 mm to (40.6, 45.0)
- moved D2 64.8 mm to (44.7, 23.0), turned to 180 degrees
- moved J1 63.3 mm to (5.00, 19.0)
- moved SW1 60.6 mm to (66.0, 20.0)
- moved F1 42.1 mm to (13.3, 28.0), turned to 90 degrees
- moved C2 28.1 mm to (52.0, 18.0), turned to -90 degrees
- moved Q1 21.0 mm to (25.4, 17.5), turned to 90 degrees
- moved MES1 20.0 mm to (38.0, 31.3)
- moved J4 19.6 mm to (47.5, 5.00), turned to 180 degrees
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Other:
- outline, holes or cut-outs redrawn

Commit message: LargeMDほぼ完成
Parts:
- removed H1, H2, H3, H4: MountingHole, MountingHole:MountingHole_3.2mm_M3
- moved C2 40.3 mm to (52.0, -22.3)
- moved D2 40.3 mm to (44.7, -17.3)
- moved F1 40.3 mm to (13.3, -12.3)
- moved J1 40.3 mm to (5.00, -21.3)
- moved J2 40.3 mm to (19.5, -35.3)
- moved J3 40.3 mm to (33.5, -35.3)
- moved J4 40.3 mm to (47.5, -35.3)
- moved J5 40.3 mm to (61.5, -35.3)
- moved MES1 40.3 mm to (38.0, -9.00)
- moved Q1 40.3 mm to (25.4, -22.8)
- moved Q3 40.3 mm to (38.2, -23.0)
- moved SW1 40.3 mm to (66.0, -20.3)
Other:
- board size 28.3 x 11 mm -> 76 x 40 mm

Commit message: SmallMDほぼ完成
Parts:
- C1: footprint Capacitor_SMD:C_0402_1005Metric -> Capacitor_SMD:C_0603_1608Metric_Pad1.08x0.95mm_HandSolder; moved to B.Cu
- D2, Q2, R5: moved to B.Cu
- R1, R2, R3: footprint Resistor_SMD:R_0402_1005Metric -> Resistor_SMD:R_0603_1608Metric_Pad0.98x0.95mm_HandSolder; moved to B.Cu
- moved J1 129.3 mm to (98.5, 68.0)
- moved D2 128.9 mm to (143.8, 65.0), turned to -90 degrees
- moved Q1 128.7 mm to (118.9, 65.5)
- moved J2 127.9 mm to (113.0, 52.0)
- moved J3 127.9 mm to (127.0, 52.0)
- moved J4 127.9 mm to (141.0, 52.0)
- moved J5 127.9 mm to (155.0, 52.0)
- moved MES1 127.9 mm to (131.5, 78.3)
- moved Q2 127.8 mm to (154.5, 70.0), turned to 90 degrees
- moved SW1 127.6 mm to (159.0, 67.0)
- moved Q3 127.4 mm to (131.0, 64.3)
- moved C2 126.7 mm to (143.8, 65.0)
- moved F1 126.2 mm to (106.8, 72.4)
- moved R5 117.2 mm to (154.5, 72.8), turned to 180 degrees
- moved R3 107.0 mm to (154.5, 67.3), turned to 180 degrees
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Routing:
- net GND: track 0.00 -> 76.0 mm, vias 0 -> 189
- net /S-S: track 0.00 -> 38.2 mm, vias 0 -> 41
- net 主電源スイッチ: track 0.00 -> 36.4 mm, vias 0 -> 1
- net VDD: track 0.00 -> 34.5 mm, vias 0 -> 1
- net Net-(Q2-Pad1): track 0.00 -> 5.50 mm
- net Net-(F1-Pad2): track 0.00 -> 3.40 mm
- net Net-(Q2-Pad3): track 0.00 -> 2.19 mm
- net /12VBAT: vias 0 -> 108
- added copper zone on B.Cu, net /12VBAT
- added copper zone on F.Cu, net /12VBAT
- added copper zone on B.Cu, net /S-S
- added copper zone on F.Cu, net /S-S
- added copper zone on B.Cu, net GND
- added copper zone on F.Cu, net GND
- added copper zone on F.Cu, net Net-(F1-Pad2)
- added copper zone on F.Cu, net VDD
Other:
- board text added: "BAT"
- board text added: "Board"
- board text added: "Conn to"
- board text added: "Designed by @cat_nekonekone"
- board text added: "Tomoshibi"
- board text added: "燈"

Commit message: 製造ファイル出力
Other:
- board text added: "JLCJLCJLCJLC"
Changed lines of the file:
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@@
     (effects (font (size 1.1 1.1) (thickness 0.15) italic))
+  )
+  (gr_text "JLCJLCJLCJLC" (at 158.8 64.3) (layer "F.SilkS")
+    (effects (font (size 1 1) (thickness 0.15)))
   )
   (gr_text "BAT" (at 98.75 61) (layer "F.SilkS")
@@
   )
   (gr_text "Tomoshibi" (at 108.87 84.5) (layer "F.SilkS")
-    (effects (font (size 1.4 1.4) (thickness 0.19)))
+    (effects (font (size 1.4 1.4) (thickness 0.17)))
   )
   (gr_text "Designed by\n@cat_nekonekone" (at 154 82.25) (layer "F.SilkS")
-    (effects (font (size 0.9 0.9) (thickness 0.13)))
+    (effects (font (size 1 1) (thickness 0.13)))
   )
   (segment (start 154.680339 66.260339) (end 156.67 68.25) (width 0.25) (layer "F.Cu") (net 1))
