File: Pole/Pole.kicad_sch (KiCad schematic)
At the start: 169 parts

Commit message: 構成図追加
Parts:
- removed C? (x2): 4.7uF, Capacitor_SMD:C_0603_1608Metric, symbol Device:C
- added C2, C8: 10uF, Capacitor_SMD:C_0805_2012Metric_Pad1.18x1.45mm_HandSolder, symbol Device:C
- D9: renamed from D?; value MA10EB045 -> ?; footprint Diode_Schottky:DO-221BC -> (none)
- L1: renamed from L?; footprint (none) -> Inductor_Power:ETQ-P4M_KVK
- Q11, Q13, Q15, Q17, Q6: renamed from Q?; value 2PB709AR -> S8050; footprint Package_TO_SOT_SMD:SC-59_Handsoldering -> Package_TO_SOT_SMD:SOT-23
- Q5: renamed from Q?; footprint Package_TO_SOT_SMD:SC-59_Handsoldering -> Package_TO_SOT_SMD:SOT-23
- RV1: renamed from RV?; footprint (none) -> Potentiometer:PVZ3A
- gave numbers to parts that had none: 158
Connections:
- net VBUS is gone; now on net 5VBUS: C3.2, J4.A4 (VBUS), J4.A9 (VBUS), J4.B4 (VBUS), J4.B9 (VBUS), J5.A4 (VBUS)
- net 5VSYS: now also C8.1
- net GND: now also C2.2, C8.2
- net at D3.1 (K), U1.6 (Vin), U1.7 (Ipk): now also C2.1

Commit message: diagram_SmallPW
Parts:
- removed C1, C10: 4.7uF, Capacitor_SMD:C_0603_1608Metric, symbol Device:C
- added C? (x2): 1uF, Capacitor_SMD:C_0402_1005Metric, symbol Device:C
Connections:
- net 5VSYS: now also C?.1
- net S-S: now also C?.1
- net at Q3.1 (G), R3.2, R4.1: now also C?.2
- net at Q12.1 (G), R35.2, R36.1: now also C?.2
Changed lines of the file:
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@@
     (pin "1")
   )
+  (symbol (lib_id "Device:C") (at 86.36 124.46 0) (unit 1)
+    (in_bom yes) (on_board yes) (fields_autoplaced)
+    (property "Reference" "C?" (id 0) (at 90.17 123.1899 0)
+      (effects (font (size 1.27 1.27)) (justify left))
+    )
+    (property "Value" "1uF" (id 1) (at 90.17 125.7299 0)
+      (effects (font (size 1.27 1.27)) (justify left))
+    )
+    (property "Footprint" "Capacitor_SMD:C_0402_1005Metric" (id 2) (at 87.3252 128.27 0)
+      (effects (font (size 1.27 1.27)) hide)
+    )
+    (property "Datasheet" "~" (id 3) (at 86.36 124.46 0)
+      (effects (font (size 1.27 1.27)) hide)
+    )
+    (pin "1")
+    (pin "2")
+  )
   (symbol (lib_id "Device:C") (at 535.94 299.72 0) (unit 1)
     (in_bom yes) (on_board yes)
@@
     (pin "1")
   )
-  (symbol (lib_id "Device:C") (at 86.36 124.46 0) (unit 1)
-    (in_bom yes) (on_board yes) (fields_autoplaced)
-    (property "Reference" "C1" (id 0) (at 90.17 123.1899 0)
-      (effects (font (size 1.27 1.27)) (justify left))
-    )
-    (property "Value" "4.7uF" (id 1) (at 90.17 125.7299 0)
-      (effects (font (size 1.27 1.27)) (justify left))
-    )
-    (property "Footprint" "Capacitor_SMD:C_0603_1608Metric" (id 2) (at 87.3252 128.27 0)
-      (effects (font (size 1.27 1.27)) hide)
-    )
-    (property "Datasheet" "~" (id 3) (at 86.36 124.46 0)
-      (effects (font (size 1.27 1.27)) hide)
-    )
-    (pin "1")
-    (pin "2")
-  )
   (symbol (lib_id "power:+3.3V") (at 86.36 477.52 0) (unit 1)
     (in_bom yes) (on_board yes)
@@
     (pin "2")
   )
-  (symbol (lib_id "Device:C") (at 271.78 68.58 0) (unit 1)
-    (in_bom yes) (on_board yes) (fields_autoplaced)
-    (property "Reference" "C10" (id 0) (at 275.59 67.3099 0)
-      (effects (font (size 1.27 1.27)) (justify left))
-    )
-    (property "Value" "4.7uF" (id 1) (at 275.59 69.8499 0)
-      (effects (font (size 1.27 1.27)) (justify left))
-    )
-    (property "Footprint" "Capacitor_SMD:C_0603_1608Metric" (id 2) (at 272.7452 72.39 0)
-      (effects (font (size 1.27 1.27)) hide)
-    )
-    (property "Datasheet" "~" (id 3) (at 271.78 68.58 0)
-      (effects (font (size 1.27 1.27)) hide)
-    )
-    (pin "1")
-    (pin "2")
-  )
   (symbol (lib_id "Device:R") (at 114.3 495.3 180) (unit 1)
     (in_bom yes) (on_board yes)
@@
     (pin "3")
   )
+  (symbol (lib_id "Device:C") (at 271.78 68.58 0) (unit 1)
+    (in_bom yes) (on_board yes) (fields_autoplaced)
+    (property "Reference" "C?" (id 0) (at 275.59 67.3099 0)
+      (effects (font (size 1.27 1.27)) (justify left))
+    )
+    (property "Value" "1uF" (id 1) (at 275.59 69.8499 0)
+      (effects (font (size 1.27 1.27)) (justify left))
+    )
+    (property "Footprint" "Capacitor_SMD:C_0402_1005Metric" (id 2) (at 272.7452 72.39 0)
+      (effects (font (size 1.27 1.27)) hide)
+    )
+    (property "Datasheet" "~" (id 3) (at 271.78 68.58 0)
+      (effects (font (size 1.27 1.27)) hide)
+    )
+    (pin "1")
+    (pin "2")
+  )
   (symbol (lib_id "CH340:CH340K") (at 175.26 314.96 0) (unit 1)
     (in_bom yes) (on_board yes)
@@
       (reference "#PWR0188") (unit 1) (value "+5V") (footprint "")
     )
-    (path "/c3a3a00c-41f4-4e49-8328-3123d9395fcd"
-      (reference "C1") (unit 1) (value "4.7uF") (footprint "Capacitor_SMD:C_0603_1608Metric")
-    )
     (path "/3ef05710-0896-433c-8154-4f6c98cf53f6"
       (reference "C2") (unit 1) (value "10uF") (footprint "Capacitor_SMD:C_0805_2012Metric_Pad1.18x1.45mm_HandSolder")
@@
       (reference "C9") (unit 1) (value "470uF") (footprint "")
     )
-    (path "/d6aa6537-9211-4363-9aca-eac86919e41a"
-      (reference "C10") (unit 1) (value "4.7uF") (footprint "Capacitor_SMD:C_0603_1608Metric")
-    )
     (path "/0922cf10-ac75-4624-9ed7-a888b39d0e48"
       (reference "C11") (unit 1) (value "1uF") (footprint "Capacitor_SMD:C_0402_1005Metric")
@@
       (reference "C26") (unit 1) (value "0.1uF") (footprint "Capacitor_SMD:C_0402_1005Metric")
     )
+    (path "/106f4248-2b07-421e-9a4a-617a559f3274"
+      (reference "C?") (unit 1) (value "1uF") (footprint "Capacitor_SMD:C_0402_1005Metric")
+    )
+    (path "/dd7391d4-3349-4aed-b3c7-ec69253dd48c"
+      (reference "C?") (unit 1) (value "1uF") (footprint "Capacitor_SMD:C_0402_1005Metric")
+    )
     (path "/b0ef9f51-3946-44ce-8394-4ce4dea5c00f"

Commit message: 回路図pdf出力
Connections:
- net BOOT: no longer U4.25 (IO0)
- net DIP_SW1: no longer U4.10 (IO25)
- net DIP_SW2: no longer U4.30 (IO18)
- net DIP_SW3: no longer U4.31 (IO19)
- net DIP_SW4: no longer U4.37 (IO23)
- net LED1: no longer U4.24 (IO2)
- net LED2: no longer U4.14 (IO12)
- net LEDTape1_L: no longer U4.8 (IO32)
- net LEDTape2_L: no longer U4.13 (IO14)
- net MainRX0_CH340TX: no longer U4.34 (RXD0/IO3)
- net MainRX2_RS485TX: no longer U4.27 (IO16)
- net MainTX0_CH340RX: no longer U4.35 (TXD0/IO1)
- net MainTX2_RS485RX: no longer U4.28 (IO17)
- net NeoPixel_L: no longer U4.12 (IO27)
- net RESET: no longer U4.3 (EN)
- net I2C0_SCL: no longer names the net of U4.36 (IO22)
- net I2C0_SDA: no longer names the net of U4.33 (IO21)
- net LEDTape3_L: no longer names the net of U4.16 (IO13)
- net LEDTape4_L: no longer names the net of U4.9 (IO33)
- net Mic: no longer names the net of U4.7 (IO35)
- net RS485_GPIO: no longer names the net of U4.11 (IO26)
- net Slide_SW1: no longer names the net of U4.5 (SENSOR_VN)
- net Slide_SW2: no longer names the net of U4.4 (SENSOR_VP)
- net Speker: no longer names the net of U4.26 (IO4)
- net Tact_SW1: no longer names the net of U4.6 (IO34)
- net Tact_SW2: no longer names the net of U4.29 (IO5)
- net Tact_SW3: no longer names the net of U4.23 (IO15)

Commit message: 進捗
Parts:
- added R?: 10k, Resistor_SMD:R_0402_1005Metric, symbol Device:R
- added SW?: SW_SPDT, Slide_Switch:3P_SPDT_SlideSwitch, symbol Switch:SW_SPDT
- C2, C8: footprint Capacitor_SMD:C_0805_2012Metric_Pad1.18x1.45mm_HandSolder -> Capacitor_SMD:C_0805_2012Metric
- D11, D16, D17, D2: value SBR1A40SA -> 1N5819WS; footprint Diode_SMD:D_SMA_Handsoldering -> Diode_SMD:D_SOD-323_HandSoldering
- D4: value SBR1A40SA -> SS2040FL; footprint Diode_SMD:D_SMA_Handsoldering -> Diode_SMD:D_SOD-123
- gave numbers to parts that had none: 2
Connections:
- net +3.3V: now also SW?.2 (B)
- net GND: now also R?.2
- new net Slide_SW1: R?.1, SW?.1 (A)
- no-connect marks 11 -> 12
Other:
- moved on the sheet: D8, R11, R23, SW3

Commit message: エンコーダー基板配線完了
Parts:
- removed D9: ?, symbol Device:D_Schottky
- added C27: 0.1uF, Capacitor_SMD:C_0402_1005Metric, symbol Device:C
- added C28: 470uF, Capacitor_SMD:C_Elec_8x10.2, symbol Device:C_Polarized
- added D9: CBD20150VCT, Package_TO_SOT_THT:TO-220-3_Horizontal_TabDown, symbol Device:D_Schottky_AKA
- C9: footprint (none) -> Capacitor_THT:CP_Radial_D10.0mm_P2.50mm_P5.00mm
- gave numbers to parts that had none: 2
Connections:
- net +5V: now also C28.1
- net GND: now also C27.1, C28.2, D9.1 (A), D9.3 (A)
- net at C2.1, D3.1 (K), U1.6 (Vin)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: now also C27.2
- net at L1.1, Q8.2 (D): now also D9.2 (K)
Other:
- moved on the sheet: C18, C19, C2, C20

Commit message: DCDC回路図変更
Changed lines of the file:
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@@
   (junction (at 744.22 477.52) (diameter 0) (color 0 0 0 0)
   )
-  (junction (at 147.32 93.98) (diameter 0) (color 0 0 0 0)
-  )
   (junction (at 193.04 129.54) (diameter 0) (color 0 0 0 0)
   )
@@
   (junction (at 226.06 76.2) (diameter 0) (color 0 0 0 0)
   )
+  (junction (at 144.78 93.98) (diameter 0) (color 0 0 0 0)
+  )
   (junction (at 673.1 154.94) (diameter 0) (color 0 0 0 0)
   )
@@
   (junction (at 119.38 487.68) (diameter 0) (color 0 0 0 0)
   )
+  (junction (at 144.78 83.82) (diameter 0) (color 0 0 0 0)
+  )
   (junction (at 162.56 297.18) (diameter 0) (color 0 0 0 0)
   )
@@
   (junction (at 281.94 157.48) (diameter 0) (color 0 0 0 0)
   )
-  (junction (at 147.32 83.82) (diameter 0) (color 0 0 0 0)
-  )
   (junction (at 657.86 104.14) (diameter 0) (color 0 0 0 0)
   )
@@
     (stroke (width 0) (type default) (color 0 0 0 0))
   )
-  (wire (pts (xy 147.32 83.82) (xy 147.32 93.98))
+  (wire (pts (xy 144.78 83.82) (xy 144.78 93.98))
     (stroke (width 0) (type default) (color 0 0 0 0))
   )
@@
     (stroke (width 0) (type default) (color 0 0 0 0))
   )
-  (wire (pts (xy 147.32 93.98) (xy 147.32 96.52))
+  (wire (pts (xy 144.78 93.98) (xy 144.78 96.52))
     (stroke (width 0) (type default) (color 0 0 0 0))
   )
@@
     (stroke (width 0) (type default) (color 0 0 0 0))
   )
+  (wire (pts (xy 144.78 93.98) (xy 152.4 93.98))
+    (stroke (width 0) (type default) (color 0 0 0 0))
+  )
   (wire (pts (xy 571.5 269.24) (xy 576.58 269.24))
     (stroke (width 0) (type default) (color 0 0 0 0))
@@
     (stroke (width 0) (type default) (color 0 0 0 0))
   )
-  (wire (pts (xy 147.32 93.98) (xy 152.4 93.98))
-    (stroke (width 0) (type default) (color 0 0 0 0))
-  )
   (polyline (pts (xy 330.2 142.24) (xy 406.4 142.24))
     (stroke (width 0) (type solid) (color 0 0 0 0))
@@
     (stroke (width 0) (type default) (color 0 0 0 0))
   )
-  (wire (pts (xy 147.32 83.82) (xy 144.78 83.82))
+  (wire (pts (xy 144.78 83.82) (xy 149.86 83.82))
     (stroke (width 0) (type default) (color 0 0 0 0))
   )
@@
     (stroke (width 0) (type default) (color 0 0 0 0))
   )
-  (wire (pts (xy 147.32 83.82) (xy 149.86 83.82))
-    (stroke (width 0) (type default) (color 0 0 0 0))
-  )
   (wire (pts (xy 657.86 104.14) (xy 660.4 104.14))
     (stroke (width 0) (type default) (color 0 0 0 0))
@@
     (pin "1")
   )
-  (symbol (lib_id "power:GND") (at 147.32 96.52 0) (mirror y) (unit 1)
+  (symbol (lib_id "power:GND") (at 144.78 96.52 0) (mirror y) (unit 1)
     (in_bom yes) (on_board yes)
-    (property "Reference" "#PWR02" (id 0) (at 147.32 102.87 0)
+    (property "Reference" "#PWR02" (id 0) (at 144.78 102.87 0)
       (effects (font (size 1.27 1.27)) hide)
     )
-    (property "Value" "GND" (id 1) (at 147.193 100.9142 0))
-    (property "Footprint" "" (id 2) (at 147.32 96.52 0)
+    (property "Value" "GND" (id 1) (at 144.653 100.9142 0))
+    (property "Footprint" "" (id 2) (at 144.78 96.52 0)
       (effects (font (size 1.27 1.27)) hide)
     )
-    (property "Datasheet" "" (id 3) (at 147.32 96.52 0)
+    (property "Datasheet" "" (id 3) (at 144.78 96.52 0)
       (effects (font (size 1.27 1.27)) hide)
     )

Commit message: 回路図ほぼ完成
Parts:
- removed C9: 470uF, Capacitor_THT:CP_Radial_D10.0mm_P2.50mm_P5.00mm, symbol Device:C_Polarized_US
- removed D4: SS2040FL, Diode_SMD:D_SOD-123, symbol Device:D_Schottky
- removed D8: Yellow, LED_SMD:LED_0603_1608Metric_Pad1.05x0.95mm_HandSolder, symbol Device:LED
- removed D9: CBD20150VCT, Package_TO_SOT_THT:TO-220-3_Horizontal_TabDown, symbol Device:D_Schottky_AKA
- removed J6: AudioJack2_Ground, symbol Connector:AudioJack2_Ground
- removed R31: 10k, Resistor_SMD:R_0402_1005Metric, symbol Device:R
- removed U1: MC34063AD, Package_SO:SOIC-8_3.9x4.9mm_P1.27mm, symbol Regulator_Switching:MC34063AD
- added C29: 0.1uF, Capacitor_SMD:C_0402_1005Metric, symbol Device:C
- added C30: 100pF, Capacitor_SMD:C_0603_1608Metric, symbol Device:C
- added C32, C36, C9: C_snub, Capacitor_SMD:C_0603_1608Metric, symbol Device:C
- added C34: 10uF, Capacitor_SMD:C_0805_2012Metric, symbol Device:C
- added C35: 470uF, Capacitor_THT:CP_Radial_D10.0mm_P2.50mm_P5.00mm, symbol Device:C_Polarized_US
- added D28: CBD20150VCT, Package_TO_SOT_THT:TO-220-3_Horizontal_TabDown, symbol Device:D_Schottky_AKA
- added D29, D9: 1N5819WS, Diode_SMD:D_SOD-323_HandSoldering, symbol Device:D_Schottky
- added D4: Red, LED_SMD:LED_0603_1608Metric_Pad1.05x0.95mm_HandSolder, symbol Device:LED
- added D8: SS2040FL, Diode_SMD:D_SOD-123, symbol Device:D_Schottky
- added H6, H7: MountingHole_Pad, TestPoint:TestPoint_Pad_1.5x1.5mm, symbol Mechanical:MountingHole_Pad
- added J6: AudioJack3, Connector_Audio:Jack_3.5mm_Switronic_ST-005-G_horizontal, symbol Connector:AudioJack3
- added Q21: MTP4835I3, Package_TO_SOT_SMD:TO-252-3_TabPin2, symbol Device:Q_PMOS_GDS
- added R60, R69: 10k, Resistor_SMD:R_0402_1005Metric, symbol Device:R
- added R61, R67: R_snub, Resistor_SMD:R_0603_1608Metric, symbol Device:R
- added R68: 1.5k, Resistor_SMD:R_0603_1608Metric, symbol Device:R
- added R70: 5.1k, Resistor_SMD:R_0603_1608Metric, symbol Device:R
- added R71: 7.5k, Resistor_SMD:R_0603_1608Metric, symbol Device:R
- added R72: 2k, Resistor_SMD:R_0603_1608Metric, symbol Device:R
- added R73: 5.1k, Resistor_SMD:R_0402_1005Metric, symbol Device:R
- added U1: M51957B, Package_SO:SOP-8_3.9x4.9mm_P1.27mm, symbol Voltage_Supervisor:M51957B
- added U6: MC34063AD, Package_SO:SOIC-8_3.9x4.9mm_P1.27mm, symbol Regulator_Switching:MC34063AD
- C2: value 10uF -> 4700pF; footprint Capacitor_SMD:C_0805_2012Metric -> Capacitor_SMD:C_0603_1608Metric
- C27: value 0.1uF -> 10uF; footprint Capacitor_SMD:C_0402_1005Metric -> Capacitor_SMD:C_0805_2012Metric
- C4: value 100pF -> 0.1uF; footprint Capacitor_SMD:C_0603_1608Metric -> Capacitor_SMD:C_0402_1005Metric
- D7: value Red -> Yellow
- J10, J11, J9: footprint Connector_Molex:Molex_SPOX_5268-03A_1x03_P2.50mm_Horizontal -> Connector_Molex:Molex_SPOX_5267-03A_1x03_P2.50mm_Vertical
- R20: value 1k -> R_snub; footprint Resistor_SMD:R_0402_1005Metric -> Resistor_SMD:R_0603_1608Metric
- R21: value 1k -> 10k
- R22: value 510 -> 1k
- R27: value 10 -> 1k; footprint Resistor_SMD:R_0603_1608Metric -> Resistor_SMD:R_0402_1005Metric
- R29: value 1.5k -> 1k; footprint Resistor_SMD:R_0603_1608Metric -> Resistor_SMD:R_0402_1005Metric
- R32: value 5.1k -> 510; footprint Resistor_SMD:R_0603_1608Metric -> Resistor_SMD:R_0402_1005Metric
- R59: value 10k -> 10; footprint Resistor_SMD:R_0402_1005Metric -> Resistor_SMD:R_0603_1608Metric
Connections:
- net +5V: no longer C19.1
- net 5VSYS: now also C19.1, D9.2 (A), Q21.2 (D); no longer C8.1, L1.2, R32.2
- net BOOT: no longer C15.1, H4.1, R41.2, SW5.1 (A)
- net DAC_L: now also U4.10 (IO25), J6.T
- net DAC_R: now also U4.11 (IO26), J6.R
- net DIP_SW3: now also R11.2; no longer R12.2
- net DIP_SW4: now also R12.2; no longer R13.2
- net GND: now also C2.1, C27.2, R11.1, R13.2, R19.2, R21.2, C29.1, C30.1, C32.1, C34.2, C35.2, C36.1, C9.1, D28.1 (A), D28.3 (A), D4.1 (K), J6.S, R68.1, R72.2, U1.4 (GND), U6.2 (SwE), U6.3 (TC), U6.4 (GND); no longer C2.2, C27.1, R11.2, R13.1, R29.1, R59.2
- net LED0: now also R22.2; no longer R19.2
- net LED1: now also R23.2; no longer R20.2
- net LED2: now also R27.2; no longer R21.2
- net MainRX0_CH340TX: now also U4.34 (RXD0/IO3)
- net MainRX2_RS485TX: now also U4.27 (IO16)
- net MainTX0_CH340RX: now also U4.35 (TXD0/IO1)
- net MainTX2_RS485RX: now also U4.28 (IO17)
- net MonitorLED0: now also R29.2; no longer R23.2
- net RESET: now also U4.3 (EN)
- net Sensor0: now also H6.1
- net Sensor1: now also H7.1
- net Slide_SW0: now also R13.1; no longer R11.1
- net Slide_SW1: now also R21.1; no longer R59.1
- net VDD: now also C4.2, C8.1, R19.1, R20.2, R32.1, D29.1 (K), R60.2, U1.7 (VCC); no longer R22.1
- net at Q5.1 (B): now also R32.2, D8.1 (K), U6.1 (SwC), U6.8 (DC); no longer R22.2
- net at Q5.2 (E): now also R59.2, D8.2 (A); no longer R27.2
- net at D7.2 (A): now also R29.1; no longer R21.1
- net at L1.1, Q8.2 (D): now also D28.2 (K), R61.2
- net at RV1.2: now also R68.2, R69.1; no longer R29.2
- net at RV1.1: now also R69.2
- net at R23.1: now also D5.2 (A)
- net at R27.1: now also D6.2 (A); no longer Q8.1 (G)
- net Vfb: now reaches RV1.3
- net Vfb: now also R70.1, U6.5 (Vfb); no longer R32.1
- net at R20.1: now also C9.2; no longer D6.2 (A)
- net IO0: now reaches U4.25 (IO0)
- net IO0: now also C15.1, H4.1, R41.2, SW5.1 (A)
- new net: C34.1, C35.1, D29.2 (A), D9.1 (K), L1.2, Q21.3 (S), R67.2, R70.2, R71.2, R73.1
- new net: C27.1, C29.2, D3.1 (K), U6.6 (Vin), U6.7 (Ipk)
- new net: C32.2, R61.1
- new net: Q8.1 (G), R59.1, R60.1
- new net: D4.2 (A), R22.1
- new net: C36.2, R67.1
- new net: C2.2, U1.5 (Cdelay)
- new net SHDN_overV: Q21.1 (G), R73.2, U1.6 (OUT)
- new net V_Surv.: R71.1, R72.1, U1.2 (IN)
Other:
- note added: "5V監視"
- note removed: "STM"
- moved on the sheet: C10, C11, C12, C18, C19, C20, C28, C7, D10, D11, D12, D13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

Commit message: Pole,Panelほぼ完成
Parts:
- removed C19, C20: 470uF, Capacitor_SMD:C_Elec_8x10.2, symbol Device:C_Polarized
- removed H1, H2: MountingHole_Pad, TestPoint:TestPoint_Pad_1.5x1.5mm, symbol Mechanical:MountingHole_Pad
- removed J5: USB_C_Receptacle_USB2.0, USB_DIP:USB_C(simple), symbol Connector:USB_C_Receptacle_USB2.0
- removed R34, R41: 10k, Resistor_SMD:R_0402_1005Metric, symbol Device:R
- added C19: 10uF, Capacitor_SMD:C_0805_2012Metric, symbol Device:C
- added C31: 0.1uF, Capacitor_SMD:C_0402_1005Metric, symbol Device:C
- added JP3: Jumper_2_Open, Jumper:SolderJumper-2_P1.3mm_Open_TrianglePad1.0x1.5mm, symbol Jumper:Jumper_2_Open
- added R31: 10k, Resistor_SMD:R_0402_1005Metric, symbol Device:R
- Q1, Q21, Q3, Q8, U3: footprint Package_TO_SOT_SMD:TO-252-3_TabPin2 -> Package_TO_SOT_SMD:TO-252-2
Connections:
- net BOOT is gone; now on net IO0: Q10.3 (D)
- net +3.3V: now also C19.1, R31.1
- net DIP_SW0: now also U4.26 (IO4)
- net DIP_SW1: now also U4.12 (IO27)
- net DIP_SW2: now also U4.9 (IO33)
- net DIP_SW3: now also U4.5 (SENSOR_VN)
- net DIP_SW4: now also U4.4 (SENSOR_VP)
- net GND: now also C19.2, C31.1; no longer U6.3 (TC)
- net IO0: now also R31.2
- net LED0: now also U4.16 (IO13)
- net LED1: now also U4.14 (IO12)
- net LED2: now also U4.13 (IO14)
- net LEDTape0_L: now also U4.30 (IO18)
- net LEDTape1_L: now also U4.33 (IO21)
- net LEDTape2_L: now also U4.31 (IO19)
- net MonitorLED0: now also U4.24 (IO2)
- net NeoPixel_L: now also U4.23 (IO15)
- net RS485_A: now also R58.2; no longer JP2.1 (A)
- net RS485_B: now also JP2.1 (A); no longer R58.2
- net Sensor0: now also U4.7 (IO35)
- net Sensor1: now also U4.6 (IO34)
- net Slide_SW0: now also U4.36 (IO22)
- net Slide_SW1: now also U4.37 (IO23)
- net VDD: now also C31.2
- net V_Measure: now also U4.8 (IO32)
- net 5VBUS_fetF: now reaches C7.2, Q4.1 (G), R17.2
- net 5VBUS_fetF: now also JP3.1 (A)
- net 5VBUS_fetB: now reaches Q11.3 (C), Q7.1 (G), R28.2
- net 5VBUS_fetB: now also JP3.2 (B)
- net at C30.2: now also U6.3 (TC)
- net CC1: no longer names the net of J4.A5 (CC1), R15.2
- net CC2: no longer names the net of J4.B5 (CC2), R14.2
- net D+: no longer names the net of J4.A6 (D+), J4.B6 (D+), U2.1 (UD+)
- net D-: no longer names the net of J4.A7 (D-), J4.B7 (D-), U2.2 (UD-)
- no-connect marks 12 -> 13
Other:
- note removed: "SDカード"
- moved on the sheet: C7, D10, J4, JP2, Q11, Q4, Q6, Q7, R16, R17, R18, R19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
