File: Pole/Pole.kicad_sch (KiCad schematic)
At the start: 190 parts, among them J1 Conn_01x02_Male, J10 Conn_01x03_Male, J11 Conn_01x03_Male, J12 Conn_01x04_Male, J13 Conn_01x04_Male, J2 Conn_01x02_Female, J3 Conn_01x02_Female, J4 USB_C_Receptacle_USB2.0, J6 AudioJack3, J7 Conn_01x03_Male, J8 Conn_01x03_Male, J9 Conn_01x03_Male, Q1 MTP4835I3, Q10 BSS138, Q11 S8050, Q12 SSM3J332R, Q13 S8050, Q14 SSM3J332R, Q15 S8050, Q16 BSS138, Q17 S8050, Q18 BSS138, Q19 BSS138, Q2 BSS138, Q20 BSS138, Q21 MTP4835I3, Q3 MTP4835I3, Q4 SSM3J332R, Q5 2SC3265, Q6 S8050, Q7 SSM3J332R, Q8 MTP4835I3, Q9 BSS138, SW1 SW_DIP_x05, SW2 SW_SPDT, SW3 SW_SPDT, SW4 SW_SPST, SW5 SW_SPST, SW6 SW_SPDT, U1 M51957B, U2 CH340K, U3 AZ1084CD-3.3, U4 ESP32-WROOM-32, U5 MAX3485, U6 MC34063AD

Commit message: Mother_Ctrl回路図プロット
Parts:
- removed TP1, TP2, TP3, TP4: TestPoint, TestPoint:TestPoint_THTPad_D2.0mm_Drill1.0mm, symbol Connector:TestPoint
Changed lines of the file:
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@@
     (stroke (width 0) (type default) (color 0 0 0 0))
   )
-  (wire (pts (xy 480.06 160.02) (xy 480.06 162.56))
-    (stroke (width 0) (type default) (color 0 0 0 0))
-  )
   (wire (pts (xy 688.34 482.6) (xy 688.34 483.87))
     (stroke (width 0) (type default) (color 0 0 0 0))
@@
     (stroke (width 0) (type default) (color 0 0 0 0))
   )
-  (wire (pts (xy 459.74 160.02) (xy 459.74 162.56))
-    (stroke (width 0) (type default) (color 0 0 0 0))
-  )
   (wire (pts (xy 675.64 469.9) (xy 685.8 469.9))
     (stroke (width 0) (type default) (color 0 0 0 0))
@@
     (stroke (width 0) (type default) (color 0 0 0 0))
   )
-  (wire (pts (xy 469.9 160.02) (xy 469.9 162.56))
-    (stroke (width 0) (type default) (color 0 0 0 0))
-  )
   (polyline (pts (xy 441.96 109.22) (xy 441.96 38.1))
     (stroke (width 0) (type solid) (color 0 0 0 0))
@@
     (stroke (width 0) (type default) (color 0 0 0 0))
   )
-  (wire (pts (xy 490.22 160.02) (xy 490.22 162.56))
-    (stroke (width 0) (type default) (color 0 0 0 0))
-  )
   (wire (pts (xy 401.32 142.24) (xy 401.32 146.05))
     (stroke (width 0) (type default) (color 0 0 0 0))
@@
     (pin "2")
   )
-  (symbol (lib_id "power:+5V") (at 469.9 160.02 0) (mirror y) (unit 1)
-    (in_bom yes) (on_board yes) (fields_autoplaced)
-    (property "Reference" "#PWR0158" (id 0) (at 469.9 163.83 0)
-      (effects (font (size 1.27 1.27)) hide)
-    )
-    (property "Value" "+5V" (id 1) (at 469.9 156.21 0))
-    (property "Footprint" "" (id 2) (at 469.9 160.02 0)
-      (effects (font (size 1.27 1.27)) hide)
-    )
-    (property "Datasheet" "" (id 3) (at 469.9 160.02 0)
-      (effects (font (size 1.27 1.27)) hide)
-    )
-    (pin "1")
-  )
   (symbol (lib_id "Connector:Conn_01x02_Male") (at 58.42 53.34 0) (unit 1)
     (in_bom yes) (on_board yes) (fields_autoplaced)
@@
     (pin "2")
   )
-  (symbol (lib_id "power:VCC") (at 480.06 160.02 0) (mirror y) (unit 1)
-    (in_bom yes) (on_board yes)
-    (property "Reference" "#PWR0157" (id 0) (at 480.06 163.83 0)
-      (effects (font (size 1.27 1.27)) hide)
-    )
-    (property "Value" "VCC" (id 1) (at 480.06 154.94 0))
-    (property "Footprint" "" (id 2) (at 480.06 160.02 0)
-      (effects (font (size 1.27 1.27)) hide)
-    )
-    (property "Datasheet" "" (id 3) (at 480.06 160.02 0)
-      (effects (font (size 1.27 1.27)) hide)
-    )
-    (pin "1")
-  )
   (symbol (lib_id "Device:R") (at 144.78 492.76 180) (unit 1)
     (in_bom yes) (on_board yes)
@@
     (pin "2")
   )
-  (symbol (lib_id "Connector:TestPoint") (at 459.74 162.56 180) (unit 1)
-    (in_bom yes) (on_board yes)
-    (property "Reference" "TP1" (id 0) (at 459.74 170.18 0)
-      (effects (font (size 1.27 1.27)) (justify left))
-    )
-    (property "Value" "TestPoint" (id 1) (at 459.74 167.64 0)
-      (effects (font (size 1.27 1.27)) (justify left))
-    )
-    (property "Footprint" "TestPoint:TestPoint_THTPad_D2.0mm_Drill1.0mm" (id 2) (at 454.66 162.56 0)
-      (effects (font (size 1.27 1.27)) hide)
-    )
-    (property "Datasheet" "~" (id 3) (at 454.66 162.56 0)
-      (effects (font (size 1.27 1.27)) hide)
-    )
-    (pin "1")
-  )
   (symbol (lib_id "NeoPixel:WS2812C-2020-V1") (at 637.54 294.64 0) (unit 1)
     (in_bom yes) (on_board yes)
@@
     (pin "1")
   )
-  (symbol (lib_id "Connector:TestPoint") (at 469.9 162.56 180) (unit 1)
-    (in_bom yes) (on_board yes)
-    (property "Reference" "TP2" (id 0) (at 469.9 170.18 0)
-      (effects (font (size 1.27 1.27)) (justify left))
-    )
-    (property "Value" "TestPoint" (id 1) (at 469.9 167.64 0)
-      (effects (font (size 1.27 1.27)) (justify left))
-    )
-    (property "Footprint" "TestPoint:TestPoint_THTPad_D2.0mm_Drill1.0mm" (id 2) (at 464.82 162.56 0)
-      (effects (font (size 1.27 1.27)) hide)
-    )
-    (property "Datasheet" "~" (id 3) (at 464.82 162.56 0)
-      (effects (font (size 1.27 1.27)) hide)
-    )
-    (pin "1")
-  )
   (symbol (lib_id "power:+3.3V") (at 670.56 467.36 0) (unit 1)
     (in_bom yes) (on_board yes)
@@
     (pin "1")
   )
-  (symbol (lib_id "power:VDD") (at 459.74 160.02 0) (unit 1)
-    (in_bom yes) (on_board yes) (fields_autoplaced)
-    (property "Reference" "#PWR0159" (id 0) (at 459.74 163.83 0)
-      (effects (font (size 1.27 1.27)) hide)
-    )
-    (property "Value" "VDD" (id 1) (at 459.74 156.21 0))
-    (property "Footprint" "" (id 2) (at 459.74 160.02 0)
-      (effects (font (size 1.27 1.27)) hide)
-    )
-    (property "Datasheet" "" (id 3) (at 459.74 160.02 0)
-      (effects (font (size 1.27 1.27)) hide)
-    )
-    (pin "1")
-  )
   (symbol (lib_id "Device:R") (at 193.04 321.31 0) (unit 1)
     (in_bom yes) (on_board yes)
@@
     (pin "4")
   )
-  (symbol (lib_id "Connector:TestPoint") (at 480.06 162.56 180) (unit 1)
-    (in_bom yes) (on_board yes)
-    (property "Reference" "TP3" (id 0) (at 480.06 170.18 0)
-      (effects (font (size 1.27 1.27)) (justify left))
-    )
-    (property "Value" "TestPoint" (id 1) (at 480.06 167.64 0)
-      (effects (font (size 1.27 1.27)) (justify left))
-    )
-    (property "Footprint" "TestPoint:TestPoint_THTPad_D2.0mm_Drill1.0mm" (id 2) (at 474.98 162.56 0)
-      (effects (font (size 1.27 1.27)) hide)
-    )
-    (property "Datasheet" "~" (id 3) (at 474.98 162.56 0)
-      (effects (font (size 1.27 1.27)) hide)
-    )
-    (pin "1")
-  )
   (symbol (lib_id "Device:R") (at 688.34 487.68 0) (mirror x) (unit 1)
     (in_bom yes) (on_board yes) (fields_autoplaced)
@@
     (pin "2")
   )
-  (symbol (lib_id "Connector:TestPoint") (at 490.22 162.56 180) (unit 1)
-    (in_bom yes) (on_board yes)
-    (property "Reference" "TP4" (id 0) (at 490.22 170.18 0)
-      (effects (font (size 1.27 1.27)) (justify left))
-    )
-    (property "Value" "TestPoint" (id 1) (at 490.22 167.64 0)
-      (effects (font (size 1.27 1.27)) (justify left))
-    )
-    (property "Footprint" "TestPoint:TestPoint_THTPad_D2.0mm_Drill1.0mm" (id 2) (at 485.14 162.56 0)
-      (effects (font (size 1.27 1.27)) hide)
-    )
-    (property "Datasheet" "~" (id 3) (at 485.14 162.56 0)
-      (effects (font (size 1.27 1.27)) hide)
-    )
-    (pin "1")
-  )
   (symbol (lib_id "Switch:SW_DIP_x05") (at 114.3 482.6 0) (mirror y) (unit 1)
     (in_bom yes) (on_board yes) (fields_autoplaced)
@@
     (pin "2")
   )
-  (symbol (lib_id "power:+3.3V") (at 490.22 160.02 0) (unit 1)
-    (in_bom yes) (on_board yes) (fields_autoplaced)
-    (property "Reference" "#PWR0160" (id 0) (at 490.22 163.83 0)
-      (effects (font (size 1.27 1.27)) hide)
-    )
-    (property "Value" "+3.3V" (id 1) (at 490.22 156.21 0))
-    (property "Footprint" "" (id 2) (at 490.22 160.02 0)
-      (effects (font (size 1.27 1.27)) hide)
-    )
-    (property "Datasheet" "" (id 3) (at 490.22 160.02 0)
-      (effects (font (size 1.27 1.27)) hide)
-    )
-    (pin "1")
-  )
   (symbol (lib_id "Device:C") (at 147.32 302.26 270) (unit 1)
     (in_bom yes) (on_board yes)
@@
       (reference "#PWR0156") (unit 1) (value "+3.3V") (footprint "")
     )
-    (path "/257b08f1-7581-4c25-88a1-95da6ebe9a84"
-      (reference "#PWR0157") (unit 1) (value "VCC") (footprint "")
-    )
-    (path "/13e279b7-8972-4446-ad2c-ebd4f09173fa"
-      (reference "#PWR0158") (unit 1) (value "+5V") (footprint "")
-    )
-    (path "/8bb47316-7add-4708-80dc-91ed95f6e611"
-      (reference "#PWR0159") (unit 1) (value "VDD") (footprint "")
-    )
-    (path "/faf11c09-9285-4387-9773-e9edf5927b9a"
-      (reference "#PWR0160") (unit 1) (value "+3.3V") (footprint "")
-    )
     (path "/1229d043-12ba-4d6c-8ad5-8a0dc67dcb77"
       (reference "#PWR0161") (unit 1) (value "+3.3V") (footprint "")
@@
       (reference "SW6") (unit 1) (value "SW_SPDT") (footprint "Slide_Switch:3P_SPDT_SlideSwitch")
     )
-    (path "/48768add-0612-411f-84b5-26f5b57c59b0"
-      (reference "TP1") (unit 1) (value "TestPoint") (footprint "TestPoint:TestPoint_THTPad_D2.0mm_Drill1.0mm")
-    )
-    (path "/87e618e2-c83a-46d0-b5d6-914525e7b43c"
-      (reference "TP2") (unit 1) (value "TestPoint") (footprint "TestPoint:TestPoint_THTPad_D2.0mm_Drill1.0mm")
-    )
-    (path "/c35cfc87-c065-484c-9848-47bc1d1b7d54"
-      (reference "TP3") (unit 1) (value "TestPoint") (footprint "TestPoint:TestPoint_THTPad_D2.0mm_Drill1.0mm")
-    )
-    (path "/cc235018-044b-4fd4-bee0-b9e430086c9c"
-      (reference "TP4") (unit 1) (value "TestPoint") (footprint "TestPoint:TestPoint_THTPad_D2.0mm_Drill1.0mm")
-    )
     (path "/7d0ce7da-9bdb-4e4d-880d-db446d964720"
