File: Pole/Pole.kicad_pcb (KiCad board)
At the start: 2 copper layers, 100 x 60 mm, 202 parts, among them J1 Conn_01x02_Male, J10 Conn_01x03_Male, J11 Conn_01x03_Male, J12 Conn_01x04_Male, J13 Conn_01x04_Male, J2 Conn_01x02_Female, J3 Conn_01x02_Female, J4 USB_C_Receptacle_USB2.0, J5 USB_C_Receptacle_USB2.0, J6 AudioJack3, J7 Conn_01x03_Male, J8 Conn_01x03_Male, J9 Conn_01x03_Male, Q1 MTP4835I3, Q10 BSS138, Q11 S8050, Q12 SSM3J332R, Q13 S8050, Q14 SSM3J332R, Q15 S8050, Q16 BSS138, Q17 S8050, Q18 BSS138, Q19 BSS138, Q2 BSS138, Q20 BSS138, Q21 MTP4835I3, Q3 MTP4835I3, Q4 SSM3J332R, Q5 2SC3265, Q6 S8050, Q7 SSM3J332R, Q8 MTP4835I3, Q9 BSS138, SW1 SW_DIP_x05, SW2 SW_SPDT, SW3 SW_SPDT, SW4 SW_SPST, SW5 SW_SPST, SW6 SW_SPDT, U1 M51957B, U2 CH340K, U3 AZ1084CD-3.3, U4 ESP32-WROOM-32, U5 MAX3485, U6 MC34063AD

Commit message: 回路図プロット
Parts:
- removed C31: 22uF, Capacitor_SMD:C_0805_2012Metric
- removed C33: 10uF, Capacitor_SMD:C_0805_2012Metric
- removed MD1: OKL-T/6-W12N-C, DCDC_Regulator:MURATA_OKL-T-6-W12N-C
- removed R31: 10k, Resistor_SMD:R_0402_1005Metric
- removed R62: 100k, Resistor_SMD:R_0402_1005Metric
- removed R63: 1k, Resistor_SMD:R_0402_1005Metric
- removed R64: 330, Resistor_SMD:R_0402_1005Metric
- removed R65: 10, Resistor_SMD:R_0402_1005Metric
- removed R66: 1.2k, Resistor_SMD:R_0402_1005Metric
- J10, J11, J9: footprint Connector_Molex:Molex_SPOX_5268-03A_1x03_P2.50mm_Horizontal -> Connector_Molex:Molex_SPOX_5267-03A_1x03_P2.50mm_Vertical
- moved Q1 197.1 mm to (-23.3, 21.1), turned to 180 degrees
- moved J1 170.4 mm to (-29.9, -15.4)
- moved J2 137.5 mm to (-34.3, -1.20), turned to 90 degrees
- moved J3 113.1 mm to (-34.5, 14.0), turned to 90 degrees
- moved F1 108.2 mm to (-25.1, 2.06), turned to 90 degrees
- moved U4 65.1 mm to (30.3, -20.6)
Connections:
- D9 pad 1: VDD -> Net-(C34-Pad1)

Commit message: Pole,Panelほぼ完成
Parts:
- removed C20: 470uF, Capacitor_SMD:C_Elec_8x10.2
- removed H1, H2: MountingHole_Pad, TestPoint:TestPoint_Pad_1.5x1.5mm
- removed J5: USB_C_Receptacle_USB2.0, USB_DIP:USB_C(simple)
- removed R34, R41: 10k, Resistor_SMD:R_0402_1005Metric
- added C31: 0.1uF, Capacitor_SMD:C_0402_1005Metric, F.Cu at (-40.8, -30.4)
- added JP3: Jumper_2_Open, Jumper:SolderJumper-2_P1.3mm_Open_TrianglePad1.0x1.5mm, F.Cu at (-85.5, -28.4)
- added R31: 10k, Resistor_SMD:R_0402_1005Metric, F.Cu at (-66.2, -19.2)
- C19: value 470uF -> 10uF; footprint Capacitor_SMD:C_Elec_8x10.2 -> Capacitor_SMD:C_0805_2012Metric
- H6, H7, JP1: moved to B.Cu
- Q1, Q21, Q3, Q8, U3: footprint Package_TO_SOT_SMD:TO-252-3_TabPin2 -> Package_TO_SOT_SMD:TO-252-2
- moved C5 315.4 mm to (-96.7, -10.3)
- moved H4 310.0 mm to (-87.4, 49.2)
- moved TP4 310.0 mm to (-91.2, 46.9)
- moved R28 293.1 mm to (-82.4, -22.6), turned to 180 degrees
- moved TP5 292.3 mm to (-82.0, 46.1)
- moved R57 291.5 mm to (-89.6, -50.3), turned to 180 degrees
- moved C6 289.4 mm to (-93.2, -9.57), turned to -90 degrees
- moved R25 288.2 mm to (-80.4, -22.6)
- moved D20 286.4 mm to (-81.8, -37.8), turned to -90 degrees
- moved U2 286.1 mm to (-95.8, -14.1), turned to -90 degrees
- moved R38 285.8 mm to (-68.1, -36.6), turned to 90 degrees
- moved Q9 284.9 mm to (-96.5, -6.74)
- moved R52 284.2 mm to (-68.8, -53.7), turned to 180 degrees
- moved D22 283.1 mm to (-81.8, -41.2), turned to -90 degrees
- moved Q7 282.1 mm to (-84.1, -25.3), turned to 180 degrees
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Connections:
- net /CC1 renamed Net-(J4-PadA5)
- net /CC2 renamed Net-(J4-PadB5)
- net /D+ renamed Net-(J4-PadA6)
- net /D- renamed Net-(J4-PadA7)
- net Net-(C7-Pad2) renamed /5VBUS_fetF
- net Net-(H2-Pad1) renamed /5VBUS_fetB
- C19 pad 1: /5VSYS -> +3.3V
- C30 pad 2: unconnected-(C30-Pad2) -> Net-(C30-Pad2)
- JP2 pad 1: RS485_A -> RS485_B
- Q10 pad 3: BOOT -> IO0
- R58 pad 2: RS485_B -> RS485_A
- U4 pad 12: unconnected-(U4-Pad12) -> DIP_SW1
- U4 pad 13: unconnected-(U4-Pad13) -> LED2
- U4 pad 14: unconnected-(U4-Pad14) -> LED1
- U4 pad 16: unconnected-(U4-Pad16) -> LED0
- U4 pad 23: unconnected-(U4-Pad23) -> NeoPixel_L
- U4 pad 24: unconnected-(U4-Pad24) -> MonitorLED0
- U4 pad 26: unconnected-(U4-Pad26) -> DIP_SW0
- U4 pad 30: unconnected-(U4-Pad30) -> LEDTape0_L
- U4 pad 31: unconnected-(U4-Pad31) -> LEDTape2_L
- U4 pad 33: unconnected-(U4-Pad33) -> LEDTape1_L
- U4 pad 36: unconnected-(U4-Pad36) -> Slide_SW0
- U4 pad 37: unconnected-(U4-Pad37) -> Slide_SW1
- U4 pad 4: unconnected-(U4-Pad4) -> DIP_SW4
- U4 pad 5: unconnected-(U4-Pad5) -> DIP_SW3
- U4 pad 6: unconnected-(U4-Pad6) -> Sensor1
- U4 pad 7: unconnected-(U4-Pad7) -> Sensor0
- U4 pad 8: unconnected-(U4-Pad8) -> V_Measure
- U4 pad 9: unconnected-(U4-Pad9) -> DIP_SW2
- U6 pad 3: GND -> Net-(C30-Pad2)
Routing:
- net GND: track 0.00 -> 587.4 mm, vias 0 -> 790
- net +3.3V: track 0.00 -> 247.9 mm, vias 0 -> 16
- net +5V: track 0.00 -> 203.8 mm, vias 0 -> 2
- net /5VSYS: track 0.00 -> 122.3 mm, vias 0 -> 5
- net VDD: track 0.00 -> 84.5 mm, vias 0 -> 2
- net /5V_IND: track 0.00 -> 74.2 mm, vias 0 -> 6
- net RESET: track 0.00 -> 64.1 mm, vias 0 -> 4
- net LEDTape1_L: track 0.00 -> 64.0 mm, vias 0 -> 2
- net Slide_SW0: track 0.00 -> 60.5 mm, vias 0 -> 2
- net Vfb: track 0.00 -> 58.5 mm, vias 0 -> 2
- net LEDTape2_L: track 0.00 -> 58.1 mm, vias 0 -> 2
- net DAC_L: track 0.00 -> 57.3 mm, vias 0 -> 1
- net Slide_SW1: track 0.00 -> 55.7 mm, vias 0 -> 1
- net LEDTape0_L: track 0.00 -> 55.3 mm, vias 0 -> 2
- net Sensor1: track 0.00 -> 55.1 mm, vias 0 -> 1
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- added copper zone on F.Cu, net /12VBAT
- added copper zone on F.Cu, net /5VSYS
- added copper zone on F.Cu, net /S-S
- added copper zone on B.Cu, net GND
- added copper zone on F.Cu, net GND
- added copper zone on F.Cu, net Net-(C34-Pad1)
- added copper zone on F.Cu, net Net-(D28-Pad2)
- added copper zone on F.Cu, net Net-(F1-Pad1)
- added copper zone on F.Cu, net Net-(Q12-Pad3)
- added copper zone on F.Cu, net VDD
Other:
- board size 100 x 60 mm -> 100 x 70 mm

Commit message: Mother_Ctrl回路図プロット
Parts:
- removed TP1, TP2, TP3, TP4: TestPoint, TestPoint:TestPoint_THTPad_D2.0mm_Drill1.0mm
- H3, H4: moved to B.Cu
- moved TP5 80.1 mm to (-96.4, -32.8)
- moved H4 54.7 mm to (-92.5, -5.29), turned to 180 degrees
- moved H3 39.8 mm to (-76.7, -0.47), turned to 180 degrees
Routing:
- net +3.3V: track 247.9 -> 257.4 mm
- net GND: track 587.4 -> 587.6 mm, vias 790 -> 792

Commit message: 多分完成
Parts:
- moved C1 254.9 mm to (215.0, 119.6)
- moved C10 254.9 mm to (159.3, 71.7)
- moved C11 254.9 mm to (152.4, 80.6)
- moved C12 254.9 mm to (156.4, 82.2)
- moved C13 254.9 mm to (155.8, 122.5)
- moved C14 254.9 mm to (154.7, 120.1)
- moved C15 254.9 mm to (158.2, 93.0)
- moved C16 254.9 mm to (154.2, 122.6)
- moved C17 254.9 mm to (150.2, 102.3)
- moved C18 254.9 mm to (190.2, 79.8)
- moved C19 254.9 mm to (149.7, 91.0)
- moved C2 254.9 mm to (160.7, 81.5)
- moved C21 254.9 mm to (144.7, 71.2)
- moved C22 254.9 mm to (144.5, 85.2)
- moved C23 254.9 mm to (144.6, 81.7)
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Other:
- board text added: "+3.3V"
- board text added: "+5V"
- board text added: "5VIND"
- board text added: "5VSYS"
- board text added: "Analog"
- board text added: "BOOT"
- board text added: "Designed by @cat_nekonekone"
- board text added: "IO12"
- board text added: "IO13"
- board text added: "IO14"
- board text added: "IO2"
- board text added: "IO22"
- board text added: "IO23"
- board text added: "IO27"
- board text added: "IO33"
- board text added: "IO36"
- board text added: "IO39"
- board text added: "IO4"
- board text added: "JLCJLCJLCJLC"
- board text added: "NeoPixel"
- board text added: "POWER"
- board text added: "RST"
- board text added: "RX0:IO3"
- board text added: "RX2:IO16"
- board text added: "TX0:IO1"
- board text added: "TX2:IO17"
- board text added: "Tomoshibi"
- board text added: "[Audio]"
- board text added: "[DAC_L]IO25"
- board text added: "[DAC_R]IO26"
- board text added: "[LEDTape0]"
- board text added: "[LEDTape0]IO18"
- board text added: "[LEDTape1]"
- board text added: "[LEDTape1]IO21"
- board text added: "[LEDTape2]"
- board text added: "[LEDTape2]IO19"
- board text added: "[RS485]"
- board text added: "[Sensor0]"
- board text added: "[Sensor0]IO35"
- board text added: "[Sensor1]"
- board text added: "[Sensor1]IO34"
- board text added: "[V_meas.]IO32"
- board text added: "[Write]"
- board text added: "燈"
