File: LargePW/LargePW.kicad_pcb (KiCad board)
At the start: 2 copper layers, 138.9 x 132.4 mm, 0 parts

Commit message: LargeMDほぼ完成
Parts:
- added C1: 1uF, Capacitor_SMD:C_0805_2012Metric_Pad1.18x1.45mm_HandSolder, F.Cu at (79.4, -96.8)
- added C2: 10000uF, Capacitor_THT:CP_Radial_D35.0mm_P10.00mm_SnapIn, F.Cu at (86.4, -140.0)
- added D1: CUS10F30, Diode_SMD:D_SOD-323_HandSoldering, F.Cu at (74.5, -96.8)
- added D2: CUS10F30, Diode_SMD:D_SOD-323_HandSoldering, F.Cu at (92.0, -96.8)
- added F1: Fuse, Fuse:Fuseholder_Blade_Mini_Keystone_3568, F.Cu at (75.8, -104.1)
- added H1: MountingHole_Pad, TestPoint:TestPoint_THTPad_D4.0mm_Drill2.0mm, F.Cu at (129.2, -102.6)
- added H2: MountingHole_Pad, TestPoint:TestPoint_THTPad_D4.0mm_Drill2.0mm, F.Cu at (137.7, -108.9)
- added H3: MountingHole, MountingHole:MountingHole_3.2mm_M3, F.Cu at (153.7, -123.7)
- added H4: MountingHole, MountingHole:MountingHole_3.2mm_M3, F.Cu at (141.4, -115.9)
- added H5: MountingHole, MountingHole:MountingHole_3.2mm_M3, F.Cu at (181.5, -154.3)
- added H6: MountingHole, MountingHole:MountingHole_3.2mm_M3, F.Cu at (169.1, -139.0)
- added J1: Conn_01x02_Female, Connector_Molex:Molex_SPOX_5267-02A_1x02_P2.50mm_Vertical, F.Cu at (128.7, -108.5)
- added J10: Conn_01x02_Female, Connector_AMASS:AMASS_XT30U-F_1x02_P5.0mm_Vertical, F.Cu at (144.4, -140.1)
- added J11: Conn_01x02_Female, Connector_AMASS:AMASS_XT30U-F_1x02_P5.0mm_Vertical, F.Cu at (93.1, -101.9)
- added J12: Conn_01x02_Female, Connector_AMASS:AMASS_XT30U-F_1x02_P5.0mm_Vertical, F.Cu at (144.4, -154.6)
- added J13: Conn_01x02_Female, Connector_AMASS:AMASS_XT30U-F_1x02_P5.0mm_Vertical, F.Cu at (144.4, -132.9)
- added J2: Conn_01x02_Female, Connector_AMASS:AMASS_XT30U-F_1x02_P5.0mm_Vertical, F.Cu at (141.1, -123.5)
- added J3: Conn_01x02_Female, Connector_AMASS:AMASS_XT30U-F_1x02_P5.0mm_Vertical, F.Cu at (156.6, -154.6)
- added J4: Conn_01x02_Female, Connector_AMASS:AMASS_XT30U-F_1x02_P5.0mm_Vertical, F.Cu at (144.4, -147.4)
- added J5: Conn_01x02_Female, Connector_AMASS:AMASS_XT30U-F_1x02_P5.0mm_Vertical, F.Cu at (128.8, -123.5)
- added J6: Conn_01x02_Female, Connector_AMASS:AMASS_XT30U-F_1x02_P5.0mm_Vertical, F.Cu at (105.4, -101.9)
- added J7: Conn_01x02_Female, Connector_AMASS:AMASS_XT30U-F_1x02_P5.0mm_Vertical, F.Cu at (168.9, -154.6)
- added J8: Conn_01x02_Female, Connector_AMASS:AMASS_XT30U-F_1x02_P5.0mm_Vertical, F.Cu at (156.6, -147.4)
- added J9: Conn_01x02_Female, Connector_AMASS:AMASS_XT30U-F_1x02_P5.0mm_Vertical, F.Cu at (128.8, -116.2)
- added K1: RAYEX-L90, Relay:TRV4-L-12V-Z-F, F.Cu at (125.2, -142.7)
- added MES1: Voltmeter_DC, Voltmeter:SuperSmallVoltmeter_twoline, F.Cu at (87.5, -115.1)
- added Q1: TJ60S04M3L, Package_TO_SOT_SMD:TO-252-3_TabPin2, F.Cu at (159.1, -131.7)
- added Q2: TJ60S04M3L, Package_TO_SOT_SMD:TO-252-3_TabPin2, F.Cu at (159.1, -139.7)
- added Q3: TJ60S04M3L, Package_TO_SOT_SMD:TO-252-3_TabPin2, F.Cu at (171.3, -147.0)
- added Q4: TJ60S04M3L, Package_TO_SOT_SMD:TO-252-3_TabPin2, F.Cu at (120.1, -101.5)
- added Q5: BSS138, Package_TO_SOT_SMD:SOT-23_Handsoldering, F.Cu at (112.8, -124.8)
- added R1: 10k, Resistor_SMD:R_0603_1608Metric_Pad0.98x0.95mm_HandSolder, F.Cu at (84.0, -97.0)
- added R2: 100k, Resistor_SMD:R_0603_1608Metric_Pad0.98x0.95mm_HandSolder, F.Cu at (82.8, -94.0)
- added R3: 510, Resistor_SMD:R_0603_1608Metric_Pad0.98x0.95mm_HandSolder, F.Cu at (74.1, -94.1)
- added R4: 510, Resistor_SMD:R_0603_1608Metric_Pad0.98x0.95mm_HandSolder, F.Cu at (87.2, -94.5)
- added R5: 10k, Resistor_SMD:R_0603_1608Metric_Pad0.98x0.95mm_HandSolder, F.Cu at (118.2, -125.9)
- added R6: 10k, Resistor_SMD:R_0603_1608Metric_Pad0.98x0.95mm_HandSolder, F.Cu at (78.5, -94.0)
- added SW1: SW_SPST, Rocker_Switch:DS-850K-S-ON, F.Cu at (114.1, -113.6)

Commit message: SmallMDほぼ完成
Parts:
- removed H3, H4, H5, H6: MountingHole, MountingHole:MountingHole_3.2mm_M3
- C1, D1, D2, Q5, R1, R2, R3, R4, R5, R6: moved to B.Cu
- moved J3 280.3 mm to (65.5, 110.5), turned to 180 degrees
- moved J4 255.4 mm to (79.0, 99.5), turned to 180 degrees
- moved J8 255.1 mm to (92.5, 99.5), turned to 180 degrees
- moved R5 246.5 mm to (41.0, 108.2), turned to -90 degrees
- moved Q5 245.0 mm to (37.5, 108.2)
- moved J12 239.4 mm to (101.7, 81.0), turned to -90 degrees
- moved J5 239.2 mm to (79.0, 110.5), turned to 180 degrees
- moved J10 238.5 mm to (101.7, 94.5), turned to -90 degrees
- moved J2 235.4 mm to (65.5, 99.5), turned to 180 degrees
- moved Q3 233.2 mm to (79.2, 67.2)
- moved J1 231.2 mm to (23.4, 97.3), turned to -90 degrees
- moved SW1 230.6 mm to (41.5, 105.2), turned to 90 degrees
- moved J9 229.6 mm to (92.5, 110.5), turned to 180 degrees
- moved J7 229.2 mm to (112.5, 67.5), turned to -90 degrees
- moved Q1 228.1 mm to (67.0, 77.0), turned to 180 degrees
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Other:
- board size 138.9 x 132.4 mm -> 100 x 100 mm

Commit message: DCDC回路図変更
Parts:
- added Q6: BSS138, Package_TO_SOT_SMD:SOT-23_Handsoldering, B.Cu at (30.5, 108.2)
- C1: footprint Capacitor_SMD:C_0805_2012Metric_Pad1.18x1.45mm_HandSolder -> Capacitor_SMD:C_0603_1608Metric_Pad1.08x0.95mm_HandSolder
- Q1, Q2, Q3, Q4: footprint Package_TO_SOT_SMD:TO-252-3_TabPin2 -> Package_TO_SOT_SMD:TO-252-2
- moved H1 2.61 mm to (64.8, 39.8)
- moved H2 2.37 mm to (53.8, 40.0)
Connections:
- D1 pad 1: 85 -> ESS
- D1 pad 2: GND -> RelaySW
- F1 pad 2: 30 -> /RelayIN
- J1 pad 1: 30 -> /RelayIN
- J1 pad 2: 85 -> ESS
- Q1 pad 2: 87 -> /RelayOUT
- Q2 pad 2: 87 -> /RelayOUT
- Q5 pad 1: Net-(Q5-Pad1) -> Net-(R6-Pad2)
- R6 pad 1: Net-(Q5-Pad1) -> GND
- R6 pad 2: GND -> Net-(R6-Pad2)
- SW1 pad 1: Net-(Q5-Pad1) -> Net-(R6-Pad2)
- SW1 pad 2: /S-S -> /RelayIN
Routing:
- added copper zone on F.Cu, net +12V
- added copper zone on F.Cu, net /RelayIN
- added copper zone on F.Cu, net /RelayOUT
- added copper zone on F.Cu, net /S-S
- added copper zone on B.Cu, net GND
- added copper zone on F.Cu, net GND
- added copper zone on F.Cu, net VDD
Other:
- outline, holes or cut-outs redrawn

Commit message: 回路図ほぼ完成
Other:
- board size 100 x 100 mm -> 200.4 x 332.8 mm

Commit message: 多分完成
Parts:
- added R7: 1k, Resistor_SMD:R_0603_1608Metric_Pad0.98x0.95mm_HandSolder, F.Cu at (132.6, 86.8)
- moved R1 77.5 mm to (108.3, 136.3), turned to -90 degrees
- moved R6 74.4 mm to (99.5, 143.5)
- moved D1 73.0 mm to (90.0, 135.8)
- moved J1 73.0 mm to (88.6, 130.1)
- moved Q6 72.8 mm to (96.4, 139.0), turned to 90 degrees
- moved MES1 72.2 mm to (105.0, 117.0)
- moved K1 71.9 mm to (103.2, 93.8)
- moved J2 71.1 mm to (127.5, 134.2)
- moved J4 71.1 mm to (141.0, 134.2)
- moved J8 71.1 mm to (154.5, 134.2)
- moved C1 71.0 mm to (107.8, 139.9)
- moved Q5 71.0 mm to (101.0, 139.9)
- moved R2 71.0 mm to (106.0, 139.9)
- moved R3 71.0 mm to (109.2, 139.9)
- moved R4 71.0 mm to (110.8, 139.9)
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Routing:
- net RelaySW: track 0.00 -> 67.5 mm
- net /RelayIN: track 0.00 -> 61.9 mm, vias 0 -> 162
- net Net-(Q3-Pad1): track 0.00 -> 59.4 mm, vias 0 -> 1
- net Net-(Q4-Pad1): track 0.00 -> 49.9 mm, vias 0 -> 1
- net /S-S: track 0.00 -> 49.5 mm, vias 0 -> 101
- net ESS: track 0.00 -> 44.8 mm
- net GND: track 0.00 -> 41.2 mm, vias 0 -> 266
- net VDD: track 0.00 -> 18.5 mm
- net Net-(Q5-Pad1): track 0.00 -> 10.4 mm
- net 主電源スイッチ: track 0.00 -> 6.25 mm
- net Net-(Q5-Pad3): track 0.00 -> 2.38 mm
- net /RelayOUT: vias 0 -> 198
- net +12V: vias 0 -> 58
- added copper zone on B.Cu, net +12V
- added copper zone on B.Cu, net /RelayIN
- added copper zone on B.Cu, net /RelayOUT
- added copper zone on B.Cu, net /S-S
Other:
- board size 200.4 x 332.8 mm -> 86 x 100 mm
- board text added: "Designed by @cat_nekonekone"
- board text added: "JLCJLCJLCJLC"
- board text added: "Tomoshibi"
- board text added: "燈"
