File: Mother_Ctrl/Mother_Ctrl.kicad_pcb (KiCad board)
At the start: 2 copper layers, 100 x 60 mm, 264 parts, among them J1 Conn_01x02_Male, J10 Conn_01x04_Male, J11 Conn_01x04_Male, J12 Conn_01x04_Male, J13 Conn_01x05_Male, J14 Conn_01x05_Male, J15 Conn_01x12_Female, J16 Conn_01x12_Female, J17 Conn_01x12_Female, J2 Conn_01x02_Female, J3 USB_C_Receptacle_USB2.0, J4 Conn_01x07_Female, J5 Conn_01x10_Male, J6 Conn_01x02_Male, J7 Conn_01x03_Male, J8 Conn_01x03_Male, J9 Conn_01x04_Male, Q1 MTP4835I3, Q10 SSM3J332R, Q11 S8050, Q12 S8050, Q13 SSM3J332R, Q14 S8050, Q15 SSM3J332R, Q16 S8050, Q17 SSM3J332R, Q18 S8050, Q19 SSM3J332R, Q2 BSS138, Q20 S8050, Q21 SSM3J332R, Q22 S8050, Q23 BSS138, Q24 BSS138, Q25 BSS138, Q26 BSS138, Q27 BSS138, Q28 BSS138, Q29 MTP4835I3, Q3 MTP4835I3, Q30 S8050, Q31 S8050, Q32 S8050, Q4 SSM3J332R, Q5 S8050, Q6 SSM3J332R, Q7 S8050, Q8 S8050, Q9 SSM3J332R, SW1 SW_SPDT, SW2 SW_SPST, SW3 SW_SPST, SW4 SW_DPDT_x2, SW5 SW_SPDT, SW6 SW_SPST, SW7 SW_SPST, U1 CH340E, U2 TWE-L-WX, U3 AZ1084CD-3.3, U4 STM32F446RETx, U5 BNO055, U6 MAX3485, U7 MAX3485, U8 MAX3485, Y1 16MHz, Y2 32.768kHz

Commit message: 回路図確定
Parts:
- moved R42 62.1 mm to (36.1, -19.7), turned to 0 degrees
- moved R37 60.4 mm to (27.0, -20.2), turned to 90 degrees
- moved R40 58.6 mm to (34.7, -16.0), turned to 90 degrees
- moved R38 58.3 mm to (32.0, -16.0), turned to 90 degrees
- moved R43 57.2 mm to (33.7, -16.0)
- moved R39 56.6 mm to (29.8, -15.7), turned to 180 degrees
- moved R102 49.2 mm to (22.9, -11.8)
- moved D38 42.6 mm to (16.3, -11.8), turned to 0 degrees
- moved D37 33.5 mm to (23.6, -20.2)
- moved D39 29.2 mm to (28.1, -11.8)
- moved C30 1.14 mm to (24.8, -11.2), turned to -90 degrees
Connections:
- J15 pad 12: VCC -> GND
- J15 pad 2: unconnected-(J15-Pad2) -> Slide_SW1
- J15 pad 3: unconnected-(J15-Pad3) -> Slide_SW2
- J15 pad 5: unconnected-(J15-Pad5) -> Volume
- J15 pad 7: unconnected-(J15-Pad7) -> Sensor1
- J15 pad 8: unconnected-(J15-Pad8) -> Sensor2
- J16 pad 11: GND -> VCC
- J16 pad 2: unconnected-(J16-Pad2) -> Tact_SW2
- J16 pad 3: unconnected-(J16-Pad3) -> Tact_SW0
- J16 pad 4: unconnected-(J16-Pad4) -> Tact_SW1
- J16 pad 6: unconnected-(J16-Pad6) -> Sensor3
- J16 pad 7: unconnected-(J16-Pad7) -> Conn_Detect
- U4 pad 10: unconnected-(U4-Pad10) -> Sensor2
- U4 pad 23: unconnected-(U4-Pad23) -> Sensor3
- U4 pad 24: unconnected-(U4-Pad24) -> Volume
- U4 pad 33: unconnected-(U4-Pad33) -> Tact_SW1
- U4 pad 34: unconnected-(U4-Pad34) -> Slide_SW2
- U4 pad 35: unconnected-(U4-Pad35) -> Tact_SW0
- U4 pad 36: unconnected-(U4-Pad36) -> Slide_SW1
- U4 pad 39: unconnected-(U4-Pad39) -> Tact_SW2
- U4 pad 8: unconnected-(U4-Pad8) -> Conn_Detect
- U4 pad 9: unconnected-(U4-Pad9) -> Sensor1
Routing:
- net Sensor1: track 0.00 -> 21.2 mm, vias 0 -> 1
- net Slide_SW1: track 0.00 -> 19.6 mm, vias 0 -> 1
- net Sensor2: track 0.00 -> 18.7 mm, vias 0 -> 2
- net Tact_SW2: track 0.00 -> 17.6 mm, vias 0 -> 1
- net Conn_Detect: track 0.00 -> 17.6 mm, vias 0 -> 1
- net unconnected-(U4-Pad9): track 17.5 -> 0.00 mm, vias 1 -> 0
- net Slide_SW2: track 0.00 -> 17.0 mm, vias 0 -> 1
- net unconnected-(U4-Pad36): track 16.2 -> 0.00 mm, vias 1 -> 0
- net unconnected-(U4-Pad10): track 15.8 -> 0.00 mm, vias 2 -> 0
- net Volume: track 0.00 -> 15.4 mm, vias 0 -> 1
- net unconnected-(U4-Pad8): track 14.3 -> 0.00 mm, vias 1 -> 0
- net unconnected-(U4-Pad39): track 14.1 -> 0.00 mm, vias 1 -> 0
- net Tact_SW0: track 0.00 -> 13.8 mm, vias 0 -> 1
- net unconnected-(U4-Pad34): track 13.8 -> 0.00 mm, vias 1 -> 0
- net unconnected-(U4-Pad24): track 12.2 -> 0.00 mm, vias 1 -> 0
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Other:
- board text removed: "ADC"
- board text removed: "LED"
- board text removed: "uart1"
- board text removed: "uart2"
- board text removed: "uart3"
- board text removed: "uart5"
- board text removed: "uart6"

Commit message: 多分完成
Parts:
- removed H1, H10, H12, H2, H3, H6, H9: MountingHole_Pad, TestPoint:TestPoint_Pad_1.5x1.5mm
- removed TP1, TP2, TP3, TP4: TestPoint, TestPoint:TestPoint_THTPad_D2.0mm_Drill1.0mm
- H11: moved to B.Cu
- moved H11 251.0 mm to (167.4, 81.1), turned to 180 degrees
- moved TP5 189.7 mm to (104.9, 126.0)
- moved C1 184.6 mm to (112.1, 125.1)
- moved C10 184.6 mm to (140.2, 89.9)
- moved C12 184.6 mm to (181.6, 127.8)
- moved C13 184.6 mm to (140.3, 106.1)
- moved C14 184.6 mm to (150.3, 103.3)
- moved C15 184.6 mm to (159.1, 106.5)
- moved C16 184.6 mm to (163.9, 103.3)
- moved C19 184.6 mm to (148.3, 101.3)
- moved C2 184.6 mm to (150.8, 113.3)
- moved C20 184.6 mm to (115.0, 102.6)
- moved C21 184.6 mm to (124.8, 89.8)
- moved C22 184.6 mm to (149.3, 100.8)
- moved C23 184.6 mm to (149.3, 90.1)
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Connections:
- U1 pad 4: Net-(H3-Pad1) -> unconnected-(U1-Pad4)
- U1 pad 5: Net-(H2-Pad1) -> unconnected-(U1-Pad5)
Routing:
- net GND: track 24.2 -> 1169.5 mm, vias 0 -> 515
- net +3.3V: track 396.0 -> 400.7 mm
- net Sensor0: track 24.9 -> 27.7 mm
- net LED0: track 10.7 -> 11.6 mm
- net LED1: track 13.7 -> 14.5 mm
- added copper zone on B.Cu, net GND
- added copper zone on F.Cu, net GND
Other:
- board text added: "+3.3V"
- board text added: "+5V"
- board text added: "3V3IND"
- board text added: "5VIND"
- board text added: "Analog"
- board text added: "BOOT0"
- board text added: "DIO11"
- board text added: "DIO16"
- board text added: "DIO17"
- board text added: "Designed by @cat_nekonekone"
- board text added: "GND"
- board text added: "JLCJLCJLCJLC"
- board text added: "NRST"
- board text added: "NeoPixel"
- board text added: "PA11"
- board text added: "PA12"
- board text added: "PA15"
- board text added: "PA5"
- board text added: "PA8"
- board text added: "PB2"
- board text added: "PB4"
- board text added: "PB9"
- board text added: "PC10"
- board text added: "PC11"
- board text added: "POWER"
- board text added: "PRG"
- board text added: "RST"
- board text added: "RX1:PA10"
- board text added: "RX2:PA3"
- board text added: "RX3:PC5"
- board text added: "RX5:PD2"
- board text added: "RX6:PC7"
- board text added: "SCL1:PB8"
- board text added: "SDA1:PB7"
- board text added: "TX1:PA9"
- board text added: "TX2:PA2"
- board text added: "TX3:PB10"
- board text added: "TX5:PC12"
- board text added: "TX6:PC6"
- board text added: "Tomoshibi"
- board text added: "[5VOUT]"
- board text added: "[Arm]"
- board text added: "[DAC]PA4"
- board text added: "[I2C]"
- board text added: "[LEDTape0]"
- board text added: "[LEDTape0]PA6"
- board text added: "[LEDTape1]PB0"
- board text added: "[LEDTape2]PB1"
- board text added: "[LEDTape3]PB6"
- board text added: "[NeoPixel]PB5"
- board text added: "[RS485a]"
- board text added: "[RS485b]"
- board text added: "[STLink]"
- board text added: "[Sensor0]"
- board text added: "[Sensor0]PC3"
- board text added: "[Sensor1]PC1"
- board text added: "[Sensor2]PC2"
- board text added: "[Sensor3]PA7"
- board text added: "[TweLite]"
- board text added: "[USB]"
- board text added: "[V_meas.]PA0"
- board text added: "[Volume]PC4"
- board text added: "[Write]"
- board text added: "⇔"
- board text added: "燈"
