File: Mother_Ctrl/Mother_Ctrl.kicad_sch (KiCad schematic)
At the start: 63 parts

Commit message: 回路図ほぼ完成
Parts:
- removed SW?: SW_SPDT_White, Slide_Switch:SW_Slide_SPDT_White, symbol Switch:SW_SPDT
- added C? (x2): 22pF, Capacitor_SMD:C_0603_1608Metric, symbol Device:C
- added C?: ADJ_ST, Capacitor_SMD:C_0603_1608Metric, symbol Device:C
- added C? (x17): 0.1uF, Capacitor_SMD:C_0402_1005Metric, symbol Device:C
- added C? (x2): 10uF, Capacitor_SMD:C_0805_2012Metric, symbol Device:C
- added C?: 22uF, Capacitor_SMD:C_0805_2012Metric, symbol Device:C
- added C? (x3): 1uF, Capacitor_SMD:C_0402_1005Metric, symbol Device:C
- added C?: 4.7uF, Capacitor_SMD:C_0603_1608Metric, symbol Device:C
- added D? (x20): 1N5819WS, Diode_SMD:D_SOD-323_HandSoldering, symbol Device:D_Schottky
- added D?: MA10EB045, Diode_Schottky:DO-221BC, symbol Device:D_Schottky
- added D? (x6): Red, LED_SMD:LED_0603_1608Metric_Pad1.05x0.95mm_HandSolder, symbol Device:LED
- added D? (x3): Yellow, LED_SMD:LED_0603_1608Metric_Pad1.05x0.95mm_HandSolder, symbol Device:LED
- added D?: D_Zener, Diode_SMD:D_SOD-323_HandSoldering, symbol Device:D_Zener
- added D?: D, Diode_SMD:D_SOD-123, symbol Device:D
- added H? (x9): MountingHole_Pad, TestPoint:TestPoint_Pad_1.5x1.5mm, symbol Mechanical:MountingHole_Pad
- added J?: USB_C_Receptacle_USB2.0, USB_DIP:USB_C(simple), symbol Connector:USB_C_Receptacle_USB2.0
- added J? (x2): Conn_01x04_Male, Connector_Molex:Molex_SPOX_5267-04A_1x04_P2.50mm_Vertical, symbol Connector:Conn_01x04_Male
- added J? (x2): Conn_01x04_Male, Connector_Molex:Molex_SPOX_5268-04A_1x04_P2.50mm_Horizontal, symbol Connector:Conn_01x04_Male
- added J? (x2): Conn_01x03_Male, Connector_Molex:Molex_SPOX_5268-03A_1x03_P2.50mm_Horizontal, symbol Connector:Conn_01x03_Male
- added J?: Conn_01x02_Male, Connector_Molex:Molex_SPOX_5267-02A_1x02_P2.50mm_Vertical, symbol Connector:Conn_01x02_Male
- added J?: Conn_01x07_Female, Connector_PinSocket_2.54mm:PinSocket_1x07_P2.54mm_Horizontal, symbol Connector:Conn_01x07_Female
- added J?: Conn_01x10_Female, Connector_IDC:IDC-Header_2x05_P2.54mm_Horizontal, symbol Connector:Conn_01x10_Female
- added JP? (x2): Jumper_2_Open, Connector_PinHeader_2.54mm:PinHeader_1x02_P2.54mm_Vertical, symbol Jumper:Jumper_2_Open
- added MD?: OKL-T/6-W12N-C, DCDC_Regulator:MURATA_OKL-T-6-W12N-C, symbol DCDC_Regulator:OKL-T/6-W12N-C
- added Q? (x9): S8050, Package_TO_SOT_SMD:SOT-23, symbol Device:Q_PNP_BEC
- added Q? (x6): BSS138, Package_TO_SOT_SMD:SOT-23, symbol Device:Q_NMOS_GSD
- added Q?: MTP4835I3, Package_TO_SOT_SMD:TO-252-3_TabPin2, symbol Device:Q_PMOS_GDS
- added Q? (x5): SSM3J332R, Package_TO_SOT_SMD:SOT-23W, symbol Device:Q_PMOS_GSD
- added R? (x42): 10k, Resistor_SMD:R_0402_1005Metric, symbol Device:R
- added R? (x11): 1k, Resistor_SMD:R_0402_1005Metric, symbol Device:R
- added R? (x2): 5.1k, Resistor_SMD:R_0402_1005Metric, symbol Device:R
- added R? (x2): 100k, Resistor_SMD:R_0402_1005Metric, symbol Device:R
- added R? (x2): 120, Resistor_SMD:R_0402_1005Metric, symbol Device:R
- added R? (x3): 7.5k, Resistor_SMD:R_0603_1608Metric, symbol Device:R
- added R? (x6): 2.2k, Resistor_SMD:R_0402_1005Metric, symbol Device:R
- added R? (x3): 20k, Resistor_SMD:R_0402_1005Metric, symbol Device:R
- added R?: 1.2k, Resistor_SMD:R_0402_1005Metric, symbol Device:R
- added R? (x2): PullUp, Resistor_SMD:R_0603_1608Metric_Pad0.98x0.95mm_HandSolder, symbol Device:R
- added R?: 10, Resistor_SMD:R_0402_1005Metric, symbol Device:R
- added R? (x2): PullUP?, Resistor_SMD:R_0603_1608Metric, symbol Device:R
- added R?: 330, Resistor_SMD:R_0402_1005Metric, symbol Device:R
- added SW? (x2): SW_DPDT_x2, Button_Switch_THT:SW_CuK_JS202011CQN_DPDT_Straight, symbol Switch:SW_DPDT_x2
- added SW? (x4): SW_SPST, Button_Switch_SMD:SW_Push_1P1T_NO_Vertical_Wuerth_434133025816, symbol Switch:SW_SPST
- added SW?: SW_SPDT, Slide_Switch:3P_SPDT_SlideSwitch, symbol Switch:SW_SPDT
- added SW?: SW_SPDT, Toggle_Switch:3P_SPDT_5Pin_ToggleSwitch, symbol Switch:SW_SPDT
- added U?: TWE-L-WX, RF_Module:MonoWireless_TWE-L-WX, symbol RF_ZigBee:TWE-L-WX
- added U?: CH340E, Package_SO:MSOP-10_3x3mm_P0.5mm, symbol Interface_USB:CH340E
- added U?: NJU6319AE, Package_SO:SOP-8_3.9x4.9mm_P1.27mm, symbol CrystalOSC_Control:NJU6319AE
- added U?: STM32F446RETx, Package_QFP:LQFP-64_10x10mm_P0.5mm, symbol MCU_ST_STM32F4:STM32F446RETx
- added U? (x3): MAX3485, Package_SO:SOP-8_3.9x4.9mm_P1.27mm, symbol Interface_UART:MAX3485
- added U?: BNO055, BNO055:BNO055, symbol Sensor_Motion:BNO055
- added Y?: 16MHz, Crystal:Crystal_SMD_3225-4Pin_3.2x2.5mm_HandSoldering, symbol Device:Crystal_GND24
- added Y?: 32.768kHz, Crystal:Crystal_SMD_3215-2Pin_3.2x1.5mm, symbol Device:Crystal
Connections:
- net +3.3V: now also C?.1, C?.1, C?.1, C?.1, C?.1, C?.1, C?.1, C?.1, C?.1, C?.1, C?.1, C?.2, D?.1 (K), D?.1 (K), D?.1 (K), D?.1 (K), D?.1 (K), Q?.1 (G), Q?.1 (G), Q?.1 (G), Q?.1 (G), Q?.1 (G), Q?.2 (E), Q?.2 (E), Q?.2 (E), Q?.2 (E), Q?.2 (E), Q?.2 (S), Q?.2 (S), R?.1, R?.1, R?.1, R?.1, R?.1, R?.1, R?.1, R?.2, R?.2, R?.2, R?.2, R?.2, R?.2, SW?.2 (B), SW?.2 (B), U?.1 (VBAT), U?.1 (~{CONT}), U?.13 (VDDA), U?.19 (VDD), U?.3 (VDD), U?.32 (VDD), U?.48 (VDD), U?.5 (VCC), U?.64 (VDD), U?.8 (VCC), U?.8 (VCC), U?.8 (VCC), U?.8 (VDD); no longer D?.1 (K), Q?.2 (E), Q?.2 (E), Q?.2 (S), Q?.2 (S), R?.2
- net +5V: now also D?.1 (K), Q?.2 (E), Q?.2 (E), Q?.2 (S), Q?.2 (S), R?.2, D?.2 (A), D?.2 (A), D?.2 (A), D?.2 (A), D?.2 (A), J?.2 (Pin_2), J?.2 (Pin_2), Q?.2 (E), Q?.3 (D)
- net 3.3VBUS: now also C?.1, J?.1 (Pin_1), Q?.2 (S), R?.2; no longer Q?.2 (S), R?.2
- net 3.3VSYS: now also C?.1, Q?.2 (S), R?.1, R?.1, R?.1; no longer C?.1, Q?.2 (S), R?.1, R?.1, R?.1
- net 3.3V_IND: now also Q?.2 (E), Q?.3 (D), Q?.3 (D), R?.2; no longer Q?.2 (E), Q?.3 (D), Q?.3 (D), R?.2
- net GND: now also C?.1, C?.1, C?.1, C?.1, C?.1, C?.1, C?.2, C?.2, C?.2, C?.2, C?.2, C?.2, C?.2, C?.2, C?.2, C?.2, C?.2, C?.2, C?.2, C?.2, C?.2, C?.2, C?.2, C?.2, C?.2, C?.2, D?.1 (K), D?.1 (K), D?.1 (K), D?.1 (K), D?.1 (K), D?.1 (K), D?.1 (K), D?.1 (K), D?.1 (K), D?.2 (A), J?.1 (Pin_1), J?.1 (Pin_1), J?.1 (Pin_1), J?.1 (Pin_1), J?.1 (Pin_1), J?.1 (Pin_1), J?.1 (Pin_1), J?.1 (Pin_1), J?.2 (Pin_2), J?.2 (Pin_2), J?.2 (Pin_2), J?.2 (Pin_2), J?.4 (Pin_4), J?.A1 (GND), J?.S1 (SHIELD), MD?.1 (ON/OFF), MD?.3 (GND), MD?.7 (GND), Q?.2 (S), R?.1, R?.1, R?.1, R?.1, R?.1, R?.1, R?.1, R?.1, R?.1, R?.1, R?.1, R?.1, R?.1, R?.2, R?.2, R?.2, R?.2, R?.2, R?.2, R?.2, R?.2, R?.2, R?.2, R?.2, R?.2, R?.2, R?.2, R?.2, R?.2, R?.2, R?.2, R?.2, R?.2, R?.2, R?.2, R?.2, R?.2, R?.2, R?.2, R?.2, R?.2, SW?.2 (B), SW?.2 (B), SW?.2 (B), U?.12 (VSSA), U?.18 (VSS), U?.2 (GND), U?.20 (GND), U?.22 (ADC2/AI3), U?.23 (ADC1/AI1), U?.28 (GND), U?.28 (PB2), U?.3 (GND), U?.30 (GND), U?.31 (GND), U?.31 (VSS), U?.32 (GND), U?.4 (VSS), U?.47 (VSS), U?.5 (GND), U?.5 (GND), U?.5 (GND), U?.63 (VSS), Y?.2, Y?.4
- net S-S: now also SW?.2 (B)
- net VCC: now also C?.1, D?.1 (K), D?.1 (K), MD?.2 (VIN), R?.1
- net VDD: now also D?.2 (A), Q?.3 (S), R?.2
- net V_Measure: now also U?.27 (PB1)
- net 主電源スイッチ: now also SW?.1 (A)
- new net: J?.A5 (CC1), R?.2
- new net: J?.A6 (D+), U?.1 (UD+)
- new net: J?.A7 (D-), U?.2 (UD-)
- new net: J?.B5 (CC2), R?.2
- new net: Q?.1 (B), Q?.1 (B), Q?.3 (C), R?.2 (x3)
- new net: H?.1, Q?.1 (G), Q?.3 (C), R?.2
- new net: C?.2, H?.1, Q?.1 (G), R?.2
- new net: D?.2 (A), R?.1 (x9)
- new net: C?.2, Q?.1 (G), R?.1, R?.2
- new net: JP?.2 (B), R?.1 (x2)
- new net: Q?.1 (B), R?.1 (x3)
- new net: Q?.3 (C), R?.1, U?.2 (~{RE}), U?.3 (DE) (x3)
- new net: D?.1 (K), R?.2 (x5)
- new net: Q?.2 (E), Q?.3 (D), Q?.3 (D)
- new net: Q?.1 (G), Q?.3 (D), R?.1
- new net: C?.1, U?.10 (V3)
- new net: H?.1, U?.4 (~{RTS})
- new net: H?.1, U?.5 (~{CTS})
- new net: R?.2, U?.6 (TNOW)
- new net: Q?.1 (G), Q?.3 (C), R?.2 (x2)
- new net: U?.2 (XT), Y?.1
- new net: U?.3 (~{XT}), Y?.3
- new net: J?.2 (Pin_2), Q?.2 (E), Q?.2 (S)
- new net: C?.2, U?.30 (VCAP_1)
- new net: R?.1, R?.2, U?.7 (B)
- new net: R?.1, R?.1
- new net: MD?.6 (TRIM), R?.1
- new net: R?.2, R?.2
- new net: MD?.10 (PGOOD), R?.1
- new net 5VBUS: Q?.2 (S), R?.2
- new net 5VSYS: C?.1, C?.1, D?.2 (A), MD?.4 (VOUT), MD?.5 (SENSE), Q?.2 (S), R?.1, R?.1, R?.1, R?.2, R?.2
- new net 5V_IND: Q?.2 (E), Q?.3 (D), Q?.3 (D), R?.2
- new net BOOT0: H?.1, R?.1, SW?.1 (A), U?.60 (BOOT0)
- new net DIP_SW0: D?.2 (A), D?.2 (A)
- new net DIP_SW1: D?.2 (A), D?.2 (A), U?.41 (PA8)
- new net DIP_SW2: D?.2 (A), D?.2 (A), U?.44 (PA11)
- new net DIP_SW3: D?.2 (A), D?.2 (A), U?.45 (PA12)
- new net DIP_SW4: D?.2 (A), D?.2 (A), U?.50 (PA15)
- new net F446USBRX: SW?.6 (C), U?.9 (RXD)
- new net F446USBTX: SW?.3 (C), U?.8 (TXD)
- new net F446_DIP0: D?.1 (K), R?.1
- new net F446_DIP1: D?.1 (K), R?.1
- new net F446_DIP2: D?.1 (K), R?.1
- new net F446_DIP3: D?.1 (K), R?.1
- new net F446_DIP4: D?.1 (K), R?.1
- new net Gyro_RST: U?.11 (~{RESET})
- new net HSE_IN: U?.5 (FOUT)
- new net I2C1_SCL: R?.2, U?.19 (COM1), U?.61 (PB8)
- new net I2C1_SDA: R?.2, U?.20 (COM0), U?.62 (PB9)
- new net LED0: R?.2
- new net LED1: R?.2, U?.34 (PB13)
- new net LED2: R?.2, U?.35 (PB14)
- new net LED3: U?.36 (PB15)
- new net LEDTape0_H: J?.3 (Pin_3), Q?.3 (D), R?.1
- new net LEDTape0_L: Q?.2 (S), R?.1
- new net LEDTape1_H: Q?.3 (D), R?.1
- new net LEDTape1_L: Q?.2 (S), R?.1
- new net LEDTape2_H: Q?.3 (D), R?.1
- new net LEDTape2_L: Q?.2 (S), R?.1
- new net LEDTape3_H: Q?.3 (D), R?.1
- new net LEDTape3_L: Q?.2 (S), R?.1
- new net LSE_IN: C?.2, Y?.2
- new net LSE_OUT: C?.2, Y?.1
- new net MainRX1_F446WriteTX: SW?.2 (B), U?.43 (PA10)
- new net MainRX4_TweTX1: U?.14 (DIO14/SCL), U?.15 (PA1)
- new net MainRX5_RS485TX: U?.54 (PD2)
- new net MainRX6_ArmTX: U?.38 (PC7)
- new net MainRX_ArmTX: U?.1 (RO)
- new net MainRX_RS485aTX: U?.1 (RO)
- new net MainRX_RS485bTX: U?.1 (RO)
- new net MainTX1_F446WriteRX: SW?.5 (B), U?.42 (PA9)
- new net MainTX4_TweRX1: U?.14 (PA0), U?.17 (DIO15/SDA)
- new net MainTX5_RS485RX: U?.53 (PC12)
- new net MainTX6_ArmRX: U?.37 (PC6)
- new net MainTX_ArmRX: R?.2, U?.4 (DI)
- new net MainTX_RS485aRX: R?.2, U?.4 (DI)
- new net MainTX_RS485bRX: R?.2, U?.4 (DI)
- new net MonitorLED0: R?.2
- new net MonitorLED1: R?.2
- new net NRST: C?.1, H?.1, J?.6 (Pin_6), SW?.1 (A), U?.7 (NRST)
- new net NeoPixel1_L: U?.22 (PA6)
- new net NeoPixel2_L: U?.21 (PA5)
- new net NeoPixel3_L: U?.39 (PC8)
- new net NeoPixel4_L: U?.40 (PC9)
- new net NeoPixel_H: Q?.3 (D), R?.1
- new net NeoPixel_L: Q?.2 (S), R?.1
- new net PRG: H?.1, J?.3 (Pin_3), R?.2, SW?.1 (A), U?.2 (DO1/PWM3)
- new net RS485_Arm: U?.6 (A)
- new net RS485a_A: J?.3 (Pin_3), J?.3 (Pin_3), JP?.1 (A), R?.2, U?.6 (A)
- new net RS485a_B: J?.4 (Pin_4), J?.4 (Pin_4), R?.1, R?.2, U?.7 (B)
- new net RS485b_A: J?.3 (Pin_3), J?.3 (Pin_3), JP?.1 (A), R?.2, U?.6 (A)
- new net RS485b_B: J?.4 (Pin_4), J?.4 (Pin_4), R?.1, R?.2, U?.7 (B)
- new net RST: C?.1, D?.2 (A), H?.1, J?.5 (Pin_5), R?.2, SW?.1 (A), U?.21 (~{RESET})
- new net SET: J?.7 (Pin_7), U?.13 (DIO12/DI1)
- new net STLinkRX: J?.9 (Pin_9), SW?.4 (A)
- new net STLinkTX: J?.8 (Pin_8), SW?.1 (A)
- new net SWO: J?.7 (Pin_7), U?.55 (PB3)
- new net Sensor0: D?.2 (A), H?.1, J?.3 (Pin_3)
- new net Sensor1: D?.2 (A), U?.8 (PC0)
- new net Sensor2: D?.2 (A), U?.9 (PC1)
- new net Sensor3: D?.2 (A), U?.10 (PC2)
- new net Sensor4: U?.11 (PC3)
- new net Servo_SW: Q?.1 (G), R?.2
- new net Slide_SW0: R?.1, SW?.1 (A)
- new net Slide_SW1: R?.1
- new net Slide_SW2: R?.1
- new net Slide_Switch1: U?.51 (PC10)
- new net Slide_Switch2: U?.52 (PC11)
- new net Speaker: U?.29 (PB10)
- new net TCK: J?.3 (Pin_3), U?.49 (PA14)
- new net TMS: J?.5 (Pin_5), U?.46 (PA13)
- new net Tact_SW0: R?.1
- new net Tact_SW1: R?.1
- new net Tact_SW2: R?.1
- new net Tact_Switch1: U?.57 (PB5)
- new net Tact_Switch2: U?.58 (PB6)
- new net Tact_Switch3: U?.59 (PB7)
- new net TweRST_Sig: D?.1 (K)
- new net TweWriteRX_TweTX0: J?.2 (Pin_2), U?.8 (DIO6/TX)
- new net TweWriteTX_TweRX0: J?.4 (Pin_4), U?.9 (DIO7/RX)
- new net Twe_DIP0: D?.1 (K), R?.1
- new net Twe_DIP1: D?.1 (K), R?.1
- new net Twe_DIP2: D?.1 (K), R?.1
- new net Twe_DIP3: D?.1 (K), R?.1
- new net Twe_DIP4: D?.1 (K), R?.1
- new net Twe_LED0: R?.2
- new net Twe_LED1: R?.2, U?.11 (DIO9/DO4)
- new net Twe_LED2: R?.2, U?.10 (DIO8/PWM4)
- new net Twe_SW1: U?.15 (DIO13/DI2)
- new net Twe_SW2: U?.18 (DIO16/DI4)
- new net VBUS: C?.1, C?.2, J?.A4 (VBUS), U?.7 (VCC)
- new net Vdrive: C?.1, C?.1, Q?.2 (D)
- new net Volume: R?.1
- no-connect marks 1 -> 37
Other:
- note added: "5V出力"
- note added: "5V生成"
- note added: "ADC過電圧保護"
- note added: "BNO055"
- note added: "BOOT0"
- note added: "Conn"
- note added: "Conn to LEDTape"
- note added: "Conn to sensor"
- note added: "DIP分岐"
- note added: "F446RE"
- note added: "HSE"
- note added: "I/O"
- note added: "Jumper"
- note added: "LED"
- note added: "LEDTape"
- note added: "LSE"
- note added: "MAX3485"
- note added: "NRST"
- note added: "PRG"
- note added: "PullDOWN"
- note added: "RS485a"
- note added: "RS485b"
- note added: "STLink"
- note added: "TweLite"
- note added: "TweLiteR3"
- note added: "USB-C"
- note added: "サーボ"
- note added: "サーボ過電圧保護"
- note added: "スライドスイッチ"
- note added: "パスコン"
- note added: "マイコン"
- note added: "リセット"
- note added: "レベル変換"
- note added: "レベル変換/LEDTape"
- note added: "レベル変換/NeoPixel"
- note added: "書き込み"
- note added: "理想ダイオード/5VSYS"
- note added: "監視LED"
- note added: "電源切替/USB"
- moved on the sheet: C?, D?, H?, J?, Q?, R?, TP?, U?

Commit message: Pole,Panelほぼ完成
Parts:
- removed D?: D, Diode_SMD:D_SOD-123, symbol Device:D
- removed J?: USB_C_Receptacle_USB2.0, USB_DIP:USB_C(simple), symbol Connector:USB_C_Receptacle_USB2.0
- removed J?: Conn_01x10_Female, Connector_IDC:IDC-Header_2x05_P2.54mm_Horizontal, symbol Connector:Conn_01x10_Female
- added D?: 1N5819WS, Diode_SMD:D_SOD-323_HandSoldering, symbol Device:D_Schottky
- added J?: USB_C_Receptacle_USB2.0, Connector_USB:USB_C_Receptacle_G-Switch_GT-USB-7010ASV, symbol Connector:USB_C_Receptacle_USB2.0
- added J?: Conn_01x10_Male, BoxHeader_1.27mm:BoxHeader_2x05_P1.27mm_Vertical_SMD, symbol Connector:Conn_01x10_Male
- J? (x2): footprint Connector_Molex:Molex_SPOX_5267-04A_1x04_P2.50mm_Vertical -> Connector_Molex:Molex_SPOX_5268-04A_1x04_P2.50mm_Horizontal
- J?: footprint Connector_Molex:Molex_SPOX_5267-02A_1x02_P2.50mm_Vertical -> Connector_Molex:Molex_SPOX_5268-02A_1x02_P2.50mm_Horizontal
Connections:
- net VBUS is gone; now on net 5VBUS: C?.1, C?.2, U?.7 (VCC)
- net 3.3VBUS: now also J?.1 (Pin_1)
- net 5VBUS: now also J?.A4 (VBUS), J?.A9 (VBUS), J?.B4 (VBUS), J?.B9 (VBUS)
- net 5VSYS: now also D?.2 (A)
- net GND: now also J?.4 (Pin_4), J?.A1 (GND), J?.A12 (GND), J?.B1 (GND), J?.B12 (GND), J?.S1 (SHIELD)
- net NRST: now also J?.6 (Pin_6)
- net STLinkRX: now also J?.9 (Pin_9)
- net STLinkTX: now also J?.8 (Pin_8)
- net SWO: now also J?.7 (Pin_7)
- net TCK: now also J?.3 (Pin_3)
- net TMS: now also J?.5 (Pin_5)
- net VCC: now also D?.1 (K)
- net at R?.2: now also J?.A5 (CC1)
- net at U?.1 (UD+): now also J?.A6 (D+), J?.B6 (D+)
- net at U?.2 (UD-): now also J?.A7 (D-), J?.B7 (D-)
- net at R?.2: now also J?.B5 (CC2)
- no-connect marks 37 -> 39

Commit message: Mother_Ctrl回路図プロット
Parts:
- removed C?: 0.1uF, Capacitor_SMD:C_0402_1005Metric, symbol Device:C
- removed D?: SS2040FL, Diode_SMD:D_SOD-123, symbol Device:D_Schottky
- removed D?: Red, LED_SMD:LED_0603_1608Metric_Pad1.05x0.95mm_HandSolder, symbol Device:LED
- removed R? (x2): 1k, Resistor_SMD:R_0402_1005Metric, symbol Device:R
- removed U?: NJU6319AE, Package_SO:SOP-8_3.9x4.9mm_P1.27mm, symbol CrystalOSC_Control:NJU6319AE
- added C15, C16: 22pF, Capacitor_SMD:C_0603_1608Metric, symbol Device:C
- added H12: MountingHole_Pad, TestPoint:TestPoint_Pad_1.5x1.5mm, symbol Mechanical:MountingHole_Pad
- added J13, J14: Conn_01x05_Male, Connector_Molex:Molex_SPOX_5268-05A_1x05_P2.50mm_Horizontal, symbol Connector:Conn_01x05_Male
- added J15, J16, J17: Conn_01x12_Female, Connector_PinSocket_2.54mm:PinSocket_1x12_P2.54mm_Vertical, symbol Connector:Conn_01x12_Female
- added R102, R103: 10k, Resistor_SMD:R_0402_1005Metric, symbol Device:R
- added R64: PullUP?, Resistor_SMD:R_0603_1608Metric, symbol Device:R
- H4, H5: renamed from H?; footprint TestPoint:TestPoint_Pad_1.5x1.5mm -> TestPoint:TestPoint_Pad_1.0x1.0mm
- Q1, Q29, Q3: renamed from Q?; footprint Package_TO_SOT_SMD:TO-252-3_TabPin2 -> Package_TO_SOT_SMD:TO-252-2
- R37: renamed from R?; value 10k -> 100k
- R84, R85: renamed from R?; value PullUp -> PullUP
- U3: renamed from U?; footprint Package_TO_SOT_SMD:TO-252-3_TabPin2 -> Package_TO_SOT_SMD:TO-252-2
- gave numbers to parts that had none: 244
Connections:
- net MainRX5_RS485TX is gone; now on net MainRX5_TweTX1: U4.54 (PD2)
- net MainRX_ArmTX is gone; now on net MainRX2_ArmTX: U8.1 (RO)
- net MainRX_RS485aTX is gone; now on net MainRX6_RS485aTX: U6.1 (RO)
- net MainRX_RS485bTX is gone; now on net MainRX3_RS485bTX: U7.1 (RO)
- net MainTX5_RS485RX is gone; now on net MainTX5_TweRX1: U4.53 (PC12)
- net MainTX_ArmRX is gone; now on net MainTX2_ArmRX: R92.2, U8.4 (DI)
- net MainTX_RS485aRX is gone; now on net MainTX6_RS485aRX: R88.2, U6.4 (DI)
- net NeoPixel1_L is gone; now on net LEDTape0_L: U4.22 (PA6)
- net NeoPixel2_L is gone; now on net MonitorLED1: U4.21 (PA5)
- net NeoPixel4_L is gone; now on net Gyro_RST: U4.40 (PC9)
- net Sensor4 is gone; now on net Sensor0: U4.11 (PC3)
- net Slide_Switch1 is gone; now on net F446_DIP3: U4.51 (PC10)
- net Slide_Switch2 is gone; now on net F446_DIP4: U4.52 (PC11)
- net Speaker is gone; now on net MainTX3_RS485bRX: U4.29 (PB10)
- net Tact_Switch1 is gone; now on net NeoPixel_L: U4.57 (PB5)
- net Tact_Switch2 is gone; now on net LEDTape3_L: U4.58 (PB6)
- net Tact_Switch3 is gone; now on net I2C1_SDA: U4.59 (PB7)
- net Twe_SW1 is gone; now on net Twe_DIP4: U2.15 (DIO13/DI2)
- net Twe_SW2 is gone; now on net Twe_LED1: U2.18 (DIO16/DI4)
- net +3.3V: now also J16.12 (Pin_12), R64.2
- net +5V: now also C13.1, D20.1 (K), R44.1, R71.2, U3.3 (VI), J15.10 (Pin_10), J16.10 (Pin_10)
- net 3.3VSYS: no longer R71.2
- net 5V_IND: now also R70.2
- net BOOT0: now also J15.4 (Pin_4)
- net Conn_Detect: now also R102.1
- net DIP_SW0: now also J17.6 (Pin_6)
- net DIP_SW1: now also J17.7 (Pin_7); no longer U4.41 (PA8)
- net DIP_SW2: now also J17.8 (Pin_8); no longer U4.44 (PA11)
- net DIP_SW3: now also J17.9 (Pin_9); no longer U4.45 (PA12)
- net DIP_SW4: now also J17.10 (Pin_10); no longer U4.50 (PA15)
- net F446_DIP0: now also U4.45 (PA12)
- net F446_DIP1: now also U4.44 (PA11)
- net F446_DIP2: now also U4.41 (PA8)
- net GND: now also C15.1, C16.1, J13.1 (Pin_1), J13.2 (Pin_2), J13.3 (Pin_3), J14.1 (Pin_1), J14.2 (Pin_2), J14.3 (Pin_3), J15.11 (Pin_11), J15.9 (Pin_9), J16.11 (Pin_11), J16.9 (Pin_9), R102.2, R103.2; no longer U4.28 (PB2)
- net HSE_IN: now also U4.5 (PH0), Y1.1, C15.2
- net I2C1_SCL: now also J17.2 (Pin_2)
- net I2C1_SDA: now also J17.1 (Pin_1); no longer U4.62 (PB9)
- net LED0: now also U4.56 (PB4)
- net LED1: now also U4.50 (PA15); no longer U4.34 (PB13)
- net LEDTape1_H: now also J16.1 (Pin_1)
- net LEDTape1_L: now also U4.26 (PB0)
- net LEDTape2_H: now also J15.1 (Pin_1)
- net LEDTape2_L: now also U4.27 (PB1)
- net LEDTape3_H: now also J17.4 (Pin_4)
- net LSE_IN: now also U4.3 (PC14)
- net LSE_OUT: now also U4.4 (PC15)
- net MonitorLED0: now also U4.28 (PB2), H12.1, J16.5 (Pin_5), R103.1
- net MonitorLED1: now also J15.6 (Pin_6)
- net NRST: now also J17.5 (Pin_5)
- net NeoPixel_H: now also J17.3 (Pin_3)
- net PRG: now also J17.11 (Pin_11)
- net RS485_Arm: now also J13.5 (Pin_5), J14.5 (Pin_5)
- net RST: now also J17.12 (Pin_12)
- net Sensor1: no longer U4.8 (PC0)
- net Sensor2: no longer U4.9 (PC1)
- net Sensor3: no longer U4.10 (PC2)
- net Servo_SW: now also U4.15 (PA1)
- net Slide_SW0: now also U4.62 (PB9)
- net TweRST_Sig: now also U4.2 (PC13)
- net Twe_DIP0: now also U2.7 (DIO5/PWM1)
- net Twe_DIP1: now also U2.11 (DIO9/DO4)
- net Twe_DIP2: now also U2.10 (DIO8/PWM4)
- net Twe_DIP3: now also U2.12 (DIO10/M1)
- net Twe_LED0: now also U2.19 (DIO17/BPS)
- net Twe_LED1: no longer U2.11 (DIO9/DO4)
- net Twe_LED2: now also U2.16 (DIO11/DI3); no longer U2.10 (DIO8/PWM4)
- net VCC: now also J15.12 (Pin_12); no longer C13.1, D20.1 (K), R44.1, R70.2, U3.3 (VI)
- net V_Measure: now also U4.14 (PA0); no longer U4.27 (PB1)
- net Vdrive: now also J13.4 (Pin_4), J14.4 (Pin_4)
- net at U2.1 (DO0/PWM2): now also R64.1
- net HSE_OUT: now reaches Y1.3
- net HSE_OUT: now also U4.6 (PH1), C16.2
- net MainTX2_ArmRX: now reaches U4.16 (PA2)
- net MainRX2_ArmTX: now reaches U4.17 (PA3)
- net DAC: now reaches U4.20 (PA4)
- net DAC: now also J16.8 (Pin_8)
- net MainRX3_RS485bTX: now reaches U4.25 (PC5)
- net LED2: no longer names the net of U4.35 (PB14)
- net LED3: no longer names the net of U4.36 (PB15)
- net MainRX4_TweTX1 renamed MainRX5_TweTX1
- net MainRX5_TweTX1: no longer U4.15 (PA1)
- net MainRX6_ArmTX renamed MainRX6_RS485aTX
- net MainTX4_TweRX1 renamed MainTX5_TweRX1
- net MainTX5_TweRX1: no longer U4.14 (PA0)
- net MainTX6_ArmRX renamed MainTX6_RS485aRX
- net MainTX_RS485bRX renamed MainTX3_RS485bRX
- net NeoPixel3_L: no longer names the net of U4.39 (PC8)
- no-connect marks 39 -> 20
Other:
- note added: "FETのゲートの間にダイオードつけるのありかも"
- note added: "基板間コネクタ"
- moved on the sheet: C13, C14, C36, C37, D20, H6, J6, Q11, Q8, Q9, R28, R31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

Commit message: 回路図確定
Connections:
- net Conn_Detect: now also J16.7 (Pin_7), U4.8 (PC0)
- net GND: now also J15.12 (Pin_12); no longer J16.11 (Pin_11)
- net Sensor1: now also J15.7 (Pin_7), U4.9 (PC1)
- net Sensor2: now also J15.8 (Pin_8), U4.10 (PC2)
- net Sensor3: now also J16.6 (Pin_6), U4.23 (PA7)
- net Slide_SW1: now also J15.2 (Pin_2), U4.36 (PB15)
- net Slide_SW2: now also J15.3 (Pin_3), U4.34 (PB13)
- net Tact_SW0: now also J16.3 (Pin_3), U4.35 (PB14)
- net Tact_SW1: now also J16.4 (Pin_4), U4.33 (PB12)
- net Tact_SW2: now also J16.2 (Pin_2), U4.39 (PC8)
- net VCC: now also J16.11 (Pin_11); no longer J15.12 (Pin_12)
- net Volume: now also J15.5 (Pin_5), U4.24 (PC4)

Commit message: 多分完成
Parts:
- removed H1, H10, H12, H2, H3, H6, H9: MountingHole_Pad, TestPoint:TestPoint_Pad_1.5x1.5mm, symbol Mechanical:MountingHole_Pad
- removed TP1, TP2, TP3, TP4: TestPoint, TestPoint:TestPoint_THTPad_D2.0mm_Drill1.0mm, symbol Connector:TestPoint
Connections:
- no-connect marks 20 -> 22
