File: Mother_Ctrl/Mother_Ctrl.kicad_sch (KiCad schematic)
At the start: 253 parts, among them J1 Conn_01x02_Male, J10 Conn_01x04_Male, J11 Conn_01x04_Male, J12 Conn_01x04_Male, J13 Conn_01x05_Male, J14 Conn_01x05_Male, J15 Conn_01x12_Female, J16 Conn_01x12_Female, J17 Conn_01x12_Female, J2 Conn_01x02_Female, J3 USB_C_Receptacle_USB2.0, J4 Conn_01x07_Female, J5 Conn_01x10_Male, J6 Conn_01x02_Male, J7 Conn_01x03_Male, J8 Conn_01x03_Male, J9 Conn_01x04_Male, Q1 MTP4835I3, Q10 SSM3J332R, Q11 S8050, Q12 S8050, Q13 SSM3J332R, Q14 S8050, Q15 SSM3J332R, Q16 S8050, Q17 SSM3J332R, Q18 S8050, Q19 SSM3J332R, Q2 BSS138, Q20 S8050, Q21 SSM3J332R, Q22 S8050, Q23 BSS138, Q24 BSS138, Q25 BSS138, Q26 BSS138, Q27 BSS138, Q28 BSS138, Q29 MTP4835I3, Q3 MTP4835I3, Q30 S8050, Q31 S8050, Q32 S8050, Q4 SSM3J332R, Q5 S8050, Q6 SSM3J332R, Q7 S8050, Q8 S8050, Q9 SSM3J332R, SW1 SW_SPDT, SW2 SW_SPST, SW3 SW_SPST, SW4 SW_DPDT_x2, SW5 SW_SPDT, SW6 SW_SPST, SW7 SW_SPST, U1 CH340E, U2 TWE-L-WX, U3 AZ1084CD-3.3, U4 STM32F446RETx, U5 BNO055, U6 MAX3485, U7 MAX3485, U8 MAX3485, Y1 16MHz, Y2 32.768kHz

Commit message: 更新
Parts:
- MD1: symbol DCDC_Regulator:OKL-T/6-W12N-C -> DCDC_Regulator:OKL-T/6-W12N-C
Other:
- note added: "Mother_Ctrl"
- moved on the sheet: C1, C10, C11, C12, C13, C14, C15, C16, C17, C18, C19, C2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
