File: Mother_UI/Mother_UI.kicad_pcb (KiCad board)
At the start: 2 copper layers, 100 x 60 mm, 99 parts, among them J1 Conn_01x02_Male, J10 Conn_01x12_Female, J11 Conn_01x12_Female, J2 Conn_01x03_Male, J3 Conn_01x03_Male, J4 Conn_01x03_Male, J5 Conn_01x03_Male, J6 Conn_01x03_Male, J7 Conn_01x03_Male, J8 AudioJack3, J9 Conn_01x12_Female, Q1 S8050, Q2 SSM3J332R, Q3 S8050, SW1 SW_DIP_x05, SW10 SW_SPST, SW11 SW_SPST, SW2 SW_SPDT, SW3 SW_SPST, SW4 SW_SPST, SW5 SW_SPDT, SW6 SW_SPST, SW7 SW_SPDT_White, SW8 SW_SPST, SW9 SW_SPST, U1 OLED_akitsuki, U2 NJM4580

Commit message: 回路図確定
Parts:
- moved H4 41.2 mm to (16.1, 11.5), turned to -90 degrees
- moved LS1 39.4 mm to (33.8, 8.50), turned to 90 degrees
- moved C15 24.1 mm to (15.4, -5.83), turned to -90 degrees
- moved C22 23.2 mm to (15.7, 8.98)
- moved C16 22.5 mm to (15.4, -2.32), turned to -90 degrees
- moved R6 21.2 mm to (13.8, -1.57)
- moved R5 21.2 mm to (13.8, -4.51), turned to 90 degrees
- moved R14 20.0 mm to (15.5, 3.20), turned to 90 degrees
- moved R16 19.6 mm to (15.0, 6.34), turned to -90 degrees
- moved R18 19.3 mm to (18.4, 9.43)
- moved R13 18.0 mm to (16.6, 6.30), turned to 90 degrees
- moved RV1 14.5 mm to (34.0, -5.76)
- moved R10 12.6 mm to (16.8, 3.72), turned to -90 degrees
- moved C19 11.9 mm to (19.7, 2.31), turned to 180 degrees
- moved SW7 11.0 mm to (21.3, -5.51)
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Connections:
- J10 pad 1: unconnected-(J10-Pad1) -> LEDTape1_H
- J10 pad 10: unconnected-(J10-Pad10) -> +5V
- J10 pad 11: unconnected-(J10-Pad11) -> VCC
- J10 pad 12: unconnected-(J10-Pad12) -> +3.3V
- J10 pad 2: unconnected-(J10-Pad2) -> Tact_SW2
- J10 pad 3: unconnected-(J10-Pad3) -> Tact_SW0
- J10 pad 4: unconnected-(J10-Pad4) -> Tact_SW1
- J10 pad 5: unconnected-(J10-Pad5) -> MonitorLED0
- J10 pad 6: unconnected-(J10-Pad6) -> Sensor3
- J10 pad 7: unconnected-(J10-Pad7) -> +3.3V
- J10 pad 8: unconnected-(J10-Pad8) -> DAC
- J10 pad 9: unconnected-(J10-Pad9) -> GND
- J11 pad 1: unconnected-(J11-Pad1) -> I2C1_SDA
- J11 pad 10: unconnected-(J11-Pad10) -> DIP_SW4
- J11 pad 11: unconnected-(J11-Pad11) -> PRG
- J11 pad 12: unconnected-(J11-Pad12) -> RST
- J11 pad 2: unconnected-(J11-Pad2) -> I2C1_SCL
- J11 pad 3: unconnected-(J11-Pad3) -> NeoPixel_H
- J11 pad 4: unconnected-(J11-Pad4) -> LEDTape3_H
- J11 pad 5: unconnected-(J11-Pad5) -> NRST
- J11 pad 6: unconnected-(J11-Pad6) -> DIP_SW0
- J11 pad 7: unconnected-(J11-Pad7) -> DIP_SW1
- J11 pad 8: unconnected-(J11-Pad8) -> DIP_SW2
- J11 pad 9: unconnected-(J11-Pad9) -> DIP_SW3
- J9 pad 1: unconnected-(J9-Pad1) -> LEDTape2_H
- J9 pad 10: unconnected-(J9-Pad10) -> +5V
- J9 pad 11: unconnected-(J9-Pad11) -> GND
- J9 pad 12: unconnected-(J9-Pad12) -> GND
- J9 pad 2: unconnected-(J9-Pad2) -> Slide_SW1
- J9 pad 3: unconnected-(J9-Pad3) -> Slide_SW2
- J9 pad 4: unconnected-(J9-Pad4) -> BOOT0
- J9 pad 5: unconnected-(J9-Pad5) -> Volume
- J9 pad 6: unconnected-(J9-Pad6) -> MonitorLED1
- J9 pad 7: unconnected-(J9-Pad7) -> Sensor1
- J9 pad 8: unconnected-(J9-Pad8) -> Sensor2
- J9 pad 9: unconnected-(J9-Pad9) -> GND
- SW7 pad 1: DAC_Jack -> DAC_Amp
- SW7 pad 3: DAC_Amp -> DAC_Jack
Routing:
- net +5V: track 0.00 -> 571.6 mm, vias 0 -> 2
- net +3.3V: track 0.00 -> 195.7 mm, vias 0 -> 7
- net NeoPixel_H: track 0.00 -> 94.2 mm
- net DIP_SW0: track 0.00 -> 80.0 mm
- net BOOT0: track 0.00 -> 76.5 mm, vias 0 -> 4
- net DIP_SW1: track 0.00 -> 75.8 mm
- net NRST: track 0.00 -> 73.7 mm, vias 0 -> 1
- net Tact_SW0: track 0.00 -> 72.9 mm, vias 0 -> 4
- net DIP_SW2: track 0.00 -> 71.7 mm
- net Sensor1: track 0.00 -> 69.5 mm, vias 0 -> 2
- net DIP_SW3: track 0.00 -> 68.4 mm
- net MonitorLED0: track 0.00 -> 66.9 mm, vias 0 -> 2
- net GNDA: track 0.00 -> 65.6 mm, vias 0 -> 5
- net DIP_SW4: track 0.00 -> 65.0 mm
- net Tact_SW1: track 0.00 -> 64.7 mm, vias 0 -> 4
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- added copper zone on B.Cu, net GND
- added copper zone on F.Cu, net GND
Other:
- board text added: "ADC"

Commit message: 多分完成
Parts:
- C18, C19: value 10uF -> 22uF
- moved R17 172.8 mm to (158.3, 113.5), turned to 90 degrees
- moved SW10 165.4 mm to (112.6, 115.2)
- moved SW9 165.4 mm to (112.6, 104.5)
- moved C15 165.1 mm to (146.7, 94.1)
- moved C18 165.1 mm to (157.2, 102.5)
- moved H4 165.1 mm to (147.4, 111.4)
- moved H7 165.1 mm to (138.3, 119.4)
- moved R13 165.1 mm to (147.9, 106.2)
- moved R15 165.1 mm to (155.5, 110.4)
- moved R16 165.1 mm to (146.3, 106.3)
- moved R9 165.1 mm to (156.7, 105.2)
- moved C1 165.1 mm to (95.1, 112.5)
- moved C10 165.1 mm to (95.1, 82.0)
- moved C11 165.1 mm to (121.3, 115.6)
- moved C12 165.1 mm to (131.3, 115.6)
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Connections:
- LS1 pad 2: GNDA -> GND
- R17 pad 2: GNDA -> GND
Routing:
- net GND: track 0.00 -> 504.6 mm, vias 0 -> 529
- net GNDA: track 65.6 -> 53.2 mm
- net Net-(C21-Pad2): track 15.3 -> 12.5 mm
- net RST: track 53.2 -> 54.5 mm
- net Net-(D20-Pad1): track 0.00 -> 0.73 mm, vias 0 -> 1
- net NRST: track 73.7 -> 73.8 mm, vias 1 -> 2
Other:
- outline, holes or cut-outs redrawn
- board text added: "BOOT0"
- board text added: "Designed by @cat_nekonekone"
- board text added: "JLCJLCJLCJLC"
- board text added: "NRST"
- board text added: "PA5"
- board text added: "PB12"
- board text added: "PB13"
- board text added: "PB14"
- board text added: "PB15"
- board text added: "PB2"
- board text added: "PC8"
- board text added: "POWER"
- board text added: "PRG"
- board text added: "RST"
- board text added: "Tomoshibi"
- board text added: "[5VOUT]"
- board text added: "[Audio]"
- board text added: "[F446]"
- board text added: "[Jack]"
- board text added: "[LEDTape1]"
- board text added: "[LEDTape2]"
- board text added: "[LEDTape3]"
- board text added: "[Piezo]"
- board text added: "[Sensor1]"
- board text added: "[Sensor2]"
- board text added: "[Sensor3]"
- board text added: "[Twe]"
- board text added: "[Volume]"
- board text added: "⇔"
- board text added: "燈"
- board text removed: "ADC"
