File: Mother_UI/Mother_UI.kicad_sch (KiCad schematic)
At the start: 91 parts

Commit message: Pole,Panelほぼ完成
Parts:
- added JP?: Jumper_2_Open, Jumper:SolderJumper-2_P1.3mm_Open_TrianglePad1.0x1.5mm, symbol Jumper:Jumper_2_Open
Connections:
- net DAC_Amp: now also JP?.1 (A); no longer C?.1
- new net: C?.1, JP?.2 (B)
Changed lines of the file:
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@@
     (stroke (width 0) (type default) (color 0 0 0 0))
   )
+  (wire (pts (xy 419.1 106.68) (xy 419.1 111.76))
+    (stroke (width 0) (type default) (color 0 0 0 0))
+  )
   (wire (pts (xy 441.96 83.82) (xy 459.74 83.82))
     (stroke (width 0) (type default) (color 0 0 0 0))
@@
     )
   )
-  (global_label "DAC_Amp" (shape input) (at 429.26 111.76 180) (fields_autoplaced)
-    (effects (font (size 1.27 1.27)) (justify right))
-    (property "Intersheet References" "${INTERSHEET_REFS}" (id 0) (at 418.3198 111.6806 0)
-      (effects (font (size 1.27 1.27)) (justify right) hide)
+  (global_label "DAC_Amp" (shape input) (at 419.1 106.68 90) (fields_autoplaced)
+    (effects (font (size 1.27 1.27)) (justify left))
+    (property "Intersheet References" "${INTERSHEET_REFS}" (id 0) (at 419.1794 95.7398 90)
+      (effects (font (size 1.27 1.27)) (justify left) hide)
     )
   )
@@
     (pin "4")
   )
+  (symbol (lib_id "Jumper:Jumper_2_Open") (at 424.18 111.76 0) (mirror x) (unit 1)
+    (in_bom yes) (on_board yes)
+    (property "Reference" "JP?" (id 0) (at 419.1 114.3 0))
+    (property "Value" "Jumper_2_Open" (id 1) (at 419.1 116.84 0))
+    (property "Footprint" "Jumper:SolderJumper-2_P1.3mm_Open_TrianglePad1.0x1.5mm" (id 2) (at 424.18 111.76 0)
+      (effects (font (size 1.27 1.27)) hide)
+    )
+    (property "Datasheet" "~" (id 3) (at 424.18 111.76 0)
+      (effects (font (size 1.27 1.27)) hide)
+    )
+    (pin "1")
+    (pin "2")
+  )
   (symbol (lib_id "Device:R") (at 271.78 187.96 0) (unit 1)
     (in_bom yes) (on_board yes) (fields_autoplaced)
@@
       (reference "J?") (unit 1) (value "Conn_01x03_Male") (footprint "Connector_Molex:Molex_SPOX_5268-03A_1x03_P2.50mm_Horizontal")
     )
+    (path "/e7bfcf16-7384-4a33-aa97-410fcba289c4"
+      (reference "JP?") (unit 1) (value "Jumper_2_Open") (footprint "Jumper:SolderJumper-2_P1.3mm_Open_TrianglePad1.0x1.5mm")
+    )
     (path "/1a9015a7-f340-4352-ad13-52eafb6996a4"

Commit message: Mother_Ctrl回路図プロット
Parts:
- added J1: Conn_01x02_Male, Connector_Molex:Molex_SPOX_5268-02A_1x02_P2.50mm_Horizontal, symbol Connector:Conn_01x02_Male
- added J10, J11, J9: Conn_01x12_Female, Connector_PinHeader_2.54mm:PinHeader_1x12_P2.54mm_Vertical, symbol Connector:Conn_01x12_Female
- added Q1, Q3: S8050, Package_TO_SOT_SMD:SOT-23, symbol Device:Q_PNP_BEC
- added Q2: SSM3J332R, Package_TO_SOT_SMD:SOT-23W, symbol Device:Q_PMOS_GSD
- added R7, R8: 10k, Resistor_SMD:R_0402_1005Metric, symbol Device:R
- R1, R2: renamed from R?; value R -> PullUP
- U2: renamed from U?; footprint (none) -> Package_SO:SOP-8_3.9x4.9mm_P1.27mm
- gave numbers to parts that had none: 87
Connections:
- net +5V: now also Q1.2 (E), Q2.3 (D)
- net GND: now also J1.1 (Pin_1), R7.1, R8.1
- new net: J1.2 (Pin_2), Q2.2 (S), Q3.2 (E)
- new net: Q2.1 (G), Q3.3 (C), R8.2
- new net: Q1.1 (B), Q1.3 (C), Q3.1 (B), R7.2
Other:
- note added: "5V出力"

Commit message: 回路図確定
Connections:
- net +3.3V: now also J10.12 (Pin_12), J10.7 (Pin_7)
- net +5V: now also J10.10 (Pin_10), J9.10 (Pin_10)
- net BOOT0: now also J9.4 (Pin_4)
- net DAC: now also J10.8 (Pin_8)
- net DAC_Amp: now also SW7.1 (A); no longer SW7.3 (C)
- net DAC_Jack: now also SW7.3 (C); no longer SW7.1 (A)
- net DIP_SW0: now also J11.6 (Pin_6)
- net DIP_SW1: now also J11.7 (Pin_7)
- net DIP_SW2: now also J11.8 (Pin_8)
- net DIP_SW3: now also J11.9 (Pin_9)
- net DIP_SW4: now also J11.10 (Pin_10)
- net GND: now also J10.9 (Pin_9), J9.11 (Pin_11), J9.12 (Pin_12), J9.9 (Pin_9)
- net I2C1_SCL: now also J11.2 (Pin_2)
- net I2C1_SDA: now also J11.1 (Pin_1)
- net LEDTape1_H: now also J10.1 (Pin_1)
- net LEDTape2_H: now also J9.1 (Pin_1)
- net LEDTape3_H: now also J11.4 (Pin_4)
- net MonitorLED0: now also J10.5 (Pin_5)
- net MonitorLED1: now also J9.6 (Pin_6)
- net NRST: now also J11.5 (Pin_5)
- net NeoPixel_H: now also J11.3 (Pin_3)
- net PRG: now also J11.11 (Pin_11)
- net RST: now also J11.12 (Pin_12)
- net Sensor1: now also J9.7 (Pin_7)
- net Sensor2: now also J9.8 (Pin_8)
- net Sensor3: now also J10.6 (Pin_6)
- net Slide_SW1: now also J9.2 (Pin_2)
- net Slide_SW2: now also J9.3 (Pin_3)
- net Tact_SW0: now also J10.3 (Pin_3)
- net Tact_SW1: now also J10.4 (Pin_4)
- net Tact_SW2: now also J10.2 (Pin_2)
- net VCC: now also J10.11 (Pin_11)
- net Volume: now also J9.5 (Pin_5)
Other:
- note added: "基板間コネクタ"
- moved on the sheet: J10, J11, J9

Commit message: 多分完成
Parts:
- C18, C19: value 10uF -> 22uF
Connections:
- net GND: now also LS1.2, R17.2
- net GNDA: no longer LS1.2, R17.2
Changed lines of the file:
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@@
       (effects (font (size 1.27 1.27)) (justify right))
     )
-    (property "Value" "10uF" (id 1) (at 431.8 106.68 90)
+    (property "Value" "22uF" (id 1) (at 431.8 106.68 90)
       (effects (font (size 1.27 1.27)) (justify right))
     )
@@
     (pin "3")
     (pin "4")
+  )
+  (symbol (lib_id "power:GND") (at 480.06 88.9 0) (unit 1)
+    (in_bom yes) (on_board yes) (fields_autoplaced)
+    (property "Reference" "#PWR0104" (id 0) (at 480.06 95.25 0)
+      (effects (font (size 1.27 1.27)) hide)
+    )
+    (property "Value" "GND" (id 1) (at 480.06 93.98 0))
+    (property "Footprint" "" (id 2) (at 480.06 88.9 0)
+      (effects (font (size 1.27 1.27)) hide)
+    )
+    (property "Datasheet" "" (id 3) (at 480.06 88.9 0)
+      (effects (font (size 1.27 1.27)) hide)
+    )
+    (pin "1")
   )
   (symbol (lib_id "power:GND") (at 530.86 213.36 0) (unit 1)
@@
     (pin "2")
   )
-  (symbol (lib_id "power:GNDA") (at 480.06 88.9 0) (unit 1)
-    (in_bom yes) (on_board yes)
-    (property "Reference" "#PWR045" (id 0) (at 480.06 95.25 0)
-      (effects (font (size 1.27 1.27)) hide)
-    )
-    (property "Value" "GNDA" (id 1) (at 480.06 93.98 0)
-      (effects (font (size 1.27 1.27)) (justify right))
-    )
-    (property "Footprint" "" (id 2) (at 480.06 88.9 0)
-      (effects (font (size 1.27 1.27)) hide)
-    )
-    (property "Datasheet" "" (id 3) (at 480.06 88.9 0)
-      (effects (font (size 1.27 1.27)) hide)
-    )
-    (pin "1")
-  )
   (symbol (lib_id "power:+3.3V") (at 292.1 180.34 0) (unit 1)
     (in_bom yes) (on_board yes)
@@
       (effects (font (size 1.27 1.27)) (justify right))
     )
-    (property "Value" "10uF" (id 1) (at 431.8 66.04 90)
+    (property "Value" "22uF" (id 1) (at 431.8 66.04 90)
       (effects (font (size 1.27 1.27)) (justify right))
     )
@@
       (reference "#PWR044") (unit 1) (value "GNDA") (footprint "")
     )
-    (path "/ecab8b42-20bf-4b91-b2d7-d657e95a68b5"
-      (reference "#PWR045") (unit 1) (value "GNDA") (footprint "")
-    )
     (path "/84f5a7da-a731-4739-9b3b-28fa7277dc65"
       (reference "#PWR046") (unit 1) (value "GNDA") (footprint "")
@@
       (reference "#PWR0103") (unit 1) (value "GND") (footprint "")
     )
+    (path "/a86b5b23-e7e2-48ad-96ac-4f2cb146d0a5"
+      (reference "#PWR0104") (unit 1) (value "GND") (footprint "")
+    )
     (path "/1173bd26-6417-437e-99c9-f5de4ec2c918"
       (reference "C1") (unit 1) (value "0.1uF") (footprint "Capacitor_SMD:C_0402_1005Metric")
@@
     )
     (path "/f6463945-e188-45a2-a284-543db507e5d9"
-      (reference "C18") (unit 1) (value "10uF") (footprint "Capacitor_SMD:C_0805_2012Metric")
+      (reference "C18") (unit 1) (value "22uF") (footprint "Capacitor_SMD:C_0805_2012Metric")
     )
     (path "/6b7c9542-a680-4735-9779-29dc44fb5274"
-      (reference "C19") (unit 1) (value "10uF") (footprint "Capacitor_SMD:C_0805_2012Metric")
+      (reference "C19") (unit 1) (value "22uF") (footprint "Capacitor_SMD:C_0805_2012Metric")
     )
     (path "/3f1b5640-c814-4193-b145-922f3a795c5e"
